File: Chronos.sch (KiCad schematic (older format))
At the start: 13 parts, among them U1 ATMEGA32U2-AU, Y1 16MHz

Commit message: Finish setting up most of controller
Also added RGB LED cluster
Todo: RGB LED decoupling caps
Parts:
- added RGB1, RGB10, RGB11, RGB12, RGB13, RGB14, RGB2, RGB3, RGB4, RGB5, RGB6, RGB7, RGB8, RGB9: WS2812B, symbol WS2812B
- Q1: renamed from Q?; value BCP51 -> NSS40301MZ4T1G
Connections:
- net +5V: now also RGB1.1 (VCC), RGB10.1 (VCC), RGB11.1 (VCC), RGB12.1 (VCC), RGB13.1 (VCC), RGB14.1 (VCC), RGB2.1 (VCC), RGB3.1 (VCC), RGB4.1 (VCC), RGB5.1 (VCC), RGB6.1 (VCC), RGB7.1 (VCC), RGB8.1 (VCC), RGB9.1 (VCC)
- net GND: now also RGB1.3 (GND), RGB10.3 (GND), RGB11.3 (GND), RGB12.3 (GND), RGB13.3 (GND), RGB14.3 (GND), RGB2.3 (GND), RGB3.3 (GND), RGB4.3 (GND), RGB5.3 (GND), RGB6.3 (GND), RGB7.3 (GND), RGB8.3 (GND), RGB9.3 (GND)
- new net: RGB1.2 (DOUT), RGB2.4 (DIN)
- new net: RGB2.2 (DOUT), RGB3.4 (DIN)
- new net: RGB3.2 (DOUT), RGB4.4 (DIN)
- new net: RGB4.2 (DOUT), RGB5.4 (DIN)
- new net: RGB5.2 (DOUT), RGB6.4 (DIN)
- new net: RGB6.2 (DOUT), RGB7.4 (DIN)
- new net: RGB7.2 (DOUT), RGB8.4 (DIN)
- new net: RGB8.2 (DOUT), RGB9.4 (DIN)
- new net: RGB10.4 (DIN), RGB9.2 (DOUT)
- new net: RGB10.2 (DOUT), RGB11.4 (DIN)
- new net: RGB11.2 (DOUT), RGB12.4 (DIN)
- new net: RGB12.2 (DOUT), RGB13.4 (DIN)
- new net: RGB13.2 (DOUT), RGB14.4 (DIN)
- new net RGBLED: RGB1.4 (DIN)
- no-connect marks 1 -> 2
Other:
- moved on the sheet: C1, C2, C3, F1, Q1, R1, R2, R3, R4, R5, U1, USB1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

Commit message: Create matrix sheet
Also fill out sheet descriptors
Other:
- note added: "2017-10-15\n"
- note added: "Chronos Keyboard\n"
Changed lines of the file:
@@
 F1 "Matrix.sch" 60
 $EndSheet
+Text Notes 7350 7500 0    60   ~ 0
+Chronos Keyboard\n
+Text Notes 8125 7650 0    60   ~ 0
+2017-10-15\n
 $EndSCHEMATC

Commit message: Add RGB Decoupling capacitors
Also fix label on matrix sheet being misplaced
Parts:
- added CR1, CR10, CR11, CR12, CR13, CR14, CR2, CR3, CR4, CR5, CR6, CR7, CR8, CR9: 0.1u, symbol C_Small
Connections:
- net +5V: now also CR1.1, CR10.1, CR11.1, CR12.1, CR13.1, CR14.1, CR2.1, CR3.1, CR4.1, CR5.1, CR6.1, CR7.1, CR8.1, CR9.1
- net GND: now also CR1.2, CR10.2, CR11.2, CR12.2, CR13.2, CR14.2, CR2.2, CR3.2, CR4.2, CR5.2, CR6.2, CR7.2, CR8.2, CR9.2
Changed lines of the file:
@@
 Text Notes 8125 7650 0    60   ~ 0
 2017-10-15\n
+$Comp
+L C_Small CR1
+U 1 1 59E874F1
+P 6450 925
+F 0 "CR1" H 6460 995 50  0000 L CNN
+F 1 "0.1u" H 6460 845 50  0000 L CNN
+F 2 "" H 6450 925 50  0001 C CNN
+F 3 "" H 6450 925 50  0001 C CNN
+	1    6450 925
+	1    0    0    -1
+$EndComp
+$Comp
+L C_Small CR2
+U 1 1 59E879A6
+P 6650 925
+F 0 "CR2" H 6660 995 50  0000 L CNN
+F 1 "0.1u" H 6660 845 50  0000 L CNN
+F 2 "" H 6650 925 50  0001 C CNN
+F 3 "" H 6650 925 50  0001 C CNN
+	1    6650 925
+	1    0    0    -1
+$EndComp
+$Comp
+L C_Small CR3
+U 1 1 59E87A25
+P 6850 925
+F 0 "CR3" H 6860 995 50  0000 L CNN
+F 1 "0.1u" H 6860 845 50  0000 L CNN
+F 2 "" H 6850 925 50  0001 C CNN
+F 3 "" H 6850 925 50  0001 C CNN
+	1    6850 925
+	1    0    0    -1
+$EndComp
+$Comp
+L C_Small CR4
+U 1 1 59E87A9B
+P 7050 925
+F 0 "CR4" H 7060 995 50  0000 L CNN
+F 1 "0.1u" H 7060 845 50  0000 L CNN
+F 2 "" H 7050 925 50  0001 C CNN
+F 3 "" H 7050 925 50  0001 C CNN
+	1    7050 925
+	1    0    0    -1
+$EndComp
+$Comp
+L C_Small CR5
+U 1 1 59E87B14
+P 7250 925
+F 0 "CR5" H 7260 995 50  0000 L CNN
+F 1 "0.1u" H 7260 845 50  0000 L CNN
+F 2 "" H 7250 925 50  0001 C CNN
+F 3 "" H 7250 925 50  0001 C CNN
+	1    7250 925
+	1    0    0    -1
+$EndComp
+$Comp
+L C_Small CR6
+U 1 1 59E87B94
+P 7450 925
+F 0 "CR6" H 7460 995 50  0000 L CNN
+F 1 "0.1u" H 7460 845 50  0000 L CNN
+F 2 "" H 7450 925 50  0001 C CNN
+F 3 "" H 7450 925 50  0001 C CNN
+	1    7450 925
+	1    0    0    -1
+$EndComp
+$Comp
+L C_Small CR7
+U 1 1 59E87C1F
+P 7650 925
+F 0 "CR7" H 7660 995 50  0000 L CNN
+F 1 "0.1u" H 7660 845 50  0000 L CNN
+F 2 "" H 7650 925 50  0001 C CNN
+F 3 "" H 7650 925 50  0001 C CNN
+	1    7650 925
+	1    0    0    -1
+$EndComp
+Wire Wire Line
+	6350 825  7650 825
+Connection ~ 7450 825
+Connection ~ 7250 825
+Connection ~ 7050 825
+Connection ~ 6850 825
+Connection ~ 6650 825
+$Comp
+L +5V #PWR?
+U 1 1 59E88354
+P 6350 825
+F 0 "#PWR?" H 6350 675 50  0001 C CNN
+F 1 "+5V" H 6350 965 50  0000 C CNN
+F 2 "" H 6350 825 50  0001 C CNN
+F 3 "" H 6350 825 50  0001 C CNN
+	1    6350 825
+	0    -1   -1   0
+$EndComp
+Connection ~ 6450 825
+$Comp
+L GND #PWR?
+U 1 1 59E88464
+P 6350 1025
+F 0 "#PWR?" H 6350 775 50  0001 C CNN
+F 1 "GND" H 6350 875 50  0000 C CNN
+F 2 "" H 6350 1025 50  0001 C CNN
+F 3 "" H 6350 1025 50  0001 C CNN
+	1    6350 1025
+	0    1    1    0
+$EndComp
+Wire Wire Line
+	6350 1025 7650 1025
+Connection ~ 6450 1025
+Connection ~ 6650 1025
+Connection ~ 6850 1025
+Connection ~ 7050 1025
+Connection ~ 7250 1025
+Connection ~ 7450 1025
+$Comp
+L C_Small CR8
+U 1 1 59E89B67
+P 6450 1325
+F 0 "CR8" H 6460 1395 50  0000 L CNN
+F 1 "0.1u" H 6460 1245 50  0000 L CNN
+F 2 "" H 6450 1325 50  0001 C CNN
+F 3 "" H 6450 1325 50  0001 C CNN
+	1    6450 1325
+	1    0    0    -1
+$EndComp
+$Comp
+L C_Small CR9
+U 1 1 59E89B6D
+P 6650 1325
+F 0 "CR9" H 6660 1395 50  0000 L CNN
+F 1 "0.1u" H 6660 1245 50  0000 L CNN
+F 2 "" H 6650 1325 50  0001 C CNN
+F 3 "" H 6650 1325 50  0001 C CNN
+	1    6650 1325
+	1    0    0    -1
+$EndComp
+$Comp
+L C_Small CR10
+U 1 1 59E89B73
+P 6850 1325
+F 0 "CR10" H 6860 1395 50  0000 L CNN
+F 1 "0.1u" H 6860 1245 50  0000 L CNN
+F 2 "" H 6850 1325 50  0001 C CNN
+F 3 "" H 6850 1325 50  0001 C CNN
+	1    6850 1325
+	1    0    0    -1
+$EndComp
+$Comp
+L C_Small CR11
+U 1 1 59E89B79
+P 7050 1325
+F 0 "CR11" H 7060 1395 50  0000 L CNN
+F 1 "0.1u" H 7060 1245 50  0000 L CNN
+F 2 "" H 7050 1325 50  0001 C CNN
+F 3 "" H 7050 1325 50  0001 C CNN
+	1    7050 1325
+	1    0    0    -1
+$EndComp
+$Comp
+L C_Small CR12
+U 1 1 59E89B7F
+P 7250 1325
+F 0 "CR12" H 7260 1395 50  0000 L CNN
+F 1 "0.1u" H 7260 1245 50  0000 L CNN
+F 2 "" H 7250 1325 50  0001 C CNN
+F 3 "" H 7250 1325 50  0001 C CNN
+	1    7250 1325
+	1    0    0    -1
+$EndComp
+$Comp
+L C_Small CR13
+U 1 1 59E89B85
+P 7450 1325
+F 0 "CR13" H 7460 1395 50  0000 L CNN
+F 1 "0.1u" H 7460 1245 50  0000 L CNN
+F 2 "" H 7450 1325 50  0001 C CNN
+F 3 "" H 7450 1325 50  0001 C CNN
+	1    7450 1325
+	1    0    0    -1
+$EndComp
+$Comp
+L C_Small CR14
+U 1 1 59E89B8B
+P 7650 1325
+F 0 "CR14" H 7660 1395 50  0000 L CNN
+F 1 "0.1u" H 7660 1245 50  0000 L CNN
+F 2 "" H 7650 1325 50  0001 C CNN
+F 3 "" H 7650 1325 50  0001 C CNN
+	1    7650 1325
+	1    0    0    -1
+$EndComp
+Wire Wire Line
+	6350 1225 7650 1225
+Connection ~ 7450 1225
+Connection ~ 7250 1225
+Connection ~ 7050 1225
+Connection ~ 6850 1225
+Connection ~ 6650 1225
+$Comp
+L +5V #PWR?
+U 1 1 59E89B97
+P 6350 1225
+F 0 "#PWR?" H 6350 1075 50  0001 C CNN
+F 1 "+5V" H 6350 1365 50  0000 C CNN
+F 2 "" H 6350 1225 50  0001 C CNN
+F 3 "" H 6350 1225 50  0001 C CNN
+	1    6350 1225
+	0    -1   -1   0
+$EndComp
+Connection ~ 6450 1225
+$Comp
+L GND #PWR?
+U 1 1 59E89B9E
+P 6350 1425
+F 0 "#PWR?" H 6350 1175 50  0001 C CNN
+F 1 "GND" H 6350 1275 50  0000 C CNN
+F 2 "" H 6350 1425 50  0001 C CNN
+F 3 "" H 6350 1425 50  0001 C CNN
+	1    6350 1425
+	0    1    1    0
+$EndComp
+Wire Wire Line
+	6350 1425 7650 1425
+Connection ~ 6450 1425
+Connection ~ 6650 1425
+Connection ~ 6850 1425
+Connection ~ 7050 1425
+Connection ~ 7250 1425
+Connection ~ 7450 1425
 $EndSCHEMATC

Commit message: Begin footprint associations with lib parts
Parts:
- added C4, C5: 0.1u, symbol C_Small
- added C6: 4.7u, symbol C_Small
- U1: footprint TQFP-32 -> (none)
Connections:
- net +5V: now also C4.1, C5.1, C6.1
- net GND: now also C4.2, C5.2, C6.2
Changed lines of the file:
@@
 F 0 "U1" H 2300 4350 50  0000 C CNN
 F 1 "ATMEGA32U2-AU" H 3900 1650 50  0000 C CNN
-F 2 "TQFP-32" H 3000 3050 50  0001 C CNN
+F 2 "" H 3000 3050 50  0001 C CNN
 F 3 "http://www.atmel.com/Images/doc7799.pdf" H 3250 1550 50  0001 C CNN
 	1    3150 3000
@@
 $EndComp
 $Comp
-L GND #PWR?
+L GND #PWR01
 U 1 1 59E55E19
 P 1325 2800
-F 0 "#PWR?" H 1325 2550 50  0001 C CNN
+F 0 "#PWR01" H 1325 2550 50  0001 C CNN
 F 1 "GND" H 1325 2650 50  0000 C CNN
 F 2 "" H 1325 2800 50  0001 C CNN
@@
 $EndComp
 $Comp
-L +5V #PWR?
+L +5V #PWR02
 U 1 1 59E56D55
 P 1950 2400
-F 0 "#PWR?" H 1950 2250 50  0001 C CNN
+F 0 "#PWR02" H 1950 2250 50  0001 C CNN
 F 1 "+5V" V 1950 2600 50  0000 C CNN
 F 2 "" H 1950 2400 50  0001 C CNN
@@
 $EndComp
 $Comp
-L +5V #PWR?
+L +5V #PWR03
 U 1 1 59E5754C
 P 1450 2300
-F 0 "#PWR?" H 1450 2150 50  0001 C CNN
+F 0 "#PWR03" H 1450 2150 50  0001 C CNN
 F 1 "+5V" V 1525 2375 50  0000 C CNN
 F 2 "" H 1450 2300 50  0001 C CNN
@@
 $EndComp
 $Comp
-L GND #PWR?
+L GND #PWR04
 U 1 1 59E58833
 P 1450 3200
-F 0 "#PWR?" H 1450 2950 50  0001 C CNN
+F 0 "#PWR04" H 1450 2950 50  0001 C CNN
 F 1 "GND" V 1450 3000 50  0000 C CNN
 F 2 "" H 1450 3200 50  0001 C CNN
@@
 $EndComp
 $Comp
-L +5V #PWR?
+L +5V #PWR05
 U 1 1 59E58E5F
 P 1450 3300
-F 0 "#PWR?" H 1450 3150 50  0001 C CNN
+F 0 "#PWR05" H 1450 3150 50  0001 C CNN
 F 1 "+5V" V 1450 3500 50  0000 C CNN
 F 2 "" H 1450 3300 50  0001 C CNN
@@
 DM
 $Comp
-L GND #PWR?
+L GND #PWR06
 U 1 1 59E5A934
 P 1950 3600
-F 0 "#PWR?" H 1950 3350 50  0001 C CNN
+F 0 "#PWR06" H 1950 3350 50  0001 C CNN
 F 1 "GND" V 1950 3400 50  0000 C CNN
 F 2 "" H 1950 3600 50  0001 C CNN
@@
 $EndComp
 $Comp
-L VCC #PWR?
+L VCC #PWR07
 U 1 1 59E5C00E
 P 1300 4100
-F 0 "#PWR?" H 1300 3950 50  0001 C CNN
+F 0 "#PWR07" H 1300 3950 50  0001 C CNN
 F 1 "VCC" H 1300 4250 50  0000 C CNN
 F 2 "" H 1300 4100 50  0001 C CNN
@@
 $EndComp
 $Comp
-L +5V #PWR?
+L +5V #PWR08
 U 1 1 59E5C9FB
 P 1800 4100
-F 0 "#PWR?" H 1800 3950 50  0001 C CNN
+F 0 "#PWR08" H 1800 3950 50  0001 C CNN
 F 1 "+5V" H 1800 4240 50  0000 C CNN
 F 2 "" H 1800 4100 50  0001 C CNN
@@
 NoConn ~ 1250 4400
 $Comp
-L GND #PWR?
+L GND #PWR09
 U 1 1 59E5DE55
 P 1350 4500
-F 0 "#PWR?" H 1350 4250 50  0001 C CNN
+F 0 "#PWR09" H 1350 4250 50  0001 C CNN
 F 1 "GND" H 1350 4350 50  0000 C CNN
 F 2 "" H 1350 4500 50  0001 C CNN
@@
 $EndComp
 $Comp
-L GND #PWR?
+L GND #PWR010
 U 1 1 59E5EC47
 P 3150 4500
-F 0 "#PWR?" H 3150 4250 50  0001 C CNN
+F 0 "#PWR010" H 3150 4250 50  0001 C CNN
 F 1 "GND" H 3150 4350 50  0000 C CNN
 F 2 "" H 3150 4500 50  0001 C CNN
@@
 $EndComp
 $Comp
-L +5V #PWR?
+L +5V #PWR011
 U 1 1 59E5EF79
 P 3150 1500
-F 0 "#PWR?" H 3150 1350 50  0001 C CNN
+F 0 "#PWR011" H 3150 1350 50  0001 C CNN
 F 1 "+5V" H 3150 1640 50  0000 C CNN
 F 2 "" H 3150 1500 50  0001 C CNN
@@
 LEDGND
 $Comp
-L GND #PWR?
+L GND #PWR012
 U 1 1 59E62F25
 P 5475 2300
-F 0 "#PWR?" H 5475 2050 50  0001 C CNN
+F 0 "#PWR012" H 5475 2050 50  0001 C CNN
 F 1 "GND" V 5475 2100 50  0000 C CNN
 F 2 "" H 5475 2300 50  0001 C CNN
@@
 $EndComp
 $Comp
-L GND #PWR?
+L GND #PWR013
 U 1 1 59E64F31
 P 5175 3500
-F 0 "#PWR?" H 5175 3250 50  0001 C CNN
+F 0 "#PWR013" H 5175 3250 50  0001 C CNN
 F 1 "GND" V 5175 3300 50  0000 C CNN
 F 2 "" H 5175 3500 50  0001 C CNN
@@
 F 0 "RGB1" H 8750 1625 60  0000 C CNN
 F 1 "WS2812B" H 9150 1625 60  0000 C CNN
-F 2 "" V 8900 1275 60  0000 C CNN
+F 2 "" V 8900 1275 60  0001 C CNN
 F 3 "" V 8900 1275 60  0000 C CNN
 	1    8950 1275
@@
 F 0 "RGB2" H 8750 2350 60  0000 C CNN
 F 1 "WS2812B" H 9150 2350 60  0000 C CNN
-F 2 "" V 8900 2000 60  0000 C CNN
+F 2 "" V 8900 2000 60  0001 C CNN
 F 3 "" V 8900 2000 60  0000 C CNN
 	1    8950 2000
@@
 F 0 "RGB3" H 8750 3075 60  0000 C CNN
 F 1 "WS2812B" H 9150 3075 60  0000 C CNN
-F 2 "" V 8900 2725 60  0000 C CNN
+F 2 "" V 8900 2725 60  0001 C CNN
 F 3 "" V 8900 2725 60  0000 C CNN
 	1    8950 2725
@@
 F 0 "RGB4" H 8750 3800 60  0000 C CNN
 F 1 "WS2812B" H 9150 3800 60  0000 C CNN
-F 2 "" V 8900 3450 60  0000 C CNN
+F 2 "" V 8900 3450 60  0001 C CNN
 F 3 "" V 8900 3450 60  0000 C CNN
 	1    8950 3450
@@
 F 0 "RGB5" H 8750 4525 60  0000 C CNN
 F 1 "WS2812B" H 9150 4525 60  0000 C CNN
-F 2 "" V 8900 4175 60  0000 C CNN
+F 2 "" V 8900 4175 60  0001 C CNN
 F 3 "" V 8900 4175 60  0000 C CNN
 	1    8950 4175
@@
 F 0 "RGB6" H 8750 5250 60  0000 C CNN
 F 1 "WS2812B" H 9150 5250 60  0000 C CNN
-F 2 "" V 8900 4900 60  0000 C CNN
+F 2 "" V 8900 4900 60  0001 C CNN
 F 3 "" V 8900 4900 60  0000 C CNN
 	1    8950 4900
@@
 F 0 "RGB7" H 8750 5975 60  0000 C CNN
 F 1 "WS2812B" H 9150 5975 60  0000 C CNN
-F 2 "" V 8900 5625 60  0000 C CNN
+F 2 "" V 8900 5625 60  0001 C CNN
 F 3 "" V 8900 5625 60  0000 C CNN
 	1    8950 5625
@@
 F 0 "RGB8" H 10000 1625 60  0000 C CNN
 F 1 "WS2812B" H 10400 1625 60  0000 C CNN
-F 2 "" V 10150 1275 60  0000 C CNN
+F 2 "" V 10150 1275 60  0001 C CNN
 F 3 "" V 10150 1275 60  0000 C CNN
 	1    10200 1275
@@
 F 0 "RGB9" H 10000 2350 60  0000 C CNN
 F 1 "WS2812B" H 10400 2350 60  0000 C CNN
-F 2 "" V 10150 2000 60  0000 C CNN
+F 2 "" V 10150 2000 60  0001 C CNN
 F 3 "" V 10150 2000 60  0000 C CNN
 	1    10200 2000
@@
 F 0 "RGB10" H 10000 3075 60  0000 C CNN
 F 1 "WS2812B" H 10400 3075 60  0000 C CNN
-F 2 "" V 10150 2725 60  0000 C CNN
+F 2 "" V 10150 2725 60  0001 C CNN
 F 3 "" V 10150 2725 60  0000 C CNN
 	1    10200 2725
@@
 F 0 "RGB11" H 10000 3800 60  0000 C CNN
 F 1 "WS2812B" H 10400 3800 60  0000 C CNN
-F 2 "" V 10150 3450 60  0000 C CNN
+F 2 "" V 10150 3450 60  0001 C CNN
 F 3 "" V 10150 3450 60  0000 C CNN
 	1    10200 3450
@@
 F 0 "RGB12" H 10000 4525 60  0000 C CNN
 F 1 "WS2812B" H 10400 4525 60  0000 C CNN
-F 2 "" V 10150 4175 60  0000 C CNN
+F 2 "" V 10150 4175 60  0001 C CNN
 F 3 "" V 10150 4175 60  0000 C CNN
 	1    10200 4175
@@
 F 0 "RGB13" H 10000 5250 60  0000 C CNN
 F 1 "WS2812B" H 10400 5250 60  0000 C CNN
-F 2 "" V 10150 4900 60  0000 C CNN
+F 2 "" V 10150 4900 60  0001 C CNN
 F 3 "" V 10150 4900 60  0000 C CNN
 	1    10200 4900
@@
 F 0 "RGB14" H 10000 5975 60  0000 C CNN
 F 1 "WS2812B" H 10400 5975 60  0000 C CNN
-F 2 "" V 10150 5625 60  0000 C CNN
+F 2 "" V 10150 5625 60  0001 C CNN
 F 3 "" V 10150 5625 60  0000 C CNN
 	1    10200 5625
@@
 	9450 775  9450 1075
 $Comp
-L GND #PWR?
+L GND #PWR014
 U 1 1 59E7779D
 P 9500 1375
-F 0 "#PWR?" H 9500 1125 50  0001 C CNN
+F 0 "#PWR014" H 9500 1125 50  0001 C CNN
 F 1 "GND" H 9500 1225 50  0000 C CNN
 F 2 "" H 9500 1375 50  0001 C CNN
@@
 Connection ~ 9500 1475
 $Comp
-L +5V #PWR?
+L +5V #PWR015
 U 1 1 59E77CFF
 P 8400 975
-F 0 "#PWR?" H 8400 825 50  0001 C CNN
+F 0 "#PWR015" H 8400 825 50  0001 C CNN
 F 1 "+5V" H 8400 1115 50  0000 C CNN
 F 2 "" H 8400 975 50  0001 C CNN
@@
 Connection ~ 9650 1800
 $Comp
-L +5V #PWR?
+L +5V #PWR016
 U 1 1 59E7D630
 P 9650 975
-F 0 "#PWR?" H 9650 825 50  0001 C CNN
+F 0 "#PWR016" H 9650 825 50  0001 C CNN
 F 1 "+5V" H 9650 1115 50  0000 C CNN
 F 2 "" H 9650 975 50  0001 C CNN
@@
 NoConn ~ 9700 5825
 $Comp
-L GND #PWR?
+L GND #PWR017
 U 1 1 59E81253
 P 10750 1375
-F 0 "#PWR?" H 10750 1125 50  0001 C CNN
+F 0 "#PWR017" H 10750 1125 50  0001 C CNN
 F 1 "GND" H 10750 1225 50  0000 C CNN
 F 2 "" H 10750 1375 50  0001 C CNN
@@
 Connection ~ 6650 825
 $Comp
-L +5V #PWR?
+L +5V #PWR018
 U 1 1 59E88354
 P 6350 825
-F 0 "#PWR?" H 6350 675 50  0001 C CNN
+F 0 "#PWR018" H 6350 675 50  0001 C CNN
 F 1 "+5V" H 6350 965 50  0000 C CNN
 F 2 "" H 6350 825 50  0001 C CNN
@@
 Connection ~ 6450 825
 $Comp
-L GND #PWR?
+L GND #PWR019
 U 1 1 59E88464
 P 6350 1025
-F 0 "#PWR?" H 6350 775 50  0001 C CNN
+F 0 "#PWR019" H 6350 775 50  0001 C CNN
 F 1 "GND" H 6350 875 50  0000 C CNN
 F 2 "" H 6350 1025 50  0001 C CNN
@@
 Connection ~ 6650 1225
 $Comp
-L +5V #PWR?
+L +5V #PWR020
 U 1 1 59E89B97
 P 6350 1225
-F 0 "#PWR?" H 6350 1075 50  0001 C CNN
+F 0 "#PWR020" H 6350 1075 50  0001 C CNN
 F 1 "+5V" H 6350 1365 50  0000 C CNN
 F 2 "" H 6350 1225 50  0001 C CNN
@@
 Connection ~ 6450 1225
 $Comp
-L GND #PWR?
+L GND #PWR021
 U 1 1 59E89B9E
 P 6350 1425
-F 0 "#PWR?" H 6350 1175 50  0001 C CNN
+F 0 "#PWR021" H 6350 1175 50  0001 C CNN
 F 1 "GND" H 6350 1275 50  0000 C CNN
 F 2 "" H 6350 1425 50  0001 C CNN
@@
 Connection ~ 7250 1425
 Connection ~ 7450 1425
+$Comp
+L C_Small C4
+U 1 1 59E71603
+P 1025 1175
+F 0 "C4" H 1035 1245 50  0000 L CNN
+F 1 "0.1u" H 1035 1095 50  0000 L CNN
+F 2 "" H 1025 1175 50  0001 C CNN
+F 3 "" H 1025 1175 50  0001 C CNN
+	1    1025 1175
+	-1   0    0    -1
+$EndComp
+$Comp
+L C_Small C5
+U 1 1 59E7418D
+P 1225 1175
+F 0 "C5" H 1235 1245 50  0000 L CNN
+F 1 "0.1u" H 1235 1095 50  0000 L CNN
+F 2 "" H 1225 1175 50  0001 C CNN
+F 3 "" H 1225 1175 50  0001 C CNN
+	1    1225 1175
+	-1   0    0    -1
+$EndComp
+$Comp
+L C_Small C6
+U 1 1 59E7422A
+P 1425 1175
+F 0 "C6" H 1435 1245 50  0000 L CNN
+F 1 "4.7u" H 1435 1095 50  0000 L CNN
+F 2 "" H 1425 1175 50  0001 C CNN
+F 3 "" H 1425 1175 50  0001 C CNN
+	1    1425 1175
+	-1   0    0    -1
+$EndComp
+Wire Wire Line
+	1025 1075 1425 1075
+Connection ~ 1225 1075
+Wire Wire Line
+	1025 1275 1425 1275
+Connection ~ 1225 1275
+$Comp
+L +5V #PWR?
+U 1 1 59E74DA6
+P 1225 975
+F 0 "#PWR?" H 1225 825 50  0001 C CNN
+F 1 "+5V" H 1225 1115 50  0000 C CNN
+F 2 "" H 1225 975 50  0001 C CNN
+F 3 "" H 1225 975 50  0001 C CNN
+	1    1225 975
+	1    0    0    -1
+$EndComp
+Wire Wire Line
+	1225 975  1225 1075
+$Comp
+L GND #PWR?
+U 1 1 59E74EEB
+P 1225 1375
+F 0 "#PWR?" H 1225 1125 50  0001 C CNN
+F 1 "GND" H 1225 1225 50  0000 C CNN
+F 2 "" H 1225 1375 50  0001 C CNN
+F 3 "" H 1225 1375 50  0001 C CNN
+	1    1225 1375
+	1    0    0    -1
+$EndComp
+Wire Wire Line
+	1225 1375 1225 1275
 $EndSCHEMATC

Commit message: Import the TMK footprint libraries
Parts:
- C1, C2, C3, C4, C5, C6, CR1, CR10, CR11, CR12, CR13, CR14, CR2, CR3, CR4, CR5, CR6, CR7, CR8, CR9: footprint (none) -> Capacitors_SMD:C_0805_HandSoldering
- F1: footprint (none) -> Fuse_Holders_and_Fuses:Fuse_SMD1206_HandSoldering
- R1, R2, R3, R4, R5: footprint (none) -> Resistors_SMD:R_0805_HandSoldering
- RGB1, RGB10, RGB11, RGB12, RGB13, RGB14, RGB2, RGB3, RGB4, RGB5, RGB6, RGB7, RGB8, RGB9: footprint (none) -> WS2812B:WS2812B
- U1: footprint (none) -> Housings_QFP:TQFP-32_7x7mm_Pitch0.8mm
- USB1: footprint (none) -> Molex-0548190589:Molex-0548190589
- Y1: footprint (none) -> Crystals:Crystal_SMD_3225-4pin_3.2x2.5mm_HandSoldering

Commit message: Finish linking lib parts to footprints
Parts:
- added SW1: SW_PUSH, Molex-0548190589:PushButton_6x6mm_TH, symbol SW_PUSH
- Q1: footprint TO_SOT_Packages_SMD:SOT-223 -> TO_SOT_Packages_SMD:SOT-223-3_TabPin2
Connections:
- net GND: now also SW1.1
- net at R1.2, U1.24 (PC1(~RESET~/dW)): now also SW1.2
Changed lines of the file:
@@
 F 0 "Q1" H 5575 2675 50  0000 L CNN
 F 1 "NSS40301MZ4T1G" H 5575 2600 50  0000 L CNN
-F 2 "TO_SOT_Packages_SMD:SOT-223" H 5575 2525 50  0001 L CIN
+F 2 "TO_SOT_Packages_SMD:SOT-223-3_TabPin2" H 5575 2525 50  0001 L CIN
 F 3 "" H 5375 2600 50  0001 L CNN
 	1    5375 2600
@@
 Wire Wire Line
 	1225 1375 1225 1275
+$Comp
+L SW_PUSH SW1
+U 1 1 59E77E37
+P 1575 1975
+F 0 "SW1" H 1725 2085 50  0000 C CNN
+F 1 "SW_PUSH" H 1575 1895 50  0000 C CNN
+F 2 "Molex-0548190589:PushButton_6x6mm_TH" H 1575 1975 60  0001 C CNN
+F 3 "" H 1575 1975 60  0000 C CNN
+	1    1575 1975
+	1    0    0    -1
+$EndComp
+Wire Wire Line
+	1875 1975 1925 1975
+Wire Wire Line
+	1925 1975 1925 2300
+Connection ~ 1925 2300
+$Comp
+L GND #PWR024
+U 1 1 59E7870E
+P 1175 1975
+F 0 "#PWR024" H 1175 1725 50  0001 C CNN
+F 1 "GND" V 1175 1775 50  0000 C CNN
+F 2 "" H 1175 1975 50  0001 C CNN
+F 3 "" H 1175 1975 50  0001 C CNN
+	1    1175 1975
+	0    1    1    0
+$EndComp
+Wire Wire Line
+	1175 1975 1275 1975
 $EndSCHEMATC
