File: Chronos.sch (KiCad schematic (older format))
At the start: 45 parts, among them Q1 NSS40301MZ4T1G, SW1 SW_PUSH, U1 ATMEGA32U2-AU, Y1 16MHz

Commit message: Place and breakout the controller
Connections:
- net GND: now also Q1.3 (E); no longer Q1.2 (C)
- net LEDGND: now also Q1.2 (C); no longer Q1.3 (E)
Changed lines of the file:
@@
 	0    1    1    0
 $EndComp
-Text GLabel 5475 2900 0    60   Input ~ 0
+Text GLabel 5475 2300 0    60   Input ~ 0
 LEDGND
 $Comp
 L GND #PWR012
 U 1 1 59E62F25
-P 5475 2300
-F 0 "#PWR012" H 5475 2050 50  0001 C CNN
-F 1 "GND" V 5475 2100 50  0000 C CNN
-F 2 "" H 5475 2300 50  0001 C CNN
-F 3 "" H 5475 2300 50  0001 C CNN
-	1    5475 2300
+P 5475 2900
+F 0 "#PWR012" H 5475 2650 50  0001 C CNN
+F 1 "GND" V 5475 2700 50  0000 C CNN
+F 2 "" H 5475 2900 50  0001 C CNN
+F 3 "" H 5475 2900 50  0001 C CNN
+	1    5475 2900
 	0    -1   -1   0
 $EndComp

Commit message: Change RGBLED pin
Connections:
- net RGBLED: now also U1.23 ((OC.1A/PCINT8)PC6)
Changed lines of the file:
@@
 Wire Wire Line
 	1175 1975 1275 1975
+Text GLabel 4250 4000 2    60   Input ~ 0
+RGBLED
 $EndSCHEMATC

Commit message: Wire some more LEDs
Connections:
- net D_P: now reaches R2.1, U1.29 (D+)
- net D_N: now reaches R3.1, U1.30 (D-)
Changed lines of the file:
@@
 Text GLabel 4250 4000 2    60   Input ~ 0
 RGBLED
+Text Label 1825 3400 0    60   ~ 0
+D_P
+Text Label 1825 3500 0    60   ~ 0
+D_N
 $EndSCHEMATC

Commit message: Correct pinout for secondary layouts
Connections:
- net COL1: now reaches U1.5 ((PCINT11/AIN2)PC2)
Changed lines of the file:
@@
 Text Label 1825 3500 0    60   ~ 0
 D_N
+Text GLabel 4250 3700 2    60   Input ~ 0
+COL1
 $EndSCHEMATC

Commit message: Connect probably all remaining diodes
Connections:
- net COL0: now reaches U1.6 ((OC.0B/INT0)PD0)
Changed lines of the file:
@@
 Text GLabel 4250 3700 2    60   Input ~ 0
 COL1
+Text GLabel 4250 2800 2    60   Input ~ 0
+COL0
 $EndSCHEMATC

Commit message: Work on connecting MCU to grid
Connections:
- net COL2: now reaches U1.7 ((AIN0/INT1)PD1)
Changed lines of the file:
@@
 Text GLabel 4250 2800 2    60   Input ~ 0
 COL0
+Text GLabel 4250 2900 2    60   Input ~ 0
+COL2
 $EndSCHEMATC

Commit message: Connect all cols
Connections:
- net COL7: now reaches U1.17 ((PD0/MISO/PCINT3)PB3)
- net COL6: now reaches U1.18 ((T1/PCINT4)PB4)
- net COL5: now reaches U1.19 ((PCINT5)PB5)
- net COL4: now reaches U1.20 ((PCINT6)PB6)
- net COL3: now reaches U1.22 ((INT4/ICP1/CLK0)PC7)
- net ROW8: now reaches U1.25 ((PCINT9/OC.1B)PC5)
- net ROW9: now reaches U1.26 ((PCINT10)PC4)
Changed lines of the file:
@@
 Text GLabel 4250 2900 2    60   Input ~ 0
 COL2
+Text GLabel 4250 3800 2    60   Input ~ 0
+ROW9
+Text GLabel 4250 3900 2    60   Input ~ 0
+ROW8
+Text GLabel 4250 4100 2    60   Input ~ 0
+COL3
+Text GLabel 4250 2500 2    60   Input ~ 0
+COL4
+Text GLabel 4250 2400 2    60   Input ~ 0
+COL5
+Text GLabel 4250 2300 2    60   Input ~ 0
+COL6
+Text GLabel 4250 2200 2    60   Input ~ 0
+COL7
 $EndSCHEMATC
