File: Chronos.sch (KiCad schematic (older format))
At the start: 45 parts, among them Q1 NSS40301MZ4T1G, SW1 SW_PUSH, U1 ATMEGA32U2-AU, Y1 16MHz

Commit message: Finalize netlist
Connections:
- net ROW5: now reaches U1.10 ((INT5/AIN3)PD4)
- net ROW4: now reaches U1.11 ((XCK/AIN4/PCINT12)PD5)
- net ROW3: now reaches U1.12 ((~RTS~/AIN5/INT6)PD6)
- net ROW2: now reaches U1.14 ((~SS~/PCINT0)PB0)
- net ROW1: now reaches U1.15 ((SCLK/PCINT1)PB1)
- net ROW0: now reaches U1.16 ((PDI/MOSI/PCINT2)PB2)
- net ROW7: now reaches U1.8 ((RXD1/AIN1/INT2)PD2)
- net ROW6: now reaches U1.9 ((TXD1/INT3)PD3)
Changed lines of the file:
@@
 Text GLabel 4250 2200 2    60   Input ~ 0
 COL7
+Text GLabel 4250 2100 2    60   Input ~ 0
+ROW0
+Text GLabel 4250 2000 2    60   Input ~ 0
+ROW1
+Text GLabel 4250 1900 2    60   Input ~ 0
+ROW2
+Text GLabel 4250 3400 2    60   Input ~ 0
+ROW3
+Text GLabel 4250 3300 2    60   Input ~ 0
+ROW4
+Text GLabel 4250 3200 2    60   Input ~ 0
+ROW5
+Text GLabel 4250 3100 2    60   Input ~ 0
+ROW6
+Text GLabel 4250 3000 2    60   Input ~ 0
+ROW7
 $EndSCHEMATC

Commit message: Warn users about KiCad being KiCad
Other:
- note added: "This is supposed to be a NPN transistor\nFor some reason KiCad keeps flipping the arrow the other way"
Changed lines of the file:
@@
 Text GLabel 4250 3000 2    60   Input ~ 0
 ROW7
+Text Notes 5575 2825 0    50   ~ 0
+This is supposed to be a NPN transistor\nFor some reason KiCad keeps flipping the arrow the other way
 $EndSCHEMATC
