File: Matrix.sch (KiCad schematic (older format))
At the start: 213 parts

Commit message: Rename all resistors
Parts:
- gave numbers to parts that had none: 65
- renumbered D_ISO'1 to D_ISO`1
Connections:
- net at K_F1.2 (ROW): no longer D_F1.2 (A)
- net at K_F1.4 (LEDGND): no longer R_F1.2
Other:
- moved on the sheet: K_F1

Commit message: Wire cols and 5V rails of LEDs
Connections:
- net COL0: now reaches K_ESC1.1 (COL)
- net COL0: now also K_#1.1 (COL), K_CAPS1.1 (COL), K_CTRL1.1 (COL), K_ISO\1.1 (COL), K_SHIFT1.1 (COL), K_TAB1.1 (COL), K_WIN1.1 (COL)
- net +5V: now reaches K_ESC1.3 (LED)
- net +5V: now also K_#0_1.3 (LED), K_#1.3 (LED), K_#2.3 (LED), K_#3.3 (LED), K_#4.3 (LED), K_#5.3 (LED), K_#6.3 (LED), K_#7.3 (LED), K_#8.3 (LED), K_#9.3 (LED), K_'1.3 (LED), K_,1.3 (LED), K_-1.3 (LED), K_.1.3 (LED), K_/1.3 (LED), K_/2.3 (LED), K_;1.3 (LED), K_=1.3 (LED), K_A1.3 (LED), K_ALT1.3 (LED), K_B1.3 (LED), K_BACK1.3 (LED), K_C1.3 (LED), K_CAPS1.3 (LED), K_CTRL1.3 (LED), K_D1.3 (LED), K_DEL1.3 (LED), K_DOWN1.3 (LED), K_E1.3 (LED), K_ENTER1.3 (LED), K_F1.3 (LED), K_FN1.3 (LED), K_G1.3 (LED), K_H1.3 (LED), K_I1.3 (LED), K_ISO\1.3 (LED), K_ISO`1.3 (LED), K_J1.3 (LED), K_K1.3 (LED), K_L1.3 (LED), K_LEFT1.3 (LED), K_M1.3 (LED), K_N1.3 (LED), K_O1.3 (LED), K_P1.3 (LED), K_Q1.3 (LED), K_R1.3 (LED), K_RIGHT1.3 (LED), K_RSHIFT1.3 (LED), K_S1.3 (LED), K_SHIFT1.3 (LED), K_SPACE1.3 (LED), K_T1.3 (LED), K_TAB1.3 (LED), K_U1.3 (LED), K_UP1.3 (LED), K_V1.3 (LED), K_W1.3 (LED), K_WIN1.3 (LED), K_X1.3 (LED), K_Y1.3 (LED), K_Z1.3 (LED), K_[1.3 (LED), K_\1.3 (LED), K_]1.3 (LED), K_`1.3 (LED)
- net COL1: now reaches K_#2.1 (COL)
- net COL1: now also K_#3.1 (COL), K_A1.1 (COL), K_ALT1.1 (COL), K_Q1.1 (COL), K_S1.1 (COL), K_W1.1 (COL), K_X1.1 (COL), K_Z1.1 (COL)
- net COL2: now reaches K_#4.1 (COL)
- net COL2: now also K_#5.1 (COL), K_C1.1 (COL), K_D1.1 (COL), K_E1.1 (COL), K_F1.1 (COL), K_R1.1 (COL), K_V1.1 (COL)
- net COL3: now reaches K_#6.1 (COL)
- net COL3: now also K_#7.1 (COL), K_B1.1 (COL), K_G1.1 (COL), K_H1.1 (COL), K_N1.1 (COL), K_SPACE1.2 (COL), K_T1.1 (COL), K_Y1.1 (COL)
- net COL4: now reaches K_#8.1 (COL)
- net COL4: now also K_#9.1 (COL), K_,1.1 (COL), K_I1.1 (COL), K_J1.1 (COL), K_K1.1 (COL), K_M1.1 (COL), K_U1.1 (COL)
- net COL5: now reaches K_#0_1.1 (COL)
- net COL5: now also K_-1.1 (COL), K_.1.1 (COL), K_/1.1 (COL), K_;1.1 (COL), K_FN1.1 (COL), K_L1.1 (COL), K_O1.1 (COL), K_P1.1 (COL), K_`1.1 (COL)
- net COL6: now reaches K_=1.1 (COL)
- net COL6: now also K_'1.1 (COL), K_/2.1 (COL), K_DEL1.1 (COL), K_DOWN1.1 (COL), K_ISO`1.1 (COL), K_LEFT1.1 (COL), K_UP1.1 (COL), K_[1.1 (COL), K_]1.1 (COL)
- net COL7: now reaches K_BACK1.1 (COL)
- net COL7: now also K_ENTER1.1 (COL), K_RIGHT1.1 (COL), K_RSHIFT1.1 (COL), K_\1.1 (COL)
- net at K_F1.2 (ROW): now also D_F1.2 (A)
- net at K_F1.4 (LEDGND): now also R_F1.2
Other:
- moved on the sheet: K_F1

Commit message: Wire LED GND
Connections:
- net +5V: no longer K_/2.3 (LED)
- net COL6: no longer K_/2.1 (COL)
- net GND: now reaches R_ESC1.1
- net GND: now also R_#0_1.1, R_#1.1, R_#2.1, R_#3.1, R_#4.1, R_#5.1, R_#6.1, R_#7.1, R_#8.1, R_#9.1, R_'1.1, R_,1.1, R_-1.1, R_.1.1, R_/1.1, R_;1.1, R_=1.1, R_A1.1, R_ALT1.1, R_B1.1, R_BACK1.1, R_C1.1, R_CAPS1.1, R_CTRL1.1, R_D1.1, R_DEL1.1, R_DOWN1.1, R_E1.1, R_ENTER1.1, R_F1.1, R_FN1.1, R_G1.1, R_H1.1, R_I1.1, R_ISO\1.1, R_ISO`1.1, R_J1.1, R_K1.1, R_L1.1, R_LEFT1.1, R_M1.1, R_N1.1, R_O1.1, R_P1.1, R_Q1.1, R_R1.1, R_RIGHT1.1, R_RSHIFT1.1, R_S1.1, R_SHIFT1.1, R_SPACE1.1, R_T1.1, R_TAB1.1, R_U1.1, R_UP1.1, R_V1.1, R_W1.1, R_WIN1.1, R_X1.1, R_Y1.1, R_Z1.1, R_[1.1, R_\1.1, R_]1.1, R_`1.1
Changed lines of the file:
@@
 Connection ~ 3025 2650
 Wire Wire Line
-	2975 2350 3475 2350
+	2975 2350 9325 2350
 Connection ~ 3475 2650
 Connection ~ 3025 2350
-Wire Wire Line
-	3875 2350 4375 2350
 Connection ~ 4375 2650
 Connection ~ 3925 2650
-$Comp
-L +5V #PWR?
-U 1 1 59F103C1
-P 3875 2350
-F 0 "#PWR?" H 3875 2200 50  0001 C CNN
-F 1 "+5V" H 3875 2490 50  0000 C CNN
-F 2 "" H 3875 2350 50  0001 C CNN
-F 3 "" H 3875 2350 50  0001 C CNN
-	1    3875 2350
-	0    -1   -1   0
-$EndComp
 Connection ~ 3925 2350
 Wire Wire Line
@@
 Connection ~ 4825 3550
 Wire Wire Line
-	4775 2350 5275 2350
-Wire Wire Line
 	5275 2350 5275 5350
 Wire Wire Line
 	5275 2650 5250 2650
 Connection ~ 4825 2650
-$Comp
-L +5V #PWR?
-U 1 1 59F19E21
-P 4775 2350
-F 0 "#PWR?" H 4775 2200 50  0001 C CNN
-F 1 "+5V" H 4775 2490 50  0000 C CNN
-F 2 "" H 4775 2350 50  0001 C CNN
-F 3 "" H 4775 2350 50  0001 C CNN
-	1    4775 2350
-	0    -1   -1   0
-$EndComp
 Connection ~ 4825 2350
 Wire Wire Line
@@
 	5725 2650 5700 2650
 Connection ~ 5725 3550
-Wire Wire Line
-	5675 2350 6175 2350
 Connection ~ 5725 2650
-$Comp
-L +5V #PWR?
-U 1 1 59F2CC36
-P 5675 2350
-F 0 "#PWR?" H 5675 2200 50  0001 C CNN
-F 1 "+5V" H 5675 2490 50  0000 C CNN
-F 2 "" H 5675 2350 50  0001 C CNN
-F 3 "" H 5675 2350 50  0001 C CNN
-	1    5675 2350
-	0    -1   -1   0
-$EndComp
 Connection ~ 5725 2350
 Wire Wire Line
@@
 Connection ~ 6625 3550
 Wire Wire Line
-	6575 2350 7075 2350
-Wire Wire Line
 	7075 2350 7075 5350
 Wire Wire Line
@@
 	7075 5350 7050 5350
 Connection ~ 7075 4450
-$Comp
-L +5V #PWR?
-U 1 1 59F42206
-P 6575 2350
-F 0 "#PWR?" H 6575 2200 50  0001 C CNN
-F 1 "+5V" H 6575 2490 50  0000 C CNN
-F 2 "" H 6575 2350 50  0001 C CNN
-F 3 "" H 6575 2350 50  0001 C CNN
-	1    6575 2350
-	0    -1   -1   0
-$EndComp
 Connection ~ 6625 2350
 Wire Wire Line
@@
 	7525 2350 7525 6250
 Wire Wire Line
-	7475 2350 7975 2350
-Wire Wire Line
 	7975 2350 7975 6250
 Wire Wire Line
 	7975 2650 7950 2650
-$Comp
-L +5V #PWR?
-U 1 1 59F45860
-P 7475 2350
-F 0 "#PWR?" H 7475 2200 50  0001 C CNN
-F 1 "+5V" H 7475 2490 50  0000 C CNN
-F 2 "" H 7475 2350 50  0001 C CNN
-F 3 "" H 7475 2350 50  0001 C CNN
-	1    7475 2350
-	0    -1   -1   0
-$EndComp
 Connection ~ 7525 2350
 Wire Wire Line
@@
 	8425 6250 8400 6250
 Wire Wire Line
-	8425 2350 8425 6250
-Wire Wire Line
-	8425 5350 8400 5350
-Wire Wire Line
 	8425 4450 8400 4450
-Connection ~ 8425 5350
 Wire Wire Line
 	8425 3550 8400 3550
@@
 Connection ~ 8425 3550
 Wire Wire Line
-	8375 2350 8875 2350
-Wire Wire Line
 	8875 2350 8875 6250
 Wire Wire Line
 	8875 2650 8850 2650
 Connection ~ 8425 2650
-$Comp
-L +5V #PWR?
-U 1 1 59F59D19
-P 8375 2350
-F 0 "#PWR?" H 8375 2200 50  0001 C CNN
-F 1 "+5V" H 8375 2490 50  0000 C CNN
-F 2 "" H 8375 2350 50  0001 C CNN
-F 3 "" H 8375 2350 50  0001 C CNN
-	1    8375 2350
-	0    -1   -1   0
-$EndComp
 Connection ~ 8425 2350
 Wire Wire Line
@@
 Connection ~ 9325 3550
 Connection ~ 9325 2650
-$Comp
-L +5V #PWR?
-U 1 1 59F6AF60
-P 9275 2350
-F 0 "#PWR?" H 9275 2200 50  0001 C CNN
-F 1 "+5V" H 9275 2490 50  0000 C CNN
-F 2 "" H 9275 2350 50  0001 C CNN
-F 3 "" H 9275 2350 50  0001 C CNN
-	1    9275 2350
-	0    -1   -1   0
-$EndComp
-Wire Wire Line
-	9325 2350 9275 2350
 Wire Wire Line
 	4850 2150 4850 5300
@@
 Connection ~ 8000 5300
 Connection ~ 7550 5300
-Wire Wire Line
-	8450 2150 8450 6200
-Connection ~ 8450 5300
 Connection ~ 8450 4400
 Connection ~ 8450 3500
@@
 Connection ~ 9350 4400
 Connection ~ 9350 5300
+Wire Wire Line
+	2625 2950 9275 2950
+Connection ~ 3425 2950
+Connection ~ 3875 2950
+Connection ~ 4325 2950
+Connection ~ 4775 2950
+Connection ~ 5225 2950
+Connection ~ 5675 2950
+Connection ~ 6125 2950
+Connection ~ 6575 2950
+Connection ~ 7025 2950
+Connection ~ 7475 2950
+Connection ~ 7925 2950
+Connection ~ 8375 2950
+Connection ~ 8825 2950
+Wire Wire Line
+	2625 3850 9275 3850
+Connection ~ 8825 3850
+Connection ~ 8375 3850
+Connection ~ 7925 3850
+Connection ~ 7475 3850
+Connection ~ 7025 3850
+Connection ~ 6575 3850
+Connection ~ 6125 3850
+Connection ~ 5675 3850
+Connection ~ 5225 3850
+Connection ~ 4775 3850
+Connection ~ 4325 3850
+Connection ~ 3875 3850
+Connection ~ 8875 2350
+Connection ~ 7975 2350
+Connection ~ 7075 2350
+Connection ~ 6175 2350
+Connection ~ 5275 2350
+Connection ~ 4375 2350
+Connection ~ 3475 2350
+Wire Wire Line
+	2625 2900 2625 6550
+Connection ~ 3425 3850
+Connection ~ 2975 2950
+Wire Wire Line
+	2625 4750 9275 4750
+Connection ~ 2625 3850
+Connection ~ 3425 4750
+Connection ~ 3875 4750
+Connection ~ 4325 4750
+Connection ~ 4775 4750
+Connection ~ 5225 4750
+Connection ~ 5675 4750
+Connection ~ 6125 4750
+Connection ~ 6575 4750
+Connection ~ 7025 4750
+Connection ~ 7475 4750
+Connection ~ 7925 4750
+Connection ~ 8375 4750
+Connection ~ 8825 4750
+$Comp
+L GND #PWR?
+U 1 1 59FE2F9C
+P 2625 2900
+F 0 "#PWR?" H 2625 2650 50  0001 C CNN
+F 1 "GND" H 2625 2750 50  0000 C CNN
+F 2 "" H 2625 2900 50  0001 C CNN
+F 3 "" H 2625 2900 50  0001 C CNN
+	1    2625 2900
+	-1   0    0    1
+$EndComp
+Connection ~ 2625 2950
+Wire Wire Line
+	2625 5650 9275 5650
+Connection ~ 2625 4750
+Connection ~ 2975 5650
+Connection ~ 3425 5650
+Connection ~ 3875 5650
+Connection ~ 4325 5650
+Connection ~ 4775 5650
+Connection ~ 5225 5650
+Connection ~ 5675 5650
+Connection ~ 6125 5650
+Connection ~ 6575 5650
+Connection ~ 7025 5650
+Connection ~ 7475 5650
+Connection ~ 7925 5650
+Connection ~ 8825 5650
+Wire Wire Line
+	8450 5700 8450 6200
+Wire Wire Line
+	8450 5700 8625 5700
+Wire Wire Line
+	8625 5700 8625 5000
+Wire Wire Line
+	8625 5000 8450 5000
+Wire Wire Line
+	8450 5000 8450 2150
+Wire Wire Line
+	8425 2350 8425 5025
+Wire Wire Line
+	8425 5025 8600 5025
+Wire Wire Line
+	8600 5025 8600 5675
+Wire Wire Line
+	8600 5675 8425 5675
+Wire Wire Line
+	8425 5675 8425 6250
+Wire Wire Line
+	2625 6550 9275 6550
+Connection ~ 8825 6550
+Connection ~ 8375 6550
+Connection ~ 7925 6550
+Connection ~ 7475 6550
+Connection ~ 5675 6550
+Connection ~ 3875 6550
+Connection ~ 3425 6550
+Connection ~ 2625 5650
+Connection ~ 2975 6550
 $EndSCHEMATC

Commit message: Wire the rows
Connections:
- net ROW0: now reaches D_ESC1.1 (K)
- net ROW0: now also D_#0_1.1 (K), D_#2.1 (K), D_#4.1 (K), D_#6.1 (K), D_#8.1 (K), D_=1.1 (K), D_BACK1.1 (K)
- net ROW1: now reaches D_#1.1 (K)
- net ROW1: now also D_#3.1 (K), D_#5.1 (K), D_#7.1 (K), D_#9.1 (K), D_-1.1 (K), D_DEL1.1 (K)
- net ROW3: now reaches D_TAB1.1 (K)
- net ROW3: now also D_I1.1 (K), D_P1.1 (K), D_R1.1 (K), D_W1.1 (K), D_Y1.1 (K), D_]1.1 (K)
- net ROW2: now reaches D_Q1.1 (K)
- net ROW2: now also D_E1.1 (K), D_O1.1 (K), D_T1.1 (K), D_U1.1 (K), D_[1.1 (K), D_\1.1 (K)
- net ROW5: now reaches D_CAPS1.1 (K)
- net ROW5: now also D_;1.1 (K), D_F1.1 (K), D_H1.1 (K), D_ISO`1.1 (K), D_K1.1 (K), D_S1.1 (K)
- net ROW4: now reaches D_A1.1 (K)
- net ROW4: now also D_'1.1 (K), D_D1.1 (K), D_ENTER1.1 (K), D_G1.1 (K), D_J1.1 (K), D_L1.1 (K)
- net ROW6: now reaches D_SHIFT1.1 (K)
- net ROW6: now also D_.1.1 (K), D_B1.1 (K), D_C1.1 (K), D_M1.1 (K), D_RSHIFT1.1 (K), D_Z1.1 (K)
- net ROW7: now reaches D_ISO\1.1 (K)
- net ROW7: now also D_,1.1 (K), D_/1.1 (K), D_N1.1 (K), D_UP1.1 (K), D_V1.1 (K), D_X1.1 (K)
- net ROW8: now reaches D_CTRL1.1 (K)
- net ROW8: now also D_ALT1.1 (K), D_FN1.1 (K), D_LEFT1.1 (K), D_RIGHT1.1 (K), D_SPACE1.1 (K)
- net ROW9: now reaches D_WIN1.1 (K)
- net ROW9: now also D_DOWN1.1 (K), D_`1.1 (K)

Commit message: Begin footprint associations with lib parts
Parts:
- renumbered K_ISOENTER to K_ISOENTER1
Changed lines of the file:
@@
 $EndComp
 $Comp
-L MX-ISO K_ISOENTER
+L MX-ISO K_ISOENTER1
 U 1 1 59EB378F
 P 9625 4425
-F 0 "K_ISOENTER" H 9775 4550 60  0000 C CNN
+F 0 "K_ISOENTER1" H 9775 4550 60  0000 C CNN
 F 1 "MX-ISO" H 9625 4475 20  0000 C CNN
 F 2 "" H 9600 4400 60  0001 C CNN
@@
 $EndComp
 $Comp
-L +5V #PWR?
+L +5V #PWR022
 U 1 1 59F09083
 P 2975 2350
-F 0 "#PWR?" H 2975 2200 50  0001 C CNN
+F 0 "#PWR022" H 2975 2200 50  0001 C CNN
 F 1 "+5V" H 2975 2490 50  0000 C CNN
 F 2 "" H 2975 2350 50  0001 C CNN
@@
 COL7
 $Comp
-L GND #PWR?
+L GND #PWR023
 U 1 1 59FE2F9C
 P 2625 2900
-F 0 "#PWR?" H 2625 2650 50  0001 C CNN
+F 0 "#PWR023" H 2625 2650 50  0001 C CNN
 F 1 "GND" H 2625 2750 50  0000 C CNN
 F 2 "" H 2625 2900 50  0001 C CNN

Commit message: Import the TMK footprint libraries
Parts:
- D_#0_1, D_#1, D_#2, D_#3, D_#4, D_#5, D_#6, D_#7, D_#8, D_#9, D_'1, D_,1, D_-1, D_.1, D_/1, D_;1, D_=1, D_A1, D_ALT1, D_B1, D_BACK1, D_C1, D_CAPS1, D_CTRL1, D_D1, D_DEL1, D_DOWN1, D_E1, D_ENTER1, D_ESC1, D_F1, D_FN1, D_G1, D_H1, D_I1, D_ISO\1, D_ISO`1, D_J1, D_K1, D_L1, D_LEFT1, D_M1, D_N1, D_O1, D_P1, D_Q1, D_R1, D_RIGHT1, D_RSHIFT1, D_S1, D_SHIFT1, D_SPACE1, D_T1, D_TAB1, D_U1, D_UP1, D_V1, D_W1, D_WIN1, D_X1, D_Y1, D_Z1, D_[1, D_\1, D_]1, D_`1: footprint (none) -> Diodes_THT:D_DO-35_SOD27_P7.62mm_Horizontal
- K_#0_1, K_#1, K_#2, K_#3, K_#4, K_#5, K_#6, K_#7, K_#8, K_#9, K_'1, K_,1, K_-1, K_.1, K_/2, K_;1, K_=1, K_A1, K_B1, K_BACK1, K_C1, K_D1, K_DEL1, K_DOWN1, K_E1, K_ESC1, K_F1, K_FN1, K_G1, K_H1, K_I1, K_ISO\1, K_ISO`1, K_J1, K_K1, K_L1, K_LEFT1, K_M1, K_N1, K_O1, K_P1, K_Q1, K_R1, K_RIGHT1, K_RSHIFT1, K_S1, K_T1, K_U1, K_UP1, K_V1, K_W1, K_X1, K_Y1, K_Z1, K_[1, K_]1, K_`1: footprint (none) -> MX_Alps_Hybrid:MX-1U
- R_#0_1, R_#1, R_#2, R_#3, R_#4, R_#5, R_#6, R_#7, R_#8, R_#9, R_'1, R_,1, R_-1, R_.1, R_/1, R_;1, R_=1, R_A1, R_ALT1, R_B1, R_BACK1, R_C1, R_CAPS1, R_CTRL1, R_D1, R_DEL1, R_DOWN1, R_E1, R_ENTER1, R_ESC1, R_F1, R_FN1, R_G1, R_H1, R_I1, R_ISO\1, R_ISO`1, R_J1, R_K1, R_L1, R_LEFT1, R_M1, R_N1, R_O1, R_P1, R_Q1, R_R1, R_RIGHT1, R_RSHIFT1, R_S1, R_SHIFT1, R_SPACE1, R_T1, R_TAB1, R_U1, R_UP1, R_V1, R_W1, R_WIN1, R_X1, R_Y1, R_Z1, R_[1, R_\1, R_]1, R_`1: footprint (none) -> Resistors_SMD:R_1206_HandSoldering

Commit message: Finalize schematic without wiring non-main keys
Parts:
- K_/1, K_CAPS1: footprint (none) -> MX_Alps_Hybrid:MX-1.75U
- K_ALT1, K_ALT2, K_CTRL1, K_FN2, K_MENU1, K_RALT1, K_RCTRL1, K_RWIN1, K_WIN1: footprint (none) -> MX_Alps_Hybrid:MX-1.25U
- K_BACK2: footprint (none) -> MX_Alps_Hybrid:MX-2U
- K_CMD1, K_CTRL2, K_RCMD1, K_RCTRL2, K_TAB1, K_\1: footprint (none) -> MX_Alps_Hybrid:MX-1.5U
- K_ENTER1, K_SHIFT1: footprint (none) -> MX_Alps_Hybrid:MX-2.25U
- K_ISOENTER1: footprint (none) -> MX_Alps_Hybrid:MX-ISO-Combined
- K_RSHIFT2: footprint (none) -> MX_Alps_Hybrid:MX-2.75U
- K_SPACE1: footprint (none) -> MX_Alps_Hybrid:MX-6.25U-ReversedStabilizers
- K_SPACE2: footprint (none) -> MX_Alps_Hybrid:MX-6.5U
Changed lines of the file:
@@
 F 0 "K_TAB1" H 3325 3650 60  0000 C CNN
 F 1 "MX-1.5U" H 3325 3575 20  0000 C CNN
-F 2 "" H 3300 3500 60  0001 C CNN
+F 2 "MX_Alps_Hybrid:MX-1.5U" H 3300 3500 60  0001 C CNN
 F 3 "" H 3300 3500 60  0001 C CNN
 	1    3325 3525
@@
 F 0 "K_\\1" H 9175 3650 60  0000 C CNN
 F 1 "MX-1.5U" H 9175 3575 20  0000 C CNN
-F 2 "" H 9150 3500 60  0001 C CNN
+F 2 "MX_Alps_Hybrid:MX-1.5U" H 9150 3500 60  0001 C CNN
 F 3 "" H 9150 3500 60  0001 C CNN
 	1    9175 3525
@@
 F 0 "K_CAPS1" H 3325 4550 60  0000 C CNN
 F 1 "MX-1.75U" H 3325 4475 20  0000 C CNN
-F 2 "" H 3300 4400 60  0001 C CNN
+F 2 "MX_Alps_Hybrid:MX-1.75U" H 3300 4400 60  0001 C CNN
 F 3 "" H 3300 4400 60  0001 C CNN
 	1    3325 4425
@@
 F 0 "K_ENTER1" H 9175 4550 60  0000 C CNN
 F 1 "MX-2.25U" H 9175 4475 20  0000 C CNN
-F 2 "" H 9150 4400 60  0001 C CNN
+F 2 "MX_Alps_Hybrid:MX-2.25U" H 9150 4400 60  0001 C CNN
 F 3 "" H 9150 4400 60  0001 C CNN
 	1    9175 4425
@@
 F 0 "K_SHIFT1" H 2875 5450 60  0000 C CNN
 F 1 "MX-2.25U" H 2875 5375 20  0000 C CNN
-F 2 "" H 2850 5300 60  0001 C CNN
+F 2 "MX_Alps_Hybrid:MX-2.25U" H 2850 5300 60  0001 C CNN
 F 3 "" H 2850 5300 60  0001 C CNN
 	1    2875 5325
@@
 F 0 "K_/1" H 7825 5450 60  0000 C CNN
 F 1 "MX-1.75U" H 7825 5375 20  0000 C CNN
-F 2 "" H 7800 5300 60  0001 C CNN
+F 2 "MX_Alps_Hybrid:MX-1.75U" H 7800 5300 60  0001 C CNN
 F 3 "" H 7800 5300 60  0001 C CNN
 	1    7825 5325
@@
 F 0 "K_CTRL1" H 2875 6350 60  0000 C CNN
 F 1 "MX-1.25U" H 2875 6275 20  0000 C CNN
-F 2 "" H 2850 6200 60  0001 C CNN
+F 2 "MX_Alps_Hybrid:MX-1.25U" H 2850 6200 60  0001 C CNN
 F 3 "" H 2850 6200 60  0001 C CNN
 	1    2875 6225
@@
 F 0 "K_WIN1" H 3325 6350 60  0000 C CNN
 F 1 "MX-1.25U" H 3325 6275 20  0000 C CNN
-F 2 "" H 3300 6200 60  0001 C CNN
+F 2 "MX_Alps_Hybrid:MX-1.25U" H 3300 6200 60  0001 C CNN
 F 3 "" H 3300 6200 60  0001 C CNN
 	1    3325 6225
@@
 F 0 "K_ALT1" H 3775 6350 60  0000 C CNN
 F 1 "MX-1.25U" H 3775 6275 20  0000 C CNN
-F 2 "" H 3750 6200 60  0001 C CNN
+F 2 "MX_Alps_Hybrid:MX-1.25U" H 3750 6200 60  0001 C CNN
 F 3 "" H 3750 6200 60  0001 C CNN
 	1    3775 6225
@@
 F 0 "K_SPACE1" H 5575 6350 60  0000 C CNN
 F 1 "MX-6.25U-FLIPPED" H 5575 6275 20  0000 C CNN
-F 2 "" H 5550 6200 60  0001 C CNN
+F 2 "MX_Alps_Hybrid:MX-6.25U-ReversedStabilizers" H 5550 6200 60  0001 C CNN
 F 3 "" H 5550 6200 60  0001 C CNN
 	1    5575 6225
@@
 F 0 "K_ISOENTER1" H 9775 4550 60  0000 C CNN
 F 1 "MX-ISO" H 9625 4475 20  0000 C CNN
-F 2 "" H 9600 4400 60  0001 C CNN
+F 2 "MX_Alps_Hybrid:MX-ISO-Combined" H 9600 4400 60  0001 C CNN
 F 3 "" H 9600 4400 60  0001 C CNN
 	1    9625 4425
@@
 F 0 "K_BACK2" H 9700 2750 60  0000 C CNN
 F 1 "MX-2U" H 9625 2675 20  0000 C CNN
-F 2 "" H 9600 2600 60  0001 C CNN
+F 2 "MX_Alps_Hybrid:MX-2U" H 9600 2600 60  0001 C CNN
 F 3 "" H 9600 2600 60  0001 C CNN
 	1    9625 2625
@@
 F 0 "K_RSHIFT2" H 9725 5450 60  0000 C CNN
 F 1 "MX-2.75U" H 9625 5375 20  0000 C CNN
-F 2 "" H 9600 5300 60  0001 C CNN
+F 2 "MX_Alps_Hybrid:MX-2.75U" H 9600 5300 60  0001 C CNN
 F 3 "" H 9600 5300 60  0001 C CNN
 	1    9625 5325
@@
 F 0 "K_FN2" H 7375 7250 60  0000 C CNN
 F 1 "MX-1.25U" H 7375 7175 20  0000 C CNN
-F 2 "" H 7350 7100 60  0001 C CNN
+F 2 "MX_Alps_Hybrid:MX-1.25U" H 7350 7100 60  0001 C CNN
 F 3 "" H 7350 7100 60  0001 C CNN
 	1    7375 7125
@@
 F 0 "K_RWIN1" H 7825 7250 60  0000 C CNN
 F 1 "MX-1.25U" H 7825 7175 20  0000 C CNN
-F 2 "" H 7800 7100 60  0001 C CNN
+F 2 "MX_Alps_Hybrid:MX-1.25U" H 7800 7100 60  0001 C CNN
 F 3 "" H 7800 7100 60  0001 C CNN
 	1    7825 7125
@@
 F 0 "K_RCTRL1" H 9175 7250 60  0000 C CNN
 F 1 "MX-1.25U" H 9175 7175 20  0000 C CNN
-F 2 "" H 9150 7100 60  0001 C CNN
+F 2 "MX_Alps_Hybrid:MX-1.25U" H 9150 7100 60  0001 C CNN
 F 3 "" H 9150 7100 60  0001 C CNN
 	1    9175 7125
@@
 F 0 "K_MENU1" H 8725 7250 60  0000 C CNN
 F 1 "MX-1.25U" H 8725 7175 20  0000 C CNN
-F 2 "" H 8700 7100 60  0001 C CNN
+F 2 "MX_Alps_Hybrid:MX-1.25U" H 8700 7100 60  0001 C CNN
 F 3 "" H 8700 7100 60  0001 C CNN
 	1    8725 7125
@@
 F 0 "K_CTRL2" H 2875 7250 60  0000 C CNN
 F 1 "MX-1.5U" H 2875 7175 20  0000 C CNN
-F 2 "" H 2850 7100 60  0001 C CNN
+F 2 "MX_Alps_Hybrid:MX-1.5U" H 2850 7100 60  0001 C CNN
 F 3 "" H 2850 7100 60  0001 C CNN
 	1    2875 7125
@@
 F 0 "K_ALT2" H 3325 7250 60  0000 C CNN
 F 1 "MX-1.25U" H 3325 7175 20  0000 C CNN
-F 2 "" H 3300 7100 60  0001 C CNN
+F 2 "MX_Alps_Hybrid:MX-1.25U" H 3300 7100 60  0001 C CNN
 F 3 "" H 3300 7100 60  0001 C CNN
 	1    3325 7125
@@
 F 0 "K_CMD1" H 3775 7250 60  0000 C CNN
 F 1 "MX-1.5U" H 3775 7175 20  0000 C CNN
-F 2 "" H 3750 7100 60  0001 C CNN
+F 2 "MX_Alps_Hybrid:MX-1.5U" H 3750 7100 60  0001 C CNN
 F 3 "" H 3750 7100 60  0001 C CNN
 	1    3775 7125
@@
 F 0 "K_SPACE2" H 5575 7250 60  0000 C CNN
 F 1 "MX-6.5U" H 5575 7175 20  0000 C CNN
-F 2 "" H 5550 7100 60  0001 C CNN
+F 2 "MX_Alps_Hybrid:MX-6.5U" H 5550 7100 60  0001 C CNN
 F 3 "" H 5550 7100 60  0001 C CNN
 	1    5575 7125
@@
 F 0 "K_RCMD1" H 7825 7850 60  0000 C CNN
 F 1 "MX-1.5U" H 7825 7775 20  0000 C CNN
-F 2 "" H 7800 7700 60  0001 C CNN
+F 2 "MX_Alps_Hybrid:MX-1.5U" H 7800 7700 60  0001 C CNN
 F 3 "" H 7800 7700 60  0001 C CNN
 	1    7825 7725
@@
 F 0 "K_RCTRL2" H 9175 7850 60  0000 C CNN
 F 1 "MX-1.5U" H 9175 7775 20  0000 C CNN
-F 2 "" H 9150 7700 60  0001 C CNN
+F 2 "MX_Alps_Hybrid:MX-1.5U" H 9150 7700 60  0001 C CNN
 F 3 "" H 9150 7700 60  0001 C CNN
 	1    9175 7725
@@
 F 0 "K_RALT1" H 8275 7850 60  0000 C CNN
 F 1 "MX-1.25U" H 8275 7775 20  0000 C CNN
-F 2 "" H 8250 7700 60  0001 C CNN
+F 2 "MX_Alps_Hybrid:MX-1.25U" H 8250 7700 60  0001 C CNN
 F 3 "" H 8250 7700 60  0001 C CNN
 	1    8275 7725
@@
 $EndComp
 $Comp
-L +5V #PWR024
+L +5V #PWR025
 U 1 1 59F09083
 P 2975 2350
-F 0 "#PWR024" H 2975 2200 50  0001 C CNN
+F 0 "#PWR025" H 2975 2200 50  0001 C CNN
 F 1 "+5V" H 2975 2490 50  0000 C CNN
 F 2 "" H 2975 2350 50  0001 C CNN
@@
 COL7
 $Comp
-L GND #PWR025
+L GND #PWR026
 U 1 1 59FE2F9C
 P 2625 2900
-F 0 "#PWR025" H 2625 2650 50  0001 C CNN
+F 0 "#PWR026" H 2625 2650 50  0001 C CNN
 F 1 "GND" H 2625 2750 50  0000 C CNN
 F 2 "" H 2625 2900 50  0001 C CNN

Commit message: Add missing 1.25U shift
Parts:
- added K_SHIFT2: MX-1.25U, MX_Alps_Hybrid:MX-1.25U, symbol MX-1.25U
Changed lines of the file:
@@
 LIBS:Molex-0548190589
 LIBS:ws2812b
-LIBS:keyboard_parts
-LIBS:mkl27z256vfm4
 LIBS:Chronos-cache
 EELAYER 25 0
@@
 	9150 6875 9150 6800
 Connection ~ 8250 6875
+$Comp
+L MX-1.25U K_SHIFT2
+U 1 1 59E8A45D
+P 2375 5325
+F 0 "K_SHIFT2" H 2375 5450 60  0000 C CNN
+F 1 "MX-1.25U" H 2375 5375 20  0000 C CNN
+F 2 "MX_Alps_Hybrid:MX-1.25U" H 2350 5300 60  0001 C CNN
+F 3 "" H 2350 5300 60  0001 C CNN
+	1    2375 5325
+	1    0    0    -1
+$EndComp
 $EndSCHEMATC
