File: Matrix.sch (KiCad schematic (older format))
At the start: 214 parts

Commit message: Replace some switch footprints with alps only for compatibility
Parts:
- K_RALT1: footprint MX_Alps_Hybrid:MX-1.25U -> MX_Alps_Hybrid:ALPS-1.25U
- K_RCMD1, K_RCTRL2: footprint MX_Alps_Hybrid:MX-1.5U -> MX_Alps_Hybrid:ALPS-1.5U
Changed lines of the file:
@@
 F 0 "K_RCMD1" H 7825 7850 60  0000 C CNN
 F 1 "MX-1.5U" H 7825 7775 20  0000 C CNN
-F 2 "MX_Alps_Hybrid:MX-1.5U" H 7800 7700 60  0001 C CNN
+F 2 "MX_Alps_Hybrid:ALPS-1.5U" H 7800 7700 60  0001 C CNN
 F 3 "" H 7800 7700 60  0001 C CNN
 	1    7825 7725
@@
 F 0 "K_RCTRL2" H 9175 7850 60  0000 C CNN
 F 1 "MX-1.5U" H 9175 7775 20  0000 C CNN
-F 2 "MX_Alps_Hybrid:MX-1.5U" H 9150 7700 60  0001 C CNN
+F 2 "MX_Alps_Hybrid:ALPS-1.5U" H 9150 7700 60  0001 C CNN
 F 3 "" H 9150 7700 60  0001 C CNN
 	1    9175 7725
@@
 F 0 "K_RALT1" H 8275 7850 60  0000 C CNN
 F 1 "MX-1.25U" H 8275 7775 20  0000 C CNN
-F 2 "MX_Alps_Hybrid:MX-1.25U" H 8250 7700 60  0001 C CNN
+F 2 "MX_Alps_Hybrid:ALPS-1.25U" H 8250 7700 60  0001 C CNN
 F 3 "" H 8250 7700 60  0001 C CNN
 	1    8275 7725

Commit message: Remove default bottom row
If you want it, use the GH60 >.>
Also re-added MX compatibility to AEK row
Parts:
- removed K_FN2, K_MENU1, K_RCTRL1, K_RWIN1: MX-1.25U, MX_Alps_Hybrid:MX-1.25U, symbol MX-1.25U
- K_RALT1: footprint MX_Alps_Hybrid:ALPS-1.25U -> MX_Alps_Hybrid:MX-1.25U
- K_RCMD1, K_RCTRL2: footprint MX_Alps_Hybrid:ALPS-1.5U -> MX_Alps_Hybrid:MX-1.5U
Other:
- moved on the sheet: K_RALT1, K_RCMD1, K_RCTRL2
Changed lines of the file:
@@
-$EndComp
-$Comp
-L MX-1.25U K_FN2
-U 1 1 59EEC2D4
-P 7375 7125
-F 0 "K_FN2" H 7375 7250 60  0000 C CNN
-F 1 "MX-1.25U" H 7375 7175 20  0000 C CNN
-F 2 "MX_Alps_Hybrid:MX-1.25U" H 7350 7100 60  0001 C CNN
-F 3 "" H 7350 7100 60  0001 C CNN
-	1    7375 7125
-	1    0    0    -1
-$EndComp
-$Comp
-L MX-1.25U K_RWIN1
-U 1 1 59EEC2E8
-P 7825 7125
-F 0 "K_RWIN1" H 7825 7250 60  0000 C CNN
-F 1 "MX-1.25U" H 7825 7175 20  0000 C CNN
-F 2 "MX_Alps_Hybrid:MX-1.25U" H 7800 7100 60  0001 C CNN
-F 3 "" H 7800 7100 60  0001 C CNN
-	1    7825 7125
-	1    0    0    -1
-$EndComp
-$Comp
-L MX-1.25U K_RCTRL1
-U 1 1 59EEC324
-P 9175 7125
-F 0 "K_RCTRL1" H 9175 7250 60  0000 C CNN
-F 1 "MX-1.25U" H 9175 7175 20  0000 C CNN
-F 2 "MX_Alps_Hybrid:MX-1.25U" H 9150 7100 60  0001 C CNN
-F 3 "" H 9150 7100 60  0001 C CNN
-	1    9175 7125
-	1    0    0    -1
-$EndComp
-$Comp
-L MX-1.25U K_MENU1
-U 1 1 59EEC310
-P 8725 7125
-F 0 "K_MENU1" H 8725 7250 60  0000 C CNN
-F 1 "MX-1.25U" H 8725 7175 20  0000 C CNN
-F 2 "MX_Alps_Hybrid:MX-1.25U" H 8700 7100 60  0001 C CNN
-F 3 "" H 8700 7100 60  0001 C CNN
-	1    8725 7125
-	1    0    0    -1
 $EndComp
 $Comp
@@
 L MX-1.5U K_RCMD1
 U 1 1 59F16AD5
-P 7825 7725
-F 0 "K_RCMD1" H 7825 7850 60  0000 C CNN
-F 1 "MX-1.5U" H 7825 7775 20  0000 C CNN
-F 2 "MX_Alps_Hybrid:ALPS-1.5U" H 7800 7700 60  0001 C CNN
-F 3 "" H 7800 7700 60  0001 C CNN
-	1    7825 7725
+P 7825 7125
+F 0 "K_RCMD1" H 7825 7250 60  0000 C CNN
+F 1 "MX-1.5U" H 7825 7175 20  0000 C CNN
+F 2 "MX_Alps_Hybrid:MX-1.5U" H 7800 7100 60  0001 C CNN
+F 3 "" H 7800 7100 60  0001 C CNN
+	1    7825 7125
 	1    0    0    -1
 $EndComp
@@
 L MX-1.5U K_RCTRL2
 U 1 1 59F16AE1
-P 9175 7725
-F 0 "K_RCTRL2" H 9175 7850 60  0000 C CNN
-F 1 "MX-1.5U" H 9175 7775 20  0000 C CNN
-F 2 "MX_Alps_Hybrid:ALPS-1.5U" H 9150 7700 60  0001 C CNN
-F 3 "" H 9150 7700 60  0001 C CNN
-	1    9175 7725
+P 9175 7125
+F 0 "K_RCTRL2" H 9175 7250 60  0000 C CNN
+F 1 "MX-1.5U" H 9175 7175 20  0000 C CNN
+F 2 "MX_Alps_Hybrid:MX-1.5U" H 9150 7100 60  0001 C CNN
+F 3 "" H 9150 7100 60  0001 C CNN
+	1    9175 7125
 	1    0    0    -1
 $EndComp
@@
 L MX-1.25U K_RALT1
 U 1 1 59F1A49B
-P 8275 7725
-F 0 "K_RALT1" H 8275 7850 60  0000 C CNN
-F 1 "MX-1.25U" H 8275 7775 20  0000 C CNN
-F 2 "MX_Alps_Hybrid:ALPS-1.25U" H 8250 7700 60  0001 C CNN
-F 3 "" H 8250 7700 60  0001 C CNN
-	1    8275 7725
+P 8275 7125
+F 0 "K_RALT1" H 8275 7250 60  0000 C CNN
+F 1 "MX-1.25U" H 8275 7175 20  0000 C CNN
+F 2 "MX_Alps_Hybrid:MX-1.25U" H 8250 7100 60  0001 C CNN
+F 3 "" H 8250 7100 60  0001 C CNN
+	1    8275 7125
 	1    0    0    -1
 $EndComp

Commit message: Replace all the 1N4148 diodes with SMA diodes
Surface mount size easy enough for most DIYers
Parts:
- D_#0_1, D_#1, D_#2, D_#3, D_#4, D_#5, D_#6, D_#7, D_#8, D_#9, D_'1, D_,1, D_-1, D_.1, D_/1, D_;1, D_=1, D_A1, D_ALT1, D_B1, D_BACK1, D_C1, D_CAPS1, D_CTRL1, D_D1, D_DEL1, D_DOWN1, D_E1, D_ENTER1, D_ESC1, D_F1, D_FN1, D_G1, D_H1, D_I1, D_ISO\1, D_ISO`1, D_J1, D_K1, D_L1, D_LEFT1, D_M1, D_N1, D_O1, D_P1, D_Q1, D_R1, D_RIGHT1, D_RSHIFT1, D_S1, D_SHIFT1, D_SPACE1, D_T1, D_TAB1, D_U1, D_UP1, D_V1, D_W1, D_WIN1, D_X1, D_Y1, D_Z1, D_[1, D_\1, D_]1, D_`1: value 1N4148 -> SMA-GENERIC; footprint Diodes_THT:D_DO-35_SOD27_P7.62mm_Horizontal -> Diodes_SMD:D_SMA_Handsoldering

Commit message: Reverse ISO stabilizer holes to fix major collision
Parts:
- K_ISOENTER1: footprint MX_Alps_Hybrid:MX-ISO-Combined -> MX_Alps_Hybrid:MX-ISO-Combined-ReversedStabilizers
Changed lines of the file:
@@
 F 0 "K_ISOENTER1" H 9775 4550 60  0000 C CNN
 F 1 "MX-ISO" H 9625 4475 20  0000 C CNN
-F 2 "MX_Alps_Hybrid:MX-ISO-Combined" H 9600 4400 60  0001 C CNN
+F 2 "MX_Alps_Hybrid:MX-ISO-Combined-ReversedStabilizers" H 9600 4400 60  0001 C CNN
 F 3 "" H 9600 4400 60  0001 C CNN
 	1    9625 4425

Commit message: Replace SMA handsoldering with regular
handsolder footprints were way too big
Parts:
- D_#0_1, D_#1, D_#2, D_#3, D_#4, D_#5, D_#6, D_#7, D_#8, D_#9, D_'1, D_,1, D_-1, D_.1, D_/1, D_;1, D_=1, D_A1, D_ALT1, D_B1, D_BACK1, D_C1, D_CAPS1, D_CTRL1, D_D1, D_DEL1, D_DOWN1, D_E1, D_ENTER1, D_ESC1, D_F1, D_FN1, D_G1, D_H1, D_I1, D_ISO\1, D_ISO`1, D_J1, D_K1, D_L1, D_LEFT1, D_M1, D_N1, D_O1, D_P1, D_Q1, D_R1, D_RIGHT1, D_RSHIFT1, D_S1, D_SHIFT1, D_SPACE1, D_T1, D_TAB1, D_U1, D_UP1, D_V1, D_W1, D_WIN1, D_X1, D_Y1, D_Z1, D_[1, D_\1, D_]1, D_`1: footprint Diodes_SMD:D_SMA_Handsoldering -> Diodes_SMD:D_SMA

Commit message: Even more diodes
Parts:
- added K_CAPS2: MX-1.25U, MX_Alps_Hybrid:MX-1.25U, symbol MX-1.25U
Changed lines of the file:
@@
+	1    0    0    -1
+$EndComp
+$Comp
+L MX-1.25U K_CAPS2
+U 1 1 59E9604B
+P 2800 4425
+F 0 "K_CAPS2" H 2800 4550 60  0000 C CNN
+F 1 "MX-1.25U" H 2800 4475 20  0000 C CNN
+F 2 "MX_Alps_Hybrid:MX-1.25U" H 2775 4400 60  0001 C CNN
+F 3 "" H 2775 4400 60  0001 C CNN
+	1    2800 4425
 	1    0    0    -1
 $EndComp

Commit message: Remove K_RCMD1
Overlapped perfectly with K_`1
No need
Parts:
- removed K_RCMD1: MX-1.5U, MX_Alps_Hybrid:MX-1.5U, symbol MX-1.5U
Changed lines of the file:
@@
-$EndComp
-$Comp
-L MX-1.5U K_RCMD1
-U 1 1 59F16AD5
-P 7825 7125
-F 0 "K_RCMD1" H 7825 7250 60  0000 C CNN
-F 1 "MX-1.5U" H 7825 7175 20  0000 C CNN
-F 2 "MX_Alps_Hybrid:MX-1.5U" H 7800 7100 60  0001 C CNN
-F 3 "" H 7800 7100 60  0001 C CNN
-	1    7825 7125
-	1    0    0    -1
 $EndComp
 $Comp

Commit message: Fix LED resistor pinout
Connections:
- net GND renamed LEDGND
Changed lines of the file:
@@
 Text GLabel 9300 2150 0    60   Input ~ 0
 COL7
-$Comp
-L GND #PWR026
-U 1 1 59FE2F9C
-P 2625 2900
-F 0 "#PWR026" H 2625 2650 50  0001 C CNN
-F 1 "GND" H 2625 2750 50  0000 C CNN
-F 2 "" H 2625 2900 50  0001 C CNN
-F 3 "" H 2625 2900 50  0001 C CNN
-	1    2625 2900
-	-1   0    0    1
-$EndComp
 Text GLabel 2525 3275 0    60   Input ~ 0
 ROW0
@@
 	1    0    0    -1
 $EndComp
+Text GLabel 2625 2900 1    60   Input ~ 0
+LEDGND
 $EndSCHEMATC
