File: Matrix.sch (KiCad schematic (older format))
At the start: 210 parts

Commit message: Wire some more LEDs
Parts:
- K_ALT2, K_CAPS2: footprint MX_Alps_Hybrid:MX-1.25U -> MX_Alps_Hybrid:MX-1.25U-FLIPPED; symbol MX-1.25U -> MX-1.25U-FLIPPED
- K_CTRL2: footprint MX_Alps_Hybrid:MX-1.5U -> MX_Alps_Hybrid:MX-1.5U-FLIPPED; symbol MX-1.5U -> MX-1.5U-FLIPPED
- R_#0_1, R_#1, R_#2, R_#3, R_#4, R_#5, R_#6, R_#7, R_#8, R_#9, R_'1, R_,1, R_-1, R_.1, R_/1, R_;1, R_=1, R_A1, R_ALT1, R_B1, R_BACK1, R_C1, R_CAPS1, R_CTRL1, R_D1, R_DEL1, R_DOWN1, R_E1, R_ENTER1, R_ESC1, R_F1, R_FN1, R_G1, R_H1, R_I1, R_ISO\1, R_ISO`1, R_J1, R_K1, R_L1, R_LEFT1, R_M1, R_N1, R_O1, R_P1, R_Q1, R_R1, R_RIGHT1, R_RSHIFT1, R_S1, R_SHIFT1, R_SPACE1, R_T1, R_TAB1, R_U1, R_UP1, R_V1, R_W1, R_WIN1, R_X1, R_Y1, R_Z1, R_[1, R_\1, R_]1, R_`1: footprint Resistors_SMD:R_1206_HandSoldering -> Resistors_SMD:R_0805_HandSoldering
Connections:
- net +5V: now also K_ALT2.3 (LED), K_BACK2.3 (LED), K_CAPS2.3 (LED), K_CTRL2.3 (LED)
- net COL0: now also K_ALT2.2 (COL), K_CAPS2.2 (COL), K_CTRL2.1 (ROW)
- net COL7: now also K_BACK2.1 (COL)
- net at D_BACK1.2 (A), K_BACK1.2 (ROW): now also K_BACK2.2 (ROW)
- net at K_BACK1.4 (LEDGND), R_BACK1.2: now also K_BACK2.4 (LEDGND)
- net at D_CAPS1.2 (A), K_CAPS1.2 (ROW): now also K_CAPS2.1 (ROW)
- net at K_CAPS1.4 (LEDGND), R_CAPS1.2: now also K_CAPS2.4 (LEDGND)
- net at D_CTRL1.2 (A), K_CTRL1.2 (ROW): now also K_CTRL2.2 (COL)
- net at K_CTRL1.4 (LEDGND), R_CTRL1.2: now also K_CTRL2.4 (LEDGND)
- net at D_WIN1.2 (A), K_WIN1.2 (ROW): now also K_ALT2.1 (ROW)
- net at K_WIN1.4 (LEDGND), R_WIN1.2: now also K_ALT2.4 (LEDGND)

Commit message: Wire more LEDs
Connections:
- net +5V: now also K_ISOENTER1.3 (LED)
- net COL7: now also K_ISOENTER1.1 (COL)
- net at D_ENTER1.2 (A), K_ENTER1.2 (ROW): now also K_ISOENTER1.2 (ROW)
- net at K_ENTER1.4 (LEDGND), R_ENTER1.2: now also K_ISOENTER1.4 (LEDGND)
Changed lines of the file:
@@
 	8700 4600 8700 4800
 Wire Wire Line
-	9200 4550 9275 4550
+	9200 4550 9650 4550
 Wire Wire Line
 	9150 4600 9150 4800
@@
 	9325 5350 9300 5350
 Wire Wire Line
-	9325 4450 9300 4450
+	9300 4450 9750 4450
 Connection ~ 9325 5350
 Wire Wire Line
@@
 Wire Wire Line
 	9150 2800 9600 2800
+Wire Wire Line
+	9800 4400 9350 4400
+Connection ~ 9275 4550
+Wire Wire Line
+	9600 4600 9150 4600
 $EndSCHEMATC

Commit message: Correct pinout for secondary layouts
Parts:
- K_RCTRL2: footprint MX_Alps_Hybrid:MX-1.5U -> MX_Alps_Hybrid:MX-1.5U-FLIPPED; symbol MX-1.5U -> MX-1.5U-FLIPPED
Connections:
- net +5V: now also K_CMD1.3 (LED), K_RALT1.3 (LED), K_RCTRL2.3 (LED), K_SHIFT2.3 (LED), K_SPACE2.3 (LED)
- net COL0: now also K_SHIFT2.1 (COL)
- net COL1: now also K_CMD1.2 (ROW)
- net COL3: now also K_SPACE2.1 (COL)
- net COL6: now also K_RALT1.2 (ROW)
- net COL7: now also K_RCTRL2.1 (ROW)
- net at K_SHIFT2.2 (ROW): now also D_SHIFT1.2 (A), K_SHIFT1.2 (ROW)
- net at K_SHIFT2.4 (LEDGND): now also K_SHIFT1.4 (LEDGND), R_SHIFT1.2
- net at D_ALT1.2 (A), K_ALT1.2 (ROW): now also K_CMD1.1 (COL)
- net at K_ALT1.4 (LEDGND), R_ALT1.2: now also K_CMD1.4 (LEDGND)
- net at D_SPACE1.2 (A), K_SPACE1.1 (ROW): now also K_SPACE2.2 (ROW)
- net at K_SPACE1.4 (LEDGND), R_SPACE1.2: now also K_SPACE2.4 (LEDGND)
- net at D_LEFT1.2 (A), K_LEFT1.2 (ROW): now also K_RALT1.1 (COL)
- net at K_LEFT1.4 (LEDGND), R_LEFT1.2: now also K_RALT1.4 (LEDGND)
- net at D_RIGHT1.2 (A), K_RIGHT1.2 (ROW): now also K_RCTRL2.2 (COL)
- net at K_RIGHT1.4 (LEDGND), R_RIGHT1.2: now also K_RCTRL2.4 (LEDGND)
Changed lines of the file:
@@
 $EndComp
 $Comp
-L MX-1.5U K_RCTRL2
+L MX-1.5U-FLIPPED K_RCTRL2
 U 1 1 59F16AE1
 P 9175 7125
 F 0 "K_RCTRL2" H 9175 7250 60  0000 C CNN
 F 1 "MX-1.5U" H 9175 7175 20  0000 C CNN
-F 2 "MX_Alps_Hybrid:MX-1.5U" H 9150 7100 60  0001 C CNN
+F 2 "MX_Alps_Hybrid:MX-1.5U-FLIPPED" H 9150 7100 60  0001 C CNN
 F 3 "" H 9150 7100 60  0001 C CNN
 	1    9175 7125
@@
 	9150 4600 9150 4800
 Wire Wire Line
-	2900 5450 2975 5450
+	2400 5450 2975 5450
 Wire Wire Line
 	2850 5500 2850 5700
@@
 	3025 2350 3025 7150
 Wire Wire Line
-	3025 5350 3000 5350
+	2500 5350 3025 5350
 Wire Wire Line
 	3025 6250 3000 6250
@@
 Connection ~ 3475 3550
 Wire Wire Line
-	3950 2150 3950 6200
+	3950 2150 3950 7075
 Wire Wire Line
 	3900 2150 4400 2150
@@
 	3925 6250 3900 6250
 Wire Wire Line
-	3925 2350 3925 6250
+	3925 2350 3925 7150
 Wire Wire Line
 	3925 5350 3900 5350
@@
 	5725 5350 5700 5350
 Wire Wire Line
-	5725 2350 5725 6250
+	5725 2350 5725 7150
 Wire Wire Line
 	5725 4450 5700 4450
@@
 	9325 6250 9300 6250
 Wire Wire Line
-	9325 2350 9325 6250
+	9325 2350 9325 7150
 Wire Wire Line
 	9325 5350 9300 5350
@@
 Connection ~ 5300 4400
 Wire Wire Line
-	5750 2150 5750 6200
+	5750 2150 5750 7100
 Connection ~ 5750 4400
 Connection ~ 5750 3500
@@
 	9300 2150 9350 2150
 Wire Wire Line
-	9350 2150 9350 6200
+	9350 2150 9350 7075
 Connection ~ 9350 2600
 Connection ~ 9350 3500
@@
 Connection ~ 8825 5650
 Wire Wire Line
-	8450 5700 8450 6200
+	8450 5700 8450 7075
 Wire Wire Line
 	8450 5700 8625 5700
@@
 	8600 5675 8425 5675
 Wire Wire Line
-	8425 5675 8425 6250
+	8425 5675 8425 7150
 Wire Wire Line
 	2625 6550 9275 6550
@@
 Wire Wire Line
 	9600 4600 9150 4600
+Wire Wire Line
+	3050 5300 2550 5300
+Connection ~ 3000 5350
+Connection ~ 2900 5450
+Wire Wire Line
+	2850 5500 2350 5500
+Wire Wire Line
+	3950 7075 3975 7075
+Wire Wire Line
+	3975 7075 3975 7125
+Wire Wire Line
+	3975 7125 3950 7125
+Wire Wire Line
+	3950 7125 3950 7300
+Wire Wire Line
+	3950 7300 3750 7300
+Connection ~ 3950 6200
+Wire Wire Line
+	3950 7100 3725 7100
+Wire Wire Line
+	3725 7100 3725 6400
+Wire Wire Line
+	3725 6400 3750 6400
+Wire Wire Line
+	3925 7150 3900 7150
+Connection ~ 3925 6250
+Wire Wire Line
+	3800 6350 3800 7250
+Connection ~ 5750 6200
+Wire Wire Line
+	5725 7150 5700 7150
+Connection ~ 5725 6250
+Wire Wire Line
+	5600 6350 5600 7250
+Wire Wire Line
+	5550 7300 5525 7300
+Wire Wire Line
+	5525 7300 5525 6400
+Wire Wire Line
+	5525 6400 5550 6400
+Wire Wire Line
+	8450 7075 8475 7075
+Wire Wire Line
+	8475 7075 8475 7125
+Wire Wire Line
+	8475 7125 8450 7125
+Wire Wire Line
+	8450 7125 8450 7300
+Wire Wire Line
+	8450 7300 8250 7300
+Connection ~ 8450 6200
+Wire Wire Line
+	8450 7100 8225 7100
+Wire Wire Line
+	8225 7100 8225 6400
+Wire Wire Line
+	8225 6400 8250 6400
+Wire Wire Line
+	8300 6350 8300 7250
+Wire Wire Line
+	8425 7150 8400 7150
+Connection ~ 8425 6250
+Wire Wire Line
+	9150 7300 9350 7300
+Wire Wire Line
+	9350 7300 9350 7125
+Wire Wire Line
+	9350 7125 9375 7125
+Wire Wire Line
+	9375 7125 9375 7075
+Wire Wire Line
+	9375 7075 9350 7075
+Connection ~ 9350 6200
+Wire Wire Line
+	9325 7150 9300 7150
+Connection ~ 9325 6250
+Wire Wire Line
+	9350 7100 9125 7100
+Wire Wire Line
+	9125 7100 9125 6400
+Wire Wire Line
+	9125 6400 9150 6400
+Wire Wire Line
+	9200 6350 9200 7250
 $EndSCHEMATC

Commit message: Wire more LEDs
Connections:
- net COL7: now also K_RCTRL2.2 (COL); no longer K_RCTRL2.1 (ROW)
- net at D_RIGHT1.2 (A), K_RIGHT1.2 (ROW): now also K_RCTRL2.1 (ROW); no longer K_RCTRL2.2 (COL)
Changed lines of the file:
@@
 	9300 2150 9350 2150
 Wire Wire Line
-	9350 2150 9350 7075
+	9350 2150 9350 7100
 Connection ~ 9350 2600
 Connection ~ 9350 3500
@@
 	8425 7150 8400 7150
 Connection ~ 8425 6250
-Wire Wire Line
-	9150 7300 9350 7300
-Wire Wire Line
-	9350 7300 9350 7125
-Wire Wire Line
-	9350 7125 9375 7125
-Wire Wire Line
-	9375 7125 9375 7075
-Wire Wire Line
-	9375 7075 9350 7075
 Connection ~ 9350 6200
 Wire Wire Line
@@
 Connection ~ 9325 6250
 Wire Wire Line
-	9350 7100 9125 7100
-Wire Wire Line
-	9125 7100 9125 6400
+	9200 6350 9200 7250
+Wire Wire Line
+	9150 7300 9125 7300
+Wire Wire Line
+	9125 7300 9125 6400
 Wire Wire Line
 	9125 6400 9150 6400
-Wire Wire Line
-	9200 6350 9200 7250
 $EndSCHEMATC

Commit message: Finish 5V, GND, LEDGND
Connections:
- net +5V: now also K_/2.3 (LED)
- net COL5: now also K_/2.2 (ROW)
- net at D_/1.2 (A), K_/1.2 (ROW): now also K_/2.1 (COL)
- net at K_/1.4 (LEDGND), R_/1.2: now also K_/2.4 (LEDGND)
Changed lines of the file:
@@
 	7350 5500 7350 5700
 Wire Wire Line
-	7850 5450 7925 5450
+	7850 5450 8300 5450
 Wire Wire Line
 	7800 5500 7800 5700
@@
 Connection ~ 7975 3550
 Wire Wire Line
-	7975 5350 7950 5350
+	7950 5350 8400 5350
 Connection ~ 7975 4450
 Wire Wire Line
@@
 Wire Wire Line
 	9125 6400 9150 6400
+Wire Wire Line
+	8450 5300 8125 5300
+Wire Wire Line
+	8125 5300 8125 5500
+Wire Wire Line
+	8125 5500 7800 5500
+Wire Wire Line
+	8000 5300 8100 5300
+Wire Wire Line
+	8100 5300 8100 5475
+Wire Wire Line
+	8100 5475 8250 5475
+Wire Wire Line
+	8250 5475 8250 5500
+Connection ~ 7925 5450
 $EndSCHEMATC

Commit message: Fix RShift
Parts:
- K_RSHIFT2: footprint MX_Alps_Hybrid:MX-2.75U -> MX_Alps_Hybrid:MX-2.75U-FLIPPED; symbol MX-2.75U -> MX-2.75U-FLIPPED
Connections:
- net +5V: now also K_RSHIFT2.3 (LED)
- net COL6: now also K_RSHIFT2.1 (ROW)
- net at D_UP1.2 (A), K_UP1.2 (ROW): now also K_RSHIFT2.2 (COL)
- net at K_UP1.4 (LEDGND), R_UP1.2: now also K_RSHIFT2.4 (LEDGND)
Changed lines of the file:
@@
 $EndComp
 $Comp
-L MX-2.75U K_RSHIFT2
+L MX-2.75U-FLIPPED K_RSHIFT2
 U 1 1 59ED76B9
 P 9625 5325
 F 0 "K_RSHIFT2" H 9725 5450 60  0000 C CNN
 F 1 "MX-2.75U" H 9625 5375 20  0000 C CNN
-F 2 "MX_Alps_Hybrid:MX-2.75U" H 9600 5300 60  0001 C CNN
+F 2 "MX_Alps_Hybrid:MX-2.75U-FLIPPED" H 9600 5300 60  0001 C CNN
 F 3 "" H 9600 5300 60  0001 C CNN
 	1    9625 5325
@@
 	7800 5500 7800 5700
 Wire Wire Line
-	8750 5450 8825 5450
+	8750 5450 9175 5450
 Wire Wire Line
 	8700 5500 8700 5700
@@
 Connection ~ 8875 3550
 Wire Wire Line
-	8875 5350 8850 5350
+	8850 5350 8925 5350
 Connection ~ 8875 4450
 Wire Wire Line
@@
 	8250 5475 8250 5500
 Connection ~ 7925 5450
+Wire Wire Line
+	9750 5350 9750 5375
+Wire Wire Line
+	9750 5375 8925 5375
+Wire Wire Line
+	8925 5375 8925 5350
+Wire Wire Line
+	9175 5450 9175 5425
+Wire Wire Line
+	9175 5425 9650 5425
+Wire Wire Line
+	9650 5425 9650 5450
+Connection ~ 8825 5450
+Wire Wire Line
+	9800 5300 9800 5525
+Wire Wire Line
+	9800 5525 8700 5525
+Connection ~ 8700 5525
+Wire Wire Line
+	8900 5300 8925 5300
+Wire Wire Line
+	8925 5300 8925 5275
+Wire Wire Line
+	8925 5275 9600 5275
+Wire Wire Line
+	9600 5275 9600 5500
 $EndSCHEMATC

Commit message: Update notes on schematic for Voyager 1.0 release
Other:
- note added: "1.0"
- note added: "Voyager Keyboard - Matrix"
- note removed: "Matrix"
Changed lines of the file:
@@
 LIBS:keyboard_parts
 LIBS:mkl27z256vfm4
-LIBS:Chronos-cache
+LIBS:Voyager-cache
 EELAYER 25 0
 EELAYER END
@@
 $EndDescr
 Text Notes 12175 10925 0    60   ~ 0
-Matrix
+Voyager Keyboard - Matrix
 Text Notes 12950 11075 0    60   ~ 0
 2017-10-16
@@
 Wire Wire Line
 	9600 5275 9600 5500
+Text Notes 15400 11075 0    60   ~ 0
+1.0
 $EndSCHEMATC

Commit message: CvPcb - Change all SMA diodes to SOD323-Handsoldering
Parts:
- D_#0_1, D_#1, D_#2, D_#3, D_#4, D_#5, D_#6, D_#7, D_#8, D_#9, D_'1, D_,1, D_-1, D_.1, D_/1, D_;1, D_=1, D_A1, D_ALT1, D_B1, D_BACK1, D_C1, D_CAPS1, D_CTRL1, D_D1, D_DEL1, D_DOWN1, D_E1, D_ENTER1, D_ESC1, D_F1, D_FN1, D_G1, D_H1, D_I1, D_ISO\1, D_ISO`1, D_J1, D_K1, D_L1, D_LEFT1, D_M1, D_N1, D_O1, D_P1, D_Q1, D_R1, D_RIGHT1, D_RSHIFT1, D_S1, D_SHIFT1, D_SPACE1, D_T1, D_TAB1, D_U1, D_UP1, D_V1, D_W1, D_WIN1, D_X1, D_Y1, D_Z1, D_[1, D_\1, D_]1, D_`1: footprint Diodes_SMD:D_SMA -> Diodes_SMD:D_SOD-323_HandSoldering
