File: Chronos.kicad_pcb (KiCad board)
At the start: 2 copper layers, 285 x 94.6 mm, 259 parts, among them Q1 NSS40301MZ4T1G, SW1 SW_PUSH, U1 ATMEGA32U2-AU, Y1 16MHz

Commit message: Switch fp 3rd row
Parts:
- moved K_ISOENTER1 332.7 mm to (321.5, 85.7)
- moved K_ENTER1 326.2 mm to (311.9, 95.2)
- moved K_ISO`1 314.8 mm to (300.0, 95.2)
- moved K_'1 296.7 mm to (281.0, 95.2)
- moved K_;1 278.7 mm to (261.9, 95.2)
- moved K_L1 260.9 mm to (242.9, 95.2)
- moved K_K1 243.3 mm to (223.8, 95.2)
- moved K_J1 225.9 mm to (204.8, 95.2)
- moved K_H1 208.7 mm to (185.7, 95.2)
- moved K_G1 192.0 mm to (166.7, 95.2)
- moved K_F1 175.7 mm to (147.6, 95.2)
- moved K_D1 160.0 mm to (128.6, 95.2)
- moved K_S1 145.2 mm to (109.5, 95.2)
- moved K_A1 131.4 mm to (90.5, 95.2)
- moved K_CAPS1 114.9 mm to (64.3, 95.2)
Changed lines of the file:
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@@
   )
   (module MX_Alps_Hybrid:MX-1U (layer F.Cu)
-    (at 0 0)
+    (at 280.9875 95.25)
     (fp_text reference K_'1 (at 0 3.175) (layer F.SilkS)
       (effects (font (size 1 1) (thickness 0.15)))
@@
   )
   (module MX_Alps_Hybrid:MX-1U (layer F.Cu)
-    (at 0 0)
+    (at 261.9375 95.25)
     (fp_text reference K_;1 (at 0 3.175) (layer F.SilkS)
       (effects (font (size 1 1) (thickness 0.15)))
@@
   )
   (module MX_Alps_Hybrid:MX-1U (layer F.Cu)
-    (at 0 0)
+    (at 90.4875 95.25)
     (fp_text reference K_A1 (at 0 3.175) (layer F.SilkS)
       (effects (font (size 1 1) (thickness 0.15)))
@@
   )
   (module MX_Alps_Hybrid:MX-1.75U (layer F.Cu)
-    (at 0 0)
+    (at 64.29375 95.25)
     (fp_text reference K_CAPS1 (at 0 3.175) (layer F.SilkS)
       (effects (font (size 1 1) (thickness 0.15)))
@@
   )
   (module MX_Alps_Hybrid:MX-1U (layer F.Cu)
-    (at 0 0)
+    (at 128.5875 95.25)
     (fp_text reference K_D1 (at 0 3.175) (layer F.SilkS)
       (effects (font (size 1 1) (thickness 0.15)))
@@
   )
   (module MX_Alps_Hybrid:MX-2.25U (layer F.Cu)
-    (at 0 0)
+    (at 311.94375 95.25)
     (fp_text reference K_ENTER1 (at 0 3.175) (layer F.SilkS)
       (effects (font (size 1 1) (thickness 0.15)))
@@
   )
   (module MX_Alps_Hybrid:MX-1U (layer F.Cu)
-    (at 0 0)
+    (at 147.6375 95.25)
     (fp_text reference K_F1 (at 0 3.175) (layer F.SilkS)
       (effects (font (size 1 1) (thickness 0.15)))
@@
   )
   (module MX_Alps_Hybrid:MX-1U (layer F.Cu)
-    (at 0 0)
+    (at 166.6875 95.25)
     (fp_text reference K_G1 (at 0 3.175) (layer F.SilkS)
       (effects (font (size 1 1) (thickness 0.15)))
@@
   )
   (module MX_Alps_Hybrid:MX-1U (layer F.Cu)
-    (at 0 0)
+    (at 185.7375 95.25)
     (fp_text reference K_H1 (at 0 3.175) (layer F.SilkS)
       (effects (font (size 1 1) (thickness 0.15)))
@@
   )
   (module MX_Alps_Hybrid:MX-ISO-Combined (layer F.Cu)
-    (at 0 0)
+    (at 321.46875 85.725)
     (fp_text reference K_ISOENTER1 (at 0 3.175) (layer F.SilkS)
       (effects (font (size 1 1) (thickness 0.15)))
@@
   )
   (module MX_Alps_Hybrid:MX-1U (layer F.Cu)
-    (at 0 0)
+    (at 300.0375 95.25)
     (fp_text reference K_ISO`1 (at 0 3.175) (layer F.SilkS)
       (effects (font (size 1 1) (thickness 0.15)))
@@
   )
   (module MX_Alps_Hybrid:MX-1U (layer F.Cu)
-    (at 0 0)
+    (at 204.7875 95.25)
     (fp_text reference K_J1 (at 0 3.175) (layer F.SilkS)
       (effects (font (size 1 1) (thickness 0.15)))
@@
   )
   (module MX_Alps_Hybrid:MX-1U (layer F.Cu)
-    (at 0 0)
+    (at 223.8375 95.25)
     (fp_text reference K_K1 (at 0 3.175) (layer F.SilkS)
       (effects (font (size 1 1) (thickness 0.15)))
@@
   )
   (module MX_Alps_Hybrid:MX-1U (layer F.Cu)
-    (at 0 0)
+    (at 242.8875 95.25)
     (fp_text reference K_L1 (at 0 3.175) (layer F.SilkS)
       (effects (font (size 1 1) (thickness 0.15)))
@@
   )
   (module MX_Alps_Hybrid:MX-1U (layer F.Cu)
-    (at 0 0)
+    (at 109.5375 95.25)
     (fp_text reference K_S1 (at 0 3.175) (layer F.SilkS)
       (effects (font (size 1 1) (thickness 0.15)))

Commit message: Finish primary bottom row switches
Parts:
- added K_SHIFT2: MX-1.25U, MX_Alps_Hybrid:MX-1.25U, F.Cu at (59.5, 114.3)
- moved K_RIGHT1 350.2 mm to (323.9, 133.3)
- moved K_RSHIFT1 343.4 mm to (323.9, 114.3)
- moved K_DOWN1 332.7 mm to (304.8, 133.3)
- moved K_RSHIFT2 327.8 mm to (307.2, 114.3)
- moved K_UP1 325.5 mm to (304.8, 114.3)
- moved K_LEFT1 315.3 mm to (285.8, 133.3)
- moved K_/1 301.1 mm to (278.6, 114.3)
- moved K_`1 298.2 mm to (266.7, 133.3)
- moved K_/2 294.5 mm to (271.5, 114.3)
- moved K_FN1 281.3 mm to (247.7, 133.3)
- moved K_.1 277.1 mm to (252.4, 114.3)
- moved K_,1 259.9 mm to (233.4, 114.3)
- moved K_M1 242.9 mm to (214.3, 114.3)
- moved K_N1 226.3 mm to (195.3, 114.3)
- moved K_SPACE1 222.9 mm to (178.6, 133.3)
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Changed lines of the file:
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@@
 (kicad_pcb (version 4) (host pcbnew 4.0.6)
   (general
-    (links 647)
-    (no_connects 186)
-    (area -62.187501 -106.881251 353.563451 55.043751)
+    (links 649)
+    (no_connects 266)
+    (area 0 0 0 0)
     (thickness 1.6)
     (drawings 0)
     (tracks 0)
     (zones 0)
-    (modules 259)
-    (nets 261)
+    (modules 260)
+    (nets 265)
   )
   (page A3)
@@
   (net 259 "Net-(U1-Pad26)")
   (net 260 "Net-(USB1-Pad2)")
+  (net 261 "Net-(K_SHIFT2-Pad2)")
+  (net 262 "Net-(K_SHIFT2-Pad1)")
+  (net 263 "Net-(K_SHIFT2-Pad3)")
+  (net 264 "Net-(K_SHIFT2-Pad4)")
   (net_class Default "This is the default net class."
     (clearance 0.2)
@@
     (add_net "Net-(K_S1-Pad4)")
     (add_net "Net-(K_SHIFT1-Pad4)")
+    (add_net "Net-(K_SHIFT2-Pad1)")
+    (add_net "Net-(K_SHIFT2-Pad2)")
+    (add_net "Net-(K_SHIFT2-Pad3)")
+    (add_net "Net-(K_SHIFT2-Pad4)")
     (add_net "Net-(K_SPACE1-Pad4)")
     (add_net "Net-(K_SPACE2-Pad1)")
@@
   )
   (module MX_Alps_Hybrid:MX-1U (layer F.Cu)
-    (at 0 0)
+    (at 233.3625 114.3)
     (fp_text reference K_,1 (at 0 3.175) (layer F.SilkS)
       (effects (font (size 1 1) (thickness 0.15)))
@@
   )
   (module MX_Alps_Hybrid:MX-1U (layer F.Cu)
-    (at 0 0)
+    (at 252.4125 114.3)
     (fp_text reference K_.1 (at 0 3.175) (layer F.SilkS)
       (effects (font (size 1 1) (thickness 0.15)))
@@
   )
   (module MX_Alps_Hybrid:MX-1.75U (layer F.Cu)
-    (at 0 0)
+    (at 278.60625 114.3)
     (fp_text reference K_/1 (at 0 3.175) (layer F.SilkS)
       (effects (font (size 1 1) (thickness 0.15)))
@@
   )
   (module MX_Alps_Hybrid:MX-1U (layer F.Cu)
-    (at 0 0)
+    (at 271.4625 114.3)
     (fp_text reference K_/2 (at 0 3.175) (layer F.SilkS)
       (effects (font (size 1 1) (thickness 0.15)))
@@
   )
   (module MX_Alps_Hybrid:MX-1.25U (layer F.Cu)
-    (at 0 0)
+    (at 107.15625 133.35)
     (fp_text reference K_ALT1 (at 0 3.175) (layer F.SilkS)
       (effects (font (size 1 1) (thickness 0.15)))
@@
   )
   (module MX_Alps_Hybrid:MX-1U (layer F.Cu)
-    (at 0 0)
+    (at 176.2125 114.3)
     (fp_text reference K_B1 (at 0 3.175) (layer F.SilkS)
       (effects (font (size 1 1) (thickness 0.15)))
@@
   )
   (module MX_Alps_Hybrid:MX-1U (layer F.Cu)
-    (at 0 0)
+    (at 138.1125 114.3)
     (fp_text reference K_C1 (at 0 3.175) (layer F.SilkS)
       (effects (font (size 1 1) (thickness 0.15)))
@@
   )
   (module MX_Alps_Hybrid:MX-1.25U (layer F.Cu)
-    (at 0 0)
+    (at 59.53125 133.35)
     (fp_text reference K_CTRL1 (at 0 3.175) (layer F.SilkS)
       (effects (font (size 1 1) (thickness 0.15)))
@@
   )
   (module MX_Alps_Hybrid:MX-1U (layer F.Cu)
-    (at 0 0)
+    (at 304.8 133.35)
     (fp_text reference K_DOWN1 (at 0 3.175) (layer F.SilkS)
       (effects (font (size 1 1) (thickness 0.15)))
@@
   )
   (module MX_Alps_Hybrid:MX-1U (layer F.Cu)
-    (at 0 0)
+    (at 247.65 133.35)
     (fp_text reference K_FN1 (at 0 3.175) (layer F.SilkS)
       (effects (font (size 1 1) (thickness 0.15)))
@@
   )
   (module MX_Alps_Hybrid:MX-1U (layer F.Cu)
-    (at 0 0)
+    (at 80.9625 114.3)
     (fp_text reference K_ISO\1 (at 0 3.175) (layer F.SilkS)
       (effects (font (size 1 1) (thickness 0.15)))
@@
   )
   (module MX_Alps_Hybrid:MX-1U (layer F.Cu)
-    (at 0 0)
+    (at 285.75 133.35)
     (fp_text reference K_LEFT1 (at 0 3.175) (layer F.SilkS)
       (effects (font (size 1 1) (thickness 0.15)))
@@
   )
   (module MX_Alps_Hybrid:MX-1U (layer F.Cu)
-    (at 0 0)
+    (at 214.3125 114.3)
     (fp_text reference K_M1 (at 0 3.175) (layer F.SilkS)
       (effects (font (size 1 1) (thickness 0.15)))
@@
   )
   (module MX_Alps_Hybrid:MX-1U (layer F.Cu)
-    (at 0 0)
+    (at 195.2625 114.3)
     (fp_text reference K_N1 (at 0 3.175) (layer F.SilkS)
       (effects (font (size 1 1) (thickness 0.15)))
@@
   )
   (module MX_Alps_Hybrid:MX-1U (layer F.Cu)
-    (at 0 0)
+    (at 323.85 133.35)
     (fp_text reference K_RIGHT1 (at 0 3.175) (layer F.SilkS)
       (effects (font (size 1 1) (thickness 0.15)))
@@
   )
   (module MX_Alps_Hybrid:MX-1U (layer F.Cu)
-    (at 0 0)
+    (at 323.85 114.3)
     (fp_text reference K_RSHIFT1 (at 0 3.175) (layer F.SilkS)
       (effects (font (size 1 1) (thickness 0.15)))
@@
   )
   (module MX_Alps_Hybrid:MX-2.75U (layer F.Cu)
-    (at 0 0)
+    (at 307.18125 114.3)
     (fp_text reference K_RSHIFT2 (at 0 3.175) (layer F.SilkS)
       (effects (font (size 1 1) (thickness 0.15)))
@@
   )
   (module MX_Alps_Hybrid:MX-2.25U (layer F.Cu)
-    (at 0 0)
+    (at 69.05625 114.3)
     (fp_text reference K_SHIFT1 (at 0 3.175) (layer F.SilkS)
       (effects (font (size 1 1) (thickness 0.15)))
@@
   )
   (module MX_Alps_Hybrid:MX-6.25U-ReversedStabilizers (layer F.Cu)
-    (at 0 0)
+    (at 178.59375 133.35)
     (fp_text reference K_SPACE1 (at 0 3.175) (layer F.SilkS)
       (effects (font (size 1 1) (thickness 0.15)))
@@
   )
   (module MX_Alps_Hybrid:MX-1U (layer F.Cu)
-    (at 0 0)
+    (at 304.8 114.3)
     (fp_text reference K_UP1 (at 0 3.175) (layer F.SilkS)
       (effects (font (size 1 1) (thickness 0.15)))
@@
   )
   (module MX_Alps_Hybrid:MX-1U (layer F.Cu)
-    (at 0 0)
+    (at 157.1625 114.3)
     (fp_text reference K_V1 (at 0 3.175) (layer F.SilkS)
       (effects (font (size 1 1) (thickness 0.15)))
@@
   )
   (module MX_Alps_Hybrid:MX-1.25U (layer F.Cu)
-    (at 0 0)
+    (at 83.34375 133.35)
     (fp_text reference K_WIN1 (at 0 3.175) (layer F.SilkS)
       (effects (font (size 1 1) (thickness 0.15)))
@@
   )
   (module MX_Alps_Hybrid:MX-1U (layer F.Cu)
-    (at 0 0)
+    (at 119.0625 114.3)
     (fp_text reference K_X1 (at 0 3.175) (layer F.SilkS)
       (effects (font (size 1 1) (thickness 0.15)))
@@
   )
   (module MX_Alps_Hybrid:MX-1U (layer F.Cu)
-    (at 0 0)
+    (at 100.0125 114.3)
     (fp_text reference K_Z1 (at 0 3.175) (layer F.SilkS)
       (effects (font (size 1 1) (thickness 0.15)))
@@
   )
   (module MX_Alps_Hybrid:MX-1U (layer F.Cu)
-    (at 0 0)
+    (at 266.7 133.35)
     (fp_text reference K_`1 (at 0 3.175) (layer F.SilkS)
       (effects (font (size 1 1) (thickness 0.15)))
@@
     )
   )
+  (module MX_Alps_Hybrid:MX-1.25U (layer F.Cu)
+    (at 59.53125 114.3)
+    (fp_text reference K_SHIFT2 (at 0 3.175) (layer F.SilkS)
+      (effects (font (size 1 1) (thickness 0.15)))
+    )
+    (fp_text value MX-1.25U (at 0 -7.9375) (layer Dwgs.User)
+      (effects (font (size 1 1) (thickness 0.15)))
+    )
+    (fp_line (start 5 -7) (end 7 -7) (layer Dwgs.User) (width 0.15))
+    (fp_line (start 7 -7) (end 7 -5) (layer Dwgs.User) (width 0.15))
+    (fp_line (start 5 7) (end 7 7) (layer Dwgs.User) (width 0.15))
+    (fp_line (start 7 7) (end 7 5) (layer Dwgs.User) (width 0.15))
+    (fp_line (start -7 5) (end -7 7) (layer Dwgs.User) (width 0.15))
+    (fp_line (start -7 7) (end -5 7) (layer Dwgs.User) (width 0.15))
+    (fp_line (start -5 -7) (end -7 -7) (layer Dwgs.User) (width 0.15))
+    (fp_line (start -7 -7) (end -7 -5) (layer Dwgs.User) (width 0.15))
+    (fp_line (start -11.90625 -9.525) (end 11.90625 -9.525) (layer Dwgs.User) (width 0.15))
+    (fp_line (start 11.90625 -9.525) (end 11.90625 9.525) (layer Dwgs.User) (width 0.15))
+    (fp_line (start -11.90625 9.525) (end 11.90625 9.525) (layer Dwgs.User) (width 0.15))
+    (fp_line (start -11.90625 9.525) (end -11.90625 -9.525) (layer Dwgs.User) (width 0.15))
+    (pad 2 thru_hole oval (at 2.5 -4.5 86.0548) (size 2.831378 2.25) (drill 1.47 (offset 0.290689 0)) (layers *.Cu *.Mask)
+      (net 261 "Net-(K_SHIFT2-Pad2)"))
+    (pad 2 thru_hole circle (at 2.54 -5.08) (size 2.25 2.25) (drill 1.47) (layers *.Cu *.Mask)
+      (net 261 "Net-(K_SHIFT2-Pad2)"))
+    (pad 1 thru_hole oval (at -3.81 -2.54 48.09963212) (size 4.211556 2.25) (drill 1.47 (offset 0.980778 0)) (layers *.Cu *.Mask)
+      (net 262 "Net-(K_SHIFT2-Pad1)"))
+    (pad "" np_thru_hole circle (at 0 0) (size 3.9878 3.9878) (drill 3.9878) (layers *.Cu *.Mask))
+    (pad 1 thru_hole circle (at -2.5 -4) (size 2.25 2.25) (drill 1.47) (layers *.Cu *.Mask)
+      (net 262 "Net-(K_SHIFT2-Pad1)"))
+    (pad 3 thru_hole circle (at -1.27 5.08) (size 1.905 1.905) (drill 1.04) (layers *.Cu *.Mask)
+      (net 263 "Net-(K_SHIFT2-Pad3)"))
+    (pad 4 thru_hole rect (at 1.27 5.08) (size 1.905 1.905) (drill 1.04) (layers *.Cu *.Mask)
+      (net 264 "Net-(K_SHIFT2-Pad4)"))
+    (pad "" np_thru_hole circle (at -5.08 0 48.0996) (size 1.7018 1.7018) (drill 1.7018) (layers *.Cu *.Mask))
+    (pad "" np_thru_hole circle (at 5.08 0 48.0996) (size 1.7018 1.7018) (drill 1.7018) (layers *.Cu *.Mask))
+  )
 )
