File: Chronos.kicad_pcb (KiCad board)
At the start: 2 copper layers, 285 x 94.6 mm, 256 parts, among them Q1 NSS40301MZ4T1G, SW1 SW_PUSH, U1 ATMEGA32U2-AU, Y1 16MHz

Commit message: Place 22ohm resistors and PTC
Parts:
- moved F1 88.5 mm to (63.1, 62.2), turned to 90 degrees
- moved R2 86.7 mm to (70.2, 61.9), turned to 90 degrees
- moved R3 84.4 mm to (66.7, 61.9), turned to 90 degrees
- moved R_ESC1 17.2 mm to (50.0, 52.4), turned to 270 degrees
- moved D_#1 1.31 mm to (85.7, 53.6)
- moved D_#2 1.31 mm to (104.8, 53.6)
- moved D_#3 1.31 mm to (123.8, 53.6)
Routing:
- net DP: track 0.00 -> 8.26 mm
- net DM: track 0.00 -> 7.11 mm
- net VCC: track 0.00 -> 6.97 mm
Changed lines of the file:
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@@
     (thickness 1.6)
     (drawings 0)
-    (tracks 0)
+    (tracks 9)
     (zones 0)
     (modules 256)
@@
   )
   (module Fuse_Holders_and_Fuses:Fuse_SMD1206_HandSoldering (layer B.Cu)
-    (at 0 0.134814)
+    (at 63.103125 62.20375 90)
     (descr "Fuse, Sicherung, SMD1206, Littlefuse-Wickmann 433 Series, Hand Soldering,")
     (tags "Fuse Sicherung SMD1206 Littlefuse-Wickmann 433 Series Hand Soldering ")
     (attr smd)
-    (fp_text reference F1 (at -0.05 2.2) (layer B.SilkS)
+    (fp_text reference F1 (at -0.05 2.2 90) (layer B.SilkS)
       (effects (font (size 1 1) (thickness 0.15)) (justify mirror))
     )
-    (fp_text value 500mA (at -0.15 -2.5) (layer B.Fab)
+    (fp_text value 500mA (at -0.15 -2.5 90) (layer B.Fab)
       (effects (font (size 1 1) (thickness 0.15)) (justify mirror))
     )
@@
     (fp_line (start 3.35 -1.58) (end 3.35 1.58) (layer B.CrtYd) (width 0.05))
     (fp_line (start 3.35 -1.58) (end -3.35 -1.58) (layer B.CrtYd) (width 0.05))
-    (pad 1 smd rect (at -2.09 0 270) (size 2.03 2.65) (layers B.Cu B.Paste B.Mask)
+    (pad 1 smd rect (at -2.09 0) (size 2.03 2.65) (layers B.Cu B.Paste B.Mask)
       (net 5 +5V))
-    (pad 2 smd rect (at 2.09 0 270) (size 2.03 2.65) (layers B.Cu B.Paste B.Mask)
+    (pad 2 smd rect (at 2.09 0) (size 2.03 2.65) (layers B.Cu B.Paste B.Mask)
       (net 82 VCC))
   )
@@
   )
   (module Resistors_SMD:R_0805_HandSoldering (layer B.Cu)
-    (at 11.90625 -2.246436)
+    (at 70.246875 61.9125 90)
     (descr "Resistor SMD 0805, hand soldering")
     (tags "resistor 0805")
     (attr smd)
-    (fp_text reference R2 (at 0 1.7) (layer B.SilkS)
+    (fp_text reference R2 (at 0 1.7 90) (layer B.SilkS)
       (effects (font (size 1 1) (thickness 0.15)) (justify mirror))
     )
-    (fp_text value 22 (at 0 -1.75) (layer B.Fab)
+    (fp_text value 22 (at 0 -1.75 90) (layer B.Fab)
       (effects (font (size 1 1) (thickness 0.15)) (justify mirror))
     )
-    (fp_text user %R (at 0 0) (layer B.Fab)
+    (fp_text user %R (at 0 0 90) (layer B.Fab)
       (effects (font (size 0.5 0.5) (thickness 0.075)) (justify mirror))
     )
@@
     (fp_line (start 2.35 -0.9) (end 2.35 0.9) (layer B.CrtYd) (width 0.05))
     (fp_line (start 2.35 -0.9) (end -2.35 -0.9) (layer B.CrtYd) (width 0.05))
-    (pad 1 smd rect (at -1.35 0) (size 1.5 1.3) (layers B.Cu B.Paste B.Mask)
+    (pad 1 smd rect (at -1.35 0 90) (size 1.5 1.3) (layers B.Cu B.Paste B.Mask)
       (net 204 "Net-(R2-Pad1)"))
-    (pad 2 smd rect (at 1.35 0) (size 1.5 1.3) (layers B.Cu B.Paste B.Mask)
+    (pad 2 smd rect (at 1.35 0 90) (size 1.5 1.3) (layers B.Cu B.Paste B.Mask)
       (net 205 DP))
     (model ${KISYS3DMOD}/Resistors_SMD.3dshapes/R_0805.wrl
@@
   )
   (module Resistors_SMD:R_0805_HandSoldering (layer B.Cu)
-    (at 11.90625 -2.246436)
+    (at 66.675 61.9125 90)
     (descr "Resistor SMD 0805, hand soldering")
     (tags "resistor 0805")
     (attr smd)
-    (fp_text reference R3 (at 0 1.7) (layer B.SilkS)
+    (fp_text reference R3 (at 0 1.7 90) (layer B.SilkS)
       (effects (font (size 1 1) (thickness 0.15)) (justify mirror))
     )
-    (fp_text value 22 (at 0 -1.75) (layer B.Fab)
+    (fp_text value 22 (at 0 -1.75 90) (layer B.Fab)
       (effects (font (size 1 1) (thickness 0.15)) (justify mirror))
     )
-    (fp_text user %R (at 0 0) (layer B.Fab)
+    (fp_text user %R (at 0 0 90) (layer B.Fab)
       (effects (font (size 0.5 0.5) (thickness 0.075)) (justify mirror))
     )
@@
     (fp_line (start 2.35 -0.9) (end 2.35 0.9) (layer B.CrtYd) (width 0.05))
     (fp_line (start 2.35 -0.9) (end -2.35 -0.9) (layer B.CrtYd) (width 0.05))
-    (pad 1 smd rect (at -1.35 0) (size 1.5 1.3) (layers B.Cu B.Paste B.Mask)
+    (pad 1 smd rect (at -1.35 0 90) (size 1.5 1.3) (layers B.Cu B.Paste B.Mask)
       (net 206 "Net-(R3-Pad1)"))
-    (pad 2 smd rect (at 1.35 0) (size 1.5 1.3) (layers B.Cu B.Paste B.Mask)
+    (pad 2 smd rect (at 1.35 0 90) (size 1.5 1.3) (layers B.Cu B.Paste B.Mask)
       (net 207 DM))
     (model ${KISYS3DMOD}/Resistors_SMD.3dshapes/R_0805.wrl
@@
   )
   (module Resistors_SMD:R_1206_HandSoldering (layer B.Cu)
-    (at 64.29375 61.9125 180)
+    (at 50.00625 52.3875 270)
     (descr "Resistor SMD 1206, hand soldering")
     (tags "resistor 1206")
     (attr smd)
-    (fp_text reference R_ESC1 (at 0 1.85 180) (layer B.SilkS)
+    (fp_text reference R_ESC1 (at 0 1.85 270) (layer B.SilkS)
       (effects (font (size 1 1) (thickness 0.15)) (justify mirror))
     )
-    (fp_text value 2.7k (at 0 -1.9 180) (layer B.Fab)
+    (fp_text value 2.7k (at 0 -1.9 270) (layer B.Fab)
       (effects (font (size 1 1) (thickness 0.15)) (justify mirror))
     )
-    (fp_text user %R (at 0 0 180) (layer B.Fab)
+    (fp_text user %R (at 0 0 270) (layer B.Fab)
       (effects (font (size 0.7 0.7) (thickness 0.105)) (justify mirror))
     )
@@
     (fp_line (start 3.25 -1.1) (end 3.25 1.11) (layer B.CrtYd) (width 0.05))
     (fp_line (start 3.25 -1.1) (end -3.25 -1.1) (layer B.CrtYd) (width 0.05))
-    (pad 1 smd rect (at -2 0 180) (size 2 1.7) (layers B.Cu B.Paste B.Mask)
+    (pad 1 smd rect (at -2 0 270) (size 2 1.7) (layers B.Cu B.Paste B.Mask)
       (net 2 GND))
-    (pad 2 smd rect (at 2 0 180) (size 2 1.7) (layers B.Cu B.Paste B.Mask)
+    (pad 2 smd rect (at 2 0 270) (size 2 1.7) (layers B.Cu B.Paste B.Mask)
       (net 140 "Net-(K_ESC1-Pad4)"))
     (model ${KISYS3DMOD}/Resistors_SMD.3dshapes/R_1206.wrl
@@
   )
   (module Diodes_SMD:D_SMA (layer B.Cu)
-    (at 85.725 54.8875 270)
+    (at 85.725 53.578125 270)
     (descr "Diode SMA (DO-214AC)")
     (tags "Diode SMA (DO-214AC)")
@@
   )
   (module Diodes_SMD:D_SMA (layer B.Cu)
-    (at 104.775 54.8875 270)
+    (at 104.775 53.578125 270)
     (descr "Diode SMA (DO-214AC)")
     (tags "Diode SMA (DO-214AC)")
@@
   )
   (module Diodes_SMD:D_SMA (layer B.Cu)
-    (at 123.825 54.8875 270)
+    (at 123.825 53.578125 270)
     (descr "Diode SMA (DO-214AC)")
     (tags "Diode SMA (DO-214AC)")
@@
     )
   )
+  (segment (start 64.6 54.50625) (end 64.6 59.881875) (width 0.25) (layer B.Cu) (net 82))
+  (segment (start 64.6 59.881875) (end 64.368125 60.11375) (width 0.25) (layer B.Cu) (net 82))
+  (segment (start 64.368125 60.11375) (end 63.103125 60.11375) (width 0.25) (layer B.Cu) (net 82))
+  (segment (start 66.2 54.50625) (end 66.2 57.415625) (width 0.25) (layer B.Cu) (net 205))
+  (segment (start 66.2 57.415625) (end 69.346875 60.5625) (width 0.25) (layer B.Cu) (net 205))
+  (segment (start 69.346875 60.5625) (end 70.246875 60.5625) (width 0.25) (layer B.Cu) (net 205))
+  (segment (start 65.4 54.50625) (end 65.4 60.1875) (width 0.25) (layer B.Cu) (net 207))
+  (segment (start 65.4 60.1875) (end 65.775 60.5625) (width 0.25) (layer B.Cu) (net 207))
+  (segment (start 65.775 60.5625) (end 66.675 60.5625) (width 0.25) (layer B.Cu) (net 207))
 )

Commit message: Add SteppedCaps, More diodes
Parts:
- moved D_\1 291.3 mm to (309.6, 70.2)
- moved D_]1 285.2 mm to (302.8, 72.6), turned to 270 degrees
- moved D_DEL1 275.8 mm to (297.2, 53.6), turned to 270 degrees
- moved D_BACK1 275.8 mm to (295.3, 63.1)
- moved D_=1 271.6 mm to (293.0, 53.6), turned to 270 degrees
- moved D_[1 268.8 mm to (285.8, 72.6), turned to 270 degrees
- moved D_-1 255.1 mm to (276.2, 53.6), turned to 270 degrees
- moved D_P1 250.4 mm to (266.7, 72.6), turned to 270 degrees
- moved D_#0_1 236.5 mm to (257.2, 53.6), turned to 270 degrees
- moved D_O1 232.2 mm to (247.7, 72.6), turned to 270 degrees
- moved D_#9 217.9 mm to (238.1, 53.6), turned to 270 degrees
- moved D_I1 214.1 mm to (228.6, 72.6), turned to 270 degrees
- moved D_#8 199.5 mm to (219.1, 53.6), turned to 270 degrees
- moved D_U1 196.2 mm to (209.6, 72.6), turned to 270 degrees
- moved D_#7 181.1 mm to (200.0, 53.6), turned to 270 degrees
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
Commit message: Even more diodes
Parts:
- added K_CAPS2: MX-1.25U, MX_Alps_Hybrid:MX-1.25U, F.Cu at (59.5, 95.2)
- moved D_ENTER1 292.8 mm to (308.2, 81.5)
- moved D_ISO`1 280.8 mm to (292.5, 91.7), turned to 270 degrees
- moved D_'1 276.7 mm to (288.2, 91.7), turned to 270 degrees
- moved D_;1 260.9 mm to (271.5, 91.7), turned to 270 degrees
- moved D_L1 243.1 mm to (252.4, 91.7), turned to 270 degrees
- moved D_,1 242.1 mm to (242.9, 110.7), turned to 270 degrees
- moved D_K1 225.4 mm to (233.4, 91.7), turned to 270 degrees
- moved D_M1 225.2 mm to (223.8, 110.7), turned to 270 degrees
- moved D_N1 208.7 mm to (204.8, 110.7), turned to 270 degrees
- moved D_J1 208.1 mm to (214.3, 91.7), turned to 270 degrees
- moved D_B1 192.6 mm to (185.7, 110.7), turned to 270 degrees
- moved D_H1 191.0 mm to (195.3, 91.7), turned to 270 degrees
- moved D_V1 177.2 mm to (166.7, 110.7), turned to 270 degrees
- moved D_G1 173.2 mm to (176.2, 89.3), turned to 180 degrees
- moved D_C1 162.5 mm to (147.6, 110.7), turned to 270 degrees
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
Commit message: Further diodes
Parts:
- moved D_RSHIFT1 310.9 mm to (321.5, 100.0)
- moved D_UP1 286.6 mm to (291.7, 110.7), turned to 270 degrees
- moved D_/1 282.2 mm to (286.9, 110.7), turned to 270 degrees
- moved D_ALT1 280.4 mm to (276.2, 129.8), turned to 270 degrees
- moved D_FN1 263.6 mm to (257.2, 129.8), turned to 270 degrees
- moved D_.1 259.3 mm to (261.9, 110.7), turned to 270 degrees
- moved D_SPACE1 214.3 mm to (198.8, 129.8), turned to 270 degrees
- moved D_WIN1 145.2 mm to (96.4, 129.8), turned to 270 degrees
- moved D_CTRL1 134.4 mm to (70.2, 129.8), turned to 270 degrees

Commit message: Remove K_RCMD1
Overlapped perfectly with K_`1
No need
Parts:
- removed K_RCMD1: MX-1.5U, MX_Alps_Hybrid:MX-1.5U

Commit message: Finish diodes
Parts:
- moved D_RIGHT1 330.0 mm to (331.0, 129.2), turned to 270 degrees
- moved D_DOWN1 312.5 mm to (311.9, 129.2), turned to 270 degrees
- moved D_LEFT1 282.2 mm to (278.2, 129.8), turned to 270 degrees
- moved D_`1 278.5 mm to (274.0, 129.8), turned to 270 degrees
- moved D_ALT1 153.6 mm to (122.6, 129.8)

Commit message: Change crystal
Parts:
- Y1: footprint Crystals:Crystal_SMD_3225-4pin_3.2x2.5mm_HandSoldering -> Crystals:Crystal_SMD_EuroQuartz_X22-4pin_2.5x2.0mm_HandSoldering
- moved R_RIGHT1 331.2 mm to (311.9, 138.1), turned to 270 degrees
- moved R_\1 328.6 mm to (329.8, 81.0), turned to 270 degrees
- moved R_RSHIFT1 326.9 mm to (315.5, 119.1), turned to 270 degrees
- moved R_DOWN1 319.4 mm to (298.8, 138.1), turned to 270 degrees
- moved R_BACK1 313.8 mm to (319.1, 61.9), turned to 270 degrees
- moved R_UP1 311.5 mm to (298.8, 119.1), turned to 270 degrees
- moved R_ENTER1 311.4 mm to (306.0, 100.0), turned to 270 degrees
- moved R_DEL1 304.5 mm to (309.6, 61.9), turned to 270 degrees
- moved R_/1 302.2 mm to (288.1, 120.3), turned to 180 degrees
- moved R_LEFT1 299.8 mm to (276.2, 139.3)
- moved R_ISO`1 297.2 mm to (290.5, 101.2)
- moved RGB14 291.2 mm to (231.0, 177.4)
- moved R_]1 289.6 mm to (289.3, 81.0), turned to 270 degrees
- moved RGB13 286.5 mm to (225.0, 177.4)
- moved R_`1 285.7 mm to (260.7, 138.1), turned to 270 degrees
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Other:
- net class POWER added: clearance 0.2, trace_width 0.381, via_dia 0.6, via_drill 0.4

Commit message: Change crystal back
Parts:
- Y1: footprint Crystals:Crystal_SMD_EuroQuartz_X22-4pin_2.5x2.0mm_HandSoldering -> Crystals:Crystal_SMD_3225-4pin_3.2x2.5mm_HandSoldering
- moved C2 1.85 mm to (136.4, 131.8)
- moved C1 1.80 mm to (136.4, 139.7)
- moved Y1 1.20 mm to (137.0, 135.8)
- moved C4 0.63 mm to (137.4, 127.8)
Changed lines of the file:
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@@
   (general
     (links 641)
-    (no_connects 451)
+    (no_connects 448)
     (area 0 0 0 0)
     (thickness 1.6)
@@
   )
   (module Capacitors_SMD:C_0805_HandSoldering (layer B.Cu)
-    (at 138.176 139.954 180)
+    (at 136.398 139.7 180)
     (descr "Capacitor SMD 0805, hand soldering")
     (tags "capacitor 0805")
@@
   )
   (module Capacitors_SMD:C_0805_HandSoldering (layer B.Cu)
-    (at 138.176 131.318)
+    (at 136.398 131.826)
     (descr "Capacitor SMD 0805, hand soldering")
     (tags "capacitor 0805")
@@
   )
   (module Capacitors_SMD:C_0805_HandSoldering (layer B.Cu)
-    (at 136.921875 127.396875 180)
+    (at 137.434 127.762 180)
     (descr "Capacitor SMD 0805, hand soldering")
     (tags "capacitor 0805")
@@
     (pad "" np_thru_hole circle (at 5.08 0 48.0996) (size 1.7018 1.7018) (drill 1.7018) (layers *.Cu *.Mask))
   )
-  (module Crystals:Crystal_SMD_EuroQuartz_X22-4pin_2.5x2.0mm_HandSoldering (layer B.Cu)
-    (at 138.176 135.636 180)
-    (descr "SMD Crystal EuroQuartz X22 series http://cdn-reichelt.de/documents/datenblatt/B400/DS_X22.pdf, hand-soldering, 2.5x2.0mm^2 package")
+  (module Crystals:Crystal_SMD_3225-4pin_3.2x2.5mm_HandSoldering (layer B.Cu)
+    (at 136.98 135.77 180)
+    (descr "SMD Crystal SERIES SMD3225/4 http://www.txccrystal.com/images/pdf/7m-accuracy.pdf, hand-soldering, 3.2x2.5mm^2 package")
     (tags "SMD SMT crystal hand-soldering")
     (attr smd)
-    (fp_text reference Y1 (at 0 2.6 180) (layer B.SilkS)
+    (fp_text reference Y1 (at 0 3.05 180) (layer B.SilkS)
       (effects (font (size 1 1) (thickness 0.15)) (justify mirror))
     )
-    (fp_text value 16MHz (at 0 -2.6 180) (layer B.Fab)
+    (fp_text value 16MHz (at 0 -3.05 180) (layer B.Fab)
       (effects (font (size 1 1) (thickness 0.15)) (justify mirror))
     )
     (fp_text user %R (at 0 0 180) (layer B.Fab)
-      (effects (font (size 0.6 0.6) (thickness 0.09)) (justify mirror))
+      (effects (font (size 0.7 0.7) (thickness 0.105)) (justify mirror))
     )
-    (fp_line (start -1.15 1) (end 1.15 1) (layer B.Fab) (width 0.1))
-    (fp_line (start 1.15 1) (end 1.25 0.9) (layer B.Fab) (width 0.1))
-    (fp_line (start 1.25 0.9) (end 1.25 -0.9) (layer B.Fab) (width 0.1))
-    (fp_line (start 1.25 -0.9) (end 1.15 -1) (layer B.Fab) (width 0.1))
-    (fp_line (start 1.15 -1) (end -1.15 -1) (layer B.Fab) (width 0.1))
-    (fp_line (start -1.15 -1) (end -1.25 -0.9) (layer B.Fab) (width 0.1))
-    (fp_line (start -1.25 -0.9) (end -1.25 0.9) (layer B.Fab) (width 0.1))
-    (fp_line (start -1.25 0.9) (end -1.15 1) (layer B.Fab) (width 0.1))
-    (fp_line (start -1.25 0) (end -0.25 -1) (layer B.Fab) (width 0.1))
-    (fp_line (start -2.2 1.8) (end -2.2 -1.8) (layer B.SilkS) (width 0.12))
-    (fp_line (start -2.2 -1.8) (end 2.2 -1.8) (layer B.SilkS) (width 0.12))
-    (fp_line (start -2.3 1.9) (end -2.3 -1.9) (layer B.CrtYd) (width 0.05))
-    (fp_line (start -2.3 -1.9) (end 2.3 -1.9) (layer B.CrtYd) (width 0.05))
-    (fp_line (start 2.3 -1.9) (end 2.3 1.9) (layer B.CrtYd) (width 0.05))
-    (fp_line (start 2.3 1.9) (end -2.3 1.9) (layer B.CrtYd) (width 0.05))
-    (pad 1 smd rect (at -1.1 -0.85 180) (size 1.8 1.5) (layers B.Cu B.Paste B.Mask)
+    (fp_line (start -1.6 1.25) (end -1.6 -1.25) (layer B.Fab) (width 0.1))
+    (fp_line (start -1.6 -1.25) (end 1.6 -1.25) (layer B.Fab) (width 0.1))
+    (fp_line (start 1.6 -1.25) (end 1.6 1.25) (layer B.Fab) (width 0.1))
+    (fp_line (start 1.6 1.25) (end -1.6 1.25) (layer B.Fab) (width 0.1))
+    (fp_line (start -1.6 -0.25) (end -0.6 -1.25) (layer B.Fab) (width 0.1))
+    (fp_line (start -2.7 2.25) (end -2.7 -2.25) (layer B.SilkS) (width 0.12))
+    (fp_line (start -2.7 -2.25) (end 2.7 -2.25) (layer B.SilkS) (width 0.12))
+    (fp_line (start -2.8 2.3) (end -2.8 -2.3) (layer B.CrtYd) (width 0.05))
+    (fp_line (start -2.8 -2.3) (end 2.8 -2.3) (layer B.CrtYd) (width 0.05))
+    (fp_line (start 2.8 -2.3) (end 2.8 2.3) (layer B.CrtYd) (width 0.05))
+    (fp_line (start 2.8 2.3) (end -2.8 2.3) (layer B.CrtYd) (width 0.05))
+    (pad 1 smd rect (at -1.45 -1.15 180) (size 2.1 1.8) (layers B.Cu B.Paste B.Mask)
       (net 1 "Net-(C1-Pad1)"))
-    (pad 2 smd rect (at 1.1 -0.85 180) (size 1.8 1.5) (layers B.Cu B.Paste B.Mask)
+    (pad 2 smd rect (at 1.45 -1.15 180) (size 2.1 1.8) (layers B.Cu B.Paste B.Mask)
       (net 2 GND))
-    (pad 3 smd rect (at 1.1 0.85 180) (size 1.8 1.5) (layers B.Cu B.Paste B.Mask)
+    (pad 3 smd rect (at 1.45 1.15 180) (size 2.1 1.8) (layers B.Cu B.Paste B.Mask)
       (net 3 "Net-(C2-Pad1)"))
-    (pad 4 smd rect (at -1.1 0.85 180) (size 1.8 1.5) (layers B.Cu B.Paste B.Mask)
+    (pad 4 smd rect (at -1.45 1.15 180) (size 2.1 1.8) (layers B.Cu B.Paste B.Mask)
       (net 2 GND))
-    (model ${KISYS3DMOD}/Crystals.3dshapes/Crystal_SMD_EuroQuartz_X22-4pin_2.5x2.0mm_HandSoldering.wrl
+    (model ${KISYS3DMOD}/Crystals.3dshapes/Crystal_SMD_3225-4pin_3.2x2.5mm_HandSoldering.wrl
       (at (xyz 0 0 0))
       (scale (xyz 1 1 1))
