File: Chronos.kicad_pcb (KiCad board)
At the start: 2 copper layers, 285 x 94.6 mm, 256 parts, among them Q1 NSS40301MZ4T1G, SW1 SW_PUSH, U1 ATMEGA32U2-AU, Y1 16MHz

Commit message: Place and breakout the controller
Parts:
- moved R5 51.8 mm to (145.0, 125.7)
- moved C5 49.8 mm to (141.0, 140.4), turned to 180 degrees
- moved CR14 49.7 mm to (222.5, 189.5)
- moved CR13 45.2 mm to (214.9, 189.7)
- moved C6 44.7 mm to (146.3, 140.4)
- moved CR12 42.3 mm to (205.8, 191.5)
- moved R4 39.1 mm to (154.9, 133.9), turned to 180 degrees
- moved CR11 38.9 mm to (197.9, 190.5)
- moved R1 37.9 mm to (154.9, 136.7), turned to 180 degrees
- moved CR9 37.6 mm to (182.4, 189.5)
- moved CR8 37.5 mm to (175.8, 187.5)
- moved CR10 36.2 mm to (190.2, 188.7)
- moved CR7 24.1 mm to (213.4, 152.4)
- moved Q1 23.8 mm to (164.8, 131.3)
- moved CR6 17.7 mm to (207.0, 152.1)
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Connections:
- Q1 pad 2: GND -> LEDGND
- Q1 pad 3: LEDGND -> GND
Routing:
- net GND: track 0.00 -> 66.7 mm, vias 0 -> 3
- net +5V: track 0.00 -> 23.5 mm
- net Net-(R2-Pad1): track 0.00 -> 22.3 mm, vias 0 -> 1
- net Net-(R3-Pad1): track 0.00 -> 20.5 mm, vias 0 -> 1
- net Net-(U1-Pad26): track 0.00 -> 19.8 mm
- net Net-(U1-Pad25): track 0.00 -> 17.6 mm
- net Net-(U1-Pad22): track 0.00 -> 16.8 mm
- net Net-(U1-Pad23): track 0.00 -> 15.4 mm
- net Net-(C2-Pad1): track 0.00 -> 12.1 mm
- net Net-(U1-Pad20): track 0.00 -> 10.9 mm
- net Net-(U1-Pad5): track 0.00 -> 10.3 mm
- net Net-(U1-Pad19): track 0.00 -> 9.72 mm
- net Net-(U1-Pad6): track 0.00 -> 9.28 mm
- net Net-(U1-Pad18): track 0.00 -> 8.75 mm
- net Net-(C1-Pad1): track 0.00 -> 8.38 mm
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
Commit message: Finalize controller region with proper shielding
Parts:
- moved Q1 4.06 mm to (167.8, 128.5)
- moved C3 0.76 mm to (152.4, 140.4)
- moved C5 0.76 mm to (141.7, 140.4)
- moved C6 0.76 mm to (147.0, 140.4)
- turned R1 to 0 degrees
Routing:
- net GND: track 66.7 -> 82.3 mm, vias 3 -> 4
- net +5V: track 23.5 -> 35.7 mm, vias 0 -> 2
- net Net-(Q1-Pad1): track 5.51 -> 10.2 mm
- net Net-(R1-Pad2): track 3.56 -> 7.62 mm
- net Net-(C3-Pad1): track 7.48 -> 8.15 mm
- net Net-(U1-Pad25): track 17.6 -> 18.2 mm
- added copper zone on B.Cu, net GND
- added copper zone on F.Cu, net GND

Commit message: Undo controller and move it upwards
Parts:
- moved RGB1 51.9 mm to (164.3, 123.8), turned to 90 degrees
- moved R5 10.6 mm to (155.4, 127.5), turned to 90 degrees
- moved R_V1 3.64 mm to (166.6, 118.1), turned to 180 degrees
- moved Q1 3.06 mm to (167.5, 131.6)
- moved C1 1.37 mm to (135.4, 138.2)
- moved C2 1.37 mm to (135.4, 130.3)
- moved C4 1.37 mm to (136.4, 126.2)
- moved C5 1.37 mm to (142.2, 139.2)
- moved C6 1.37 mm to (147.6, 139.2)
- moved R4 1.37 mm to (155.4, 132.6)
- moved U1 1.37 mm to (146.6, 131.8)
- moved Y1 1.37 mm to (135.9, 134.2)
- moved C3 1.37 mm to (152.9, 139.2)
- moved R1 1.37 mm to (155.4, 135.4)
Routing:
- net GND: track 82.3 -> 69.6 mm, vias 4 -> 3
- net Net-(U1-Pad25): track 18.2 -> 8.02 mm
- net Net-(U1-Pad26): track 19.8 -> 9.78 mm
- net Net-(U1-Pad23): track 15.4 -> 7.01 mm
- net Net-(R5-Pad2): track 3.15 -> 10.1 mm, vias 0 -> 2
- net Net-(Q1-Pad1): track 10.2 -> 8.17 mm
- removed copper zone on B.Cu, net GND
- removed copper zone on F.Cu, net GND

Commit message: Finalize controller gnd
Parts:
- moved RGB3 53.4 mm to (240.5, 123.8), turned to 90 degrees
- moved RGB2 41.7 mm to (202.4, 123.8), turned to 90 degrees
- moved D_SPACE1 3.70 mm to (202.4, 132.6)
- moved R_,1 3.64 mm to (242.8, 118.1), turned to 180 degrees
- moved R_N1 3.64 mm to (204.7, 118.1), turned to 180 degrees
Routing:
- added copper zone on B.Cu, net GND
- added copper zone on F.Cu, net GND
Changed lines of the file:
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@@
   )
   (module WS2812B:WS2812B (layer B.Cu)
-    (at 201.215625 165.496875)
-    (fp_text reference RGB2 (at 0 4.7) (layer B.SilkS)
+    (at 202.40625 123.825 90)
+    (fp_text reference RGB2 (at 0 4.7 90) (layer B.SilkS)
       (effects (font (size 1 1) (thickness 0.2)) (justify mirror))
     )
-    (fp_text value WS2812B (at 0 -4.8) (layer B.SilkS) hide
+    (fp_text value WS2812B (at 0 -4.8 90) (layer B.SilkS) hide
       (effects (font (size 1 1) (thickness 0.2)) (justify mirror))
     )
@@
     (fp_line (start 2.5 2.5) (end 2.5 -2.5) (layer Dwgs.User) (width 0.2))
     (fp_line (start -2.49936 -2.49936) (end -2.49936 2.49936) (layer Dwgs.User) (width 0.2))
-    (pad 1 smd rect (at 1.65 2.4) (size 1.4 1.8) (layers B.Cu B.Paste B.Mask)
+    (pad 1 smd rect (at 1.65 2.4 90) (size 1.4 1.8) (layers B.Cu B.Paste B.Mask)
       (net 5 +5V))
-    (pad 2 smd rect (at -1.65 2.4) (size 1.4 1.8) (layers B.Cu B.Paste B.Mask)
+    (pad 2 smd rect (at -1.65 2.4 90) (size 1.4 1.8) (layers B.Cu B.Paste B.Mask)
       (net 208 "Net-(RGB2-Pad2)"))
-    (pad 3 smd rect (at -1.65 -2.4) (size 1.4 1.8) (layers B.Cu B.Paste B.Mask)
+    (pad 3 smd rect (at -1.65 -2.4 90) (size 1.4 1.8) (layers B.Cu B.Paste B.Mask)
       (net 2 GND))
-    (pad 4 smd rect (at 1.65 -2.4) (size 1.4 1.8) (layers B.Cu B.Paste B.Mask)
+    (pad 4 smd rect (at 1.65 -2.4 90) (size 1.4 1.8) (layers B.Cu B.Paste B.Mask)
       (net 206 "Net-(RGB1-Pad2)"))
   )
   (module WS2812B:WS2812B (layer B.Cu)
-    (at 207.16875 165.496875)
-    (fp_text reference RGB3 (at 0 4.7) (layer B.SilkS)
+    (at 240.50625 123.825 90)
+    (fp_text reference RGB3 (at 0 4.7 90) (layer B.SilkS)
       (effects (font (size 1 1) (thickness 0.2)) (justify mirror))
     )
-    (fp_text value WS2812B (at 0 -4.8) (layer B.SilkS) hide
+    (fp_text value WS2812B (at 0 -4.8 90) (layer B.SilkS) hide
       (effects (font (size 1 1) (thickness 0.2)) (justify mirror))
     )
@@
     (fp_line (start 2.5 2.5) (end 2.5 -2.5) (layer Dwgs.User) (width 0.2))
     (fp_line (start -2.49936 -2.49936) (end -2.49936 2.49936) (layer Dwgs.User) (width 0.2))
-    (pad 1 smd rect (at 1.65 2.4) (size 1.4 1.8) (layers B.Cu B.Paste B.Mask)
+    (pad 1 smd rect (at 1.65 2.4 90) (size 1.4 1.8) (layers B.Cu B.Paste B.Mask)
       (net 5 +5V))
-    (pad 2 smd rect (at -1.65 2.4) (size 1.4 1.8) (layers B.Cu B.Paste B.Mask)
+    (pad 2 smd rect (at -1.65 2.4 90) (size 1.4 1.8) (layers B.Cu B.Paste B.Mask)
       (net 209 "Net-(RGB3-Pad2)"))
-    (pad 3 smd rect (at -1.65 -2.4) (size 1.4 1.8) (layers B.Cu B.Paste B.Mask)
+    (pad 3 smd rect (at -1.65 -2.4 90) (size 1.4 1.8) (layers B.Cu B.Paste B.Mask)
       (net 2 GND))
-    (pad 4 smd rect (at 1.65 -2.4) (size 1.4 1.8) (layers B.Cu B.Paste B.Mask)
+    (pad 4 smd rect (at 1.65 -2.4 90) (size 1.4 1.8) (layers B.Cu B.Paste B.Mask)
       (net 208 "Net-(RGB2-Pad2)"))
   )
@@
   )
   (module Resistors_SMD:R_1206_HandSoldering (layer B.Cu)
-    (at 239.315625 119.0625 270)
+    (at 242.824 118.11 180)
     (descr "Resistor SMD 1206, hand soldering")
     (tags "resistor 1206")
     (attr smd)
-    (fp_text reference R_,1 (at 0 1.85 270) (layer B.SilkS)
+    (fp_text reference R_,1 (at 0 1.85 180) (layer B.SilkS)
       (effects (font (size 1 1) (thickness 0.15)) (justify mirror))
     )
-    (fp_text value 2.7k (at 0 -1.9 270) (layer B.Fab)
+    (fp_text value 2.7k (at 0 -1.9 180) (layer B.Fab)
       (effects (font (size 1 1) (thickness 0.15)) (justify mirror))
     )
-    (fp_text user %R (at 0 0 270) (layer B.Fab)
+    (fp_text user %R (at 0 0 180) (layer B.Fab)
       (effects (font (size 0.7 0.7) (thickness 0.105)) (justify mirror))
     )
@@
     (fp_line (start 3.25 -1.1) (end 3.25 1.11) (layer B.CrtYd) (width 0.05))
     (fp_line (start 3.25 -1.1) (end -3.25 -1.1) (layer B.CrtYd) (width 0.05))
-    (pad 1 smd rect (at -2 0 270) (size 2 1.7) (layers B.Cu B.Paste B.Mask)
+    (pad 1 smd rect (at -2 0 180) (size 2 1.7) (layers B.Cu B.Paste B.Mask)
       (net 2 GND))
-    (pad 2 smd rect (at 2 0 270) (size 2 1.7) (layers B.Cu B.Paste B.Mask)
+    (pad 2 smd rect (at 2 0 180) (size 2 1.7) (layers B.Cu B.Paste B.Mask)
       (net 101 "Net-(K_,1-Pad4)"))
     (model ${KISYS3DMOD}/Resistors_SMD.3dshapes/R_1206.wrl
@@
   )
   (module Resistors_SMD:R_1206_HandSoldering (layer B.Cu)
-    (at 201.215625 119.0625 270)
+    (at 204.724 118.11 180)
     (descr "Resistor SMD 1206, hand soldering")
     (tags "resistor 1206")
     (attr smd)
-    (fp_text reference R_N1 (at 0 1.85 270) (layer B.SilkS)
+    (fp_text reference R_N1 (at 0 1.85 180) (layer B.SilkS)
       (effects (font (size 1 1) (thickness 0.15)) (justify mirror))
     )
-    (fp_text value 2.7k (at 0 -1.9 270) (layer B.Fab)
+    (fp_text value 2.7k (at 0 -1.9 180) (layer B.Fab)
       (effects (font (size 1 1) (thickness 0.15)) (justify mirror))
     )
-    (fp_text user %R (at 0 0 270) (layer B.Fab)
+    (fp_text user %R (at 0 0 180) (layer B.Fab)
       (effects (font (size 0.7 0.7) (thickness 0.105)) (justify mirror))
     )
@@
     (fp_line (start 3.25 -1.1) (end 3.25 1.11) (layer B.CrtYd) (width 0.05))
     (fp_line (start 3.25 -1.1) (end -3.25 -1.1) (layer B.CrtYd) (width 0.05))
-    (pad 1 smd rect (at -2 0 270) (size 2 1.7) (layers B.Cu B.Paste B.Mask)
+    (pad 1 smd rect (at -2 0 180) (size 2 1.7) (layers B.Cu B.Paste B.Mask)
       (net 2 GND))
-    (pad 2 smd rect (at 2 0 270) (size 2 1.7) (layers B.Cu B.Paste B.Mask)
+    (pad 2 smd rect (at 2 0 180) (size 2 1.7) (layers B.Cu B.Paste B.Mask)
       (net 157 "Net-(K_N1-Pad4)"))
     (model ${KISYS3DMOD}/Resistors_SMD.3dshapes/R_1206.wrl
@@
   )
   (module Diodes_SMD:D_SMA (layer B.Cu)
-    (at 200.025 129.778125 270)
+    (at 202.438 132.588 270)
     (descr "Diode SMA (DO-214AC)")
     (tags "Diode SMA (DO-214AC)")
@@
   (segment (start 148.6035 136.06) (end 148.6035 137.11) (width 0.25) (layer B.Cu) (net 239))
   (segment (start 148.6035 137.11) (end 149.1615 137.668) (width 0.25) (layer B.Cu) (net 239))
+  (zone (net 2) (net_name GND) (layer B.Cu) (hatch edge 0.508)
+    (connect_pads (clearance 0.254))
+    (min_thickness 0.254)
+    (fill yes (arc_segments 16) (thermal_gap 0.508) (thermal_bridge_width 0.508))
+    (polygon
+      (pts
+        (xy 131.826 140.716) (xy 138.43 140.716) (xy 138.43 137.16) (xy 139.446 137.16) (xy 139.446 128.524)
+        (xy 131.826 128.524)
+      )
+    )
+  )
+  (zone (net 2) (net_name GND) (layer B.Cu) (hatch edge 0.508)
+    (connect_pads (clearance 0.254))
+    (min_thickness 0.254)
+    (fill yes (arc_segments 16) (thermal_gap 0.508) (thermal_bridge_width 0.508))
+    (polygon
+      (pts
+        (xy 131.826 127.762) (xy 140.208 127.762) (xy 140.208 137.922) (xy 139.192 137.922) (xy 139.192 140.716)
+        (xy 159.004 140.716) (xy 159.004 123.952) (xy 131.826 123.952)
+      )
+    )
+  )
+  (zone (net 2) (net_name GND) (layer F.Cu) (hatch edge 0.508)
+    (connect_pads (clearance 0.254))
+    (min_thickness 0.254)
+    (fill yes (arc_segments 16) (thermal_gap 0.508) (thermal_bridge_width 0.508))
+    (polygon
+      (pts
+        (xy 131.826 127.762) (xy 131.826 123.952) (xy 159.004 123.952) (xy 159.004 140.716) (xy 139.192 140.716)
+        (xy 139.192 137.922) (xy 140.208 137.922) (xy 140.208 135.636) (xy 139.446 135.636) (xy 139.446 137.16)
+        (xy 138.43 137.16) (xy 138.43 140.716) (xy 131.826 140.716) (xy 131.826 128.524) (xy 139.446 128.524)
+        (xy 139.446 130.81) (xy 140.208 130.81) (xy 140.208 127.762)
+      )
+    )
+  )
 )

Commit message: Finish via fencing
Routing:
- net GND: track 69.6 -> 134.1 mm, vias 3 -> 29
Changed lines of the file:
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@@
     (thickness 1.6)
     (drawings 19)
-    (tracks 219)
+    (tracks 272)
     (zones 0)
     (modules 256)
@@
   (segment (start 142.3535 134.61) (end 138.166 134.61) (width 0.25) (layer B.Cu) (net 1))
   (segment (start 138.166 134.61) (end 137.396 135.38) (width 0.25) (layer B.Cu) (net 1))
+  (segment (start 161.289 125.475) (end 160.274 124.46) (width 0.381) (layer B.Cu) (net 2))
+  (segment (start 161.90625 125.475) (end 161.289 125.475) (width 0.381) (layer B.Cu) (net 2))
+  (segment (start 130.556 129.286) (end 130.556 126.746) (width 0.381) (layer B.Cu) (net 2))
+  (via (at 130.556 126.746) (size 0.6) (drill 0.4) (layers F.Cu B.Cu) (net 2))
+  (segment (start 130.556 131.826) (end 130.556 129.286) (width 0.381) (layer F.Cu) (net 2))
+  (via (at 130.556 129.286) (size 0.6) (drill 0.4) (layers F.Cu B.Cu) (net 2))
+  (segment (start 130.556 134.366) (end 130.556 131.826) (width 0.381) (layer B.Cu) (net 2))
+  (via (at 130.556 131.826) (size 0.6) (drill 0.4) (layers F.Cu B.Cu) (net 2))
+  (segment (start 130.556 136.906) (end 130.556 134.366) (width 0.381) (layer F.Cu) (net 2))
+  (via (at 130.556 134.366) (size 0.6) (drill 0.4) (layers F.Cu B.Cu) (net 2))
+  (segment (start 130.556 139.446) (end 130.556 136.906) (width 0.381) (layer B.Cu) (net 2))
+  (via (at 130.556 136.906) (size 0.6) (drill 0.4) (layers F.Cu B.Cu) (net 2))
+  (segment (start 130.556 141.986) (end 130.556 139.446) (width 0.381) (layer F.Cu) (net 2))
+  (via (at 130.556 139.446) (size 0.6) (drill 0.4) (layers F.Cu B.Cu) (net 2))
+  (segment (start 132.334 141.986) (end 130.556 141.986) (width 0.381) (layer B.Cu) (net 2))
+  (via (at 130.556 141.986) (size 0.6) (drill 0.4) (layers F.Cu B.Cu) (net 2))
+  (segment (start 134.874 141.986) (end 132.334 141.986) (width 0.381) (layer F.Cu) (net 2))
+  (via (at 132.334 141.986) (size 0.6) (drill 0.4) (layers F.Cu B.Cu) (net 2))
+  (segment (start 137.414 141.986) (end 134.874 141.986) (width 0.381) (layer B.Cu) (net 2))
+  (via (at 134.874 141.986) (size 0.6) (drill 0.4) (layers F.Cu B.Cu) (net 2))
+  (segment (start 139.954 141.986) (end 137.414 141.986) (width 0.381) (layer F.Cu) (net 2))
+  (via (at 137.414 141.986) (size 0.6) (drill 0.4) (layers F.Cu B.Cu) (net 2))
+  (segment (start 142.494 141.986) (end 139.954 141.986) (width 0.381) (layer B.Cu) (net 2))
+  (via (at 139.954 141.986) (size 0.6) (drill 0.4) (layers F.Cu B.Cu) (net 2))
+  (segment (start 145.034 141.986) (end 142.494 141.986) (width 0.381) (layer F.Cu) (net 2))
+  (via (at 142.494 141.986) (size 0.6) (drill 0.4) (layers F.Cu B.Cu) (net 2))
+  (segment (start 147.574 141.986) (end 145.034 141.986) (width 0.381) (layer B.Cu) (net 2))
+  (via (at 145.034 141.986) (size 0.6) (drill 0.4) (layers F.Cu B.Cu) (net 2))
+  (segment (start 150.114 141.986) (end 147.574 141.986) (width 0.381) (layer F.Cu) (net 2))
+  (via (at 147.574 141.986) (size 0.6) (drill 0.4) (layers F.Cu B.Cu) (net 2))
+  (segment (start 152.654 141.986) (end 150.114 141.986) (width 0.381) (layer B.Cu) (net 2))
+  (via (at 150.114 141.986) (size 0.6) (drill 0.4) (layers F.Cu B.Cu) (net 2))
+  (segment (start 155.194 141.986) (end 152.654 141.986) (width 0.381) (layer F.Cu) (net 2))
+  (via (at 152.654 141.986) (size 0.6) (drill 0.4) (layers F.Cu B.Cu) (net 2))
+  (segment (start 157.734 141.986) (end 155.194 141.986) (width 0.381) (layer B.Cu) (net 2))
+  (via (at 155.194 141.986) (size 0.6) (drill 0.4) (layers F.Cu B.Cu) (net 2))
+  (segment (start 160.274 141.986) (end 157.734 141.986) (width 0.381) (layer F.Cu) (net 2))
+  (via (at 157.734 141.986) (size 0.6) (drill 0.4) (layers F.Cu B.Cu) (net 2))
+  (segment (start 160.274 139.446) (end 160.274 141.986) (width 0.381) (layer B.Cu) (net 2))
+  (via (at 160.274 141.986) (size 0.6) (drill 0.4) (layers F.Cu B.Cu) (net 2))
+  (segment (start 160.274 136.906) (end 160.274 139.446) (width 0.381) (layer F.Cu) (net 2))
+  (via (at 160.274 139.446) (size 0.6) (drill 0.4) (layers F.Cu B.Cu) (net 2))
+  (segment (start 160.274 134.366) (end 160.274 136.906) (width 0.381) (layer B.Cu) (net 2))
+  (via (at 160.274 136.906) (size 0.6) (drill 0.4) (layers F.Cu B.Cu) (net 2))
+  (segment (start 160.274 131.963) (end 160.274 134.366) (width 0.381) (layer F.Cu) (net 2))
+  (via (at 160.274 134.366) (size 0.6) (drill 0.4) (layers F.Cu B.Cu) (net 2))
+  (segment (start 160.274 129.54) (end 160.274 131.963) (width 0.381) (layer F.Cu) (net 2))
+  (via (at 160.274 131.963) (size 0.6) (drill 0.4) (layers F.Cu B.Cu) (net 2))
+  (segment (start 160.274 127) (end 160.274 129.54) (width 0.381) (layer B.Cu) (net 2))
+  (via (at 160.274 129.54) (size 0.6) (drill 0.4) (layers F.Cu B.Cu) (net 2))
+  (segment (start 160.274 124.46) (end 160.274 127) (width 0.381) (layer F.Cu) (net 2))
+  (via (at 160.274 127) (size 0.6) (drill 0.4) (layers F.Cu B.Cu) (net 2))
+  (via (at 160.274 124.46) (size 0.6) (drill 0.4) (layers F.Cu B.Cu) (net 2))
   (segment (start 155.448 130.302) (end 146.044058 130.302) (width 0.381) (layer F.Cu) (net 2))
   (segment (start 146.044058 130.302) (end 143.913 132.433058) (width 0.381) (layer F.Cu) (net 2))
@@
       )
     )
+  )
+  (zone (net 2) (net_name GND) (layer B.Cu) (hatch edge 0.508)
+    (connect_pads (clearance 0.254))
+    (min_thickness 0.254)
+    (fill yes (arc_segments 16) (thermal_gap 0.508) (thermal_bridge_width 0.508))
+    (polygon
+      (pts
+        (xy 159.004 141.478) (xy 131.064 141.478) (xy 131.064 123.952) (xy 130.302 123.952) (xy 130.302 142.24)
+        (xy 130.302 143.764) (xy 160.528 143.764) (xy 160.528 123.952) (xy 159.766 123.952) (xy 159.766 141.478)
+      )
+    )
+  )
+  (zone (net 2) (net_name GND) (layer F.Cu) (hatch edge 0.508)
+    (connect_pads (clearance 0.254))
+    (min_thickness 0.254)
+    (fill yes (arc_segments 16) (thermal_gap 0.508) (thermal_bridge_width 0.508))
+    (polygon
+      (pts
+        (xy 159.766 123.952) (xy 160.528 123.952) (xy 160.528 143.764) (xy 130.302 143.764) (xy 130.302 123.952)
+        (xy 131.064 123.952) (xy 131.064 141.478) (xy 159.766 141.478)
+      )
+    )

Commit message: Fix LED resistor pinout
Parts:
- moved Q1 0.48 mm to (167.9, 131.3)
Connections:
- R_#0_1 pad 1: GND -> LEDGND
- R_#1 pad 1: GND -> LEDGND
- R_#2 pad 1: GND -> LEDGND
- R_#3 pad 1: GND -> LEDGND
- R_#4 pad 1: GND -> LEDGND
- R_#5 pad 1: GND -> LEDGND
- R_#6 pad 1: GND -> LEDGND
- R_#7 pad 1: GND -> LEDGND
- R_#8 pad 1: GND -> LEDGND
- R_#9 pad 1: GND -> LEDGND
- R_'1 pad 1: GND -> LEDGND
- R_,1 pad 1: GND -> LEDGND
- R_-1 pad 1: GND -> LEDGND
- R_.1 pad 1: GND -> LEDGND
- R_/1 pad 1: GND -> LEDGND
- R_;1 pad 1: GND -> LEDGND
- R_=1 pad 1: GND -> LEDGND
- R_A1 pad 1: GND -> LEDGND
- R_ALT1 pad 1: GND -> LEDGND
- R_B1 pad 1: GND -> LEDGND
- R_BACK1 pad 1: GND -> LEDGND
- R_C1 pad 1: GND -> LEDGND
- R_CAPS1 pad 1: GND -> LEDGND
- R_CTRL1 pad 1: GND -> LEDGND
- R_D1 pad 1: GND -> LEDGND
- R_DEL1 pad 1: GND -> LEDGND
- R_DOWN1 pad 1: GND -> LEDGND
- R_E1 pad 1: GND -> LEDGND
- R_ENTER1 pad 1: GND -> LEDGND
- R_ESC1 pad 1: GND -> LEDGND
- R_F1 pad 1: GND -> LEDGND
- R_FN1 pad 1: GND -> LEDGND
- R_G1 pad 1: GND -> LEDGND
- R_H1 pad 1: GND -> LEDGND
- R_I1 pad 1: GND -> LEDGND
- R_ISO\1 pad 1: GND -> LEDGND
- R_ISO`1 pad 1: GND -> LEDGND
- R_J1 pad 1: GND -> LEDGND
- R_K1 pad 1: GND -> LEDGND
- R_L1 pad 1: GND -> LEDGND
- R_LEFT1 pad 1: GND -> LEDGND
- R_M1 pad 1: GND -> LEDGND
- R_N1 pad 1: GND -> LEDGND
- R_O1 pad 1: GND -> LEDGND
- R_P1 pad 1: GND -> LEDGND
- R_Q1 pad 1: GND -> LEDGND
- R_R1 pad 1: GND -> LEDGND
- R_RIGHT1 pad 1: GND -> LEDGND
- R_RSHIFT1 pad 1: GND -> LEDGND
- R_S1 pad 1: GND -> LEDGND
- R_SHIFT1 pad 1: GND -> LEDGND
- R_SPACE1 pad 1: GND -> LEDGND
- R_T1 pad 1: GND -> LEDGND
- R_TAB1 pad 1: GND -> LEDGND
- R_U1 pad 1: GND -> LEDGND
- R_UP1 pad 1: GND -> LEDGND
- R_V1 pad 1: GND -> LEDGND
- R_W1 pad 1: GND -> LEDGND
- R_WIN1 pad 1: GND -> LEDGND
- R_X1 pad 1: GND -> LEDGND
- R_Y1 pad 1: GND -> LEDGND
- R_Z1 pad 1: GND -> LEDGND
- R_[1 pad 1: GND -> LEDGND
- R_\1 pad 1: GND -> LEDGND
- R_]1 pad 1: GND -> LEDGND
- R_`1 pad 1: GND -> LEDGND
Routing:
- net GND: track 134.1 -> 69.6 mm, vias 29 -> 3
- net (no net): track 0.00 -> 43.2 mm, vias 0 -> 18
