File: Voyager.kicad_pcb (KiCad board)
At the start: 2 copper layers, 285 x 94.6 mm, 258 parts, among them Q1 NSS40301MZ4T1G, SW1 SW_PUSH, U1 ATMEGA32U2-AU, Y1 16MHz

Commit message: Move a resistor inwards
Parts:
- moved R_\1 3.23 mm to (327.7, 78.5)
Routing:
- net Net-(K_\1-Pad4): track 11.0 -> 8.41 mm
- net LEDGND: track 1298.7 -> 1296.8 mm
Changed lines of the file:
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@@
     (area 45.72 16.35 335.280001 147.0774)
     (thickness 1.6)
-    (drawings 78)
-    (tracks 3248)
+    (drawings 77)
+    (tracks 3246)
     (zones 0)
     (modules 258)
@@
   )
   (module Resistors_SMD:R_0805_HandSoldering (layer B.Cu)
-    (at 329.803125 80.9625 270)
+    (at 327.7235 78.486 270)
     (descr "Resistor SMD 0805, hand soldering")
     (tags "resistor 0805")
     (attr smd)
-    (fp_text reference R_\1 (at 0 1.7 270) (layer B.SilkS)
+    (fp_text reference R_\1 (at -0.3175 1.8415 270) (layer B.SilkS)
       (effects (font (size 1 1) (thickness 0.15)) (justify mirror))
     )
@@
       (xy 0.065301 1.729321)) (layer B.SilkS) (width 0.01))
   )
+  (gr_line (start 332.994 81.661) (end 308.102 76.1365) (layer B.SilkS) (width 0.2))
   (gr_line (start 126.5555 99.06) (end 52.07 104.775) (layer F.SilkS) (width 0.2))
   (gr_line (start 176.0855 95.25) (end 130.683 98.7425) (layer F.SilkS) (width 0.2))
@@
   (gr_line (start 153.7335 91.186) (end 90.9955 79.502) (layer B.SilkS) (width 0.2))
   (gr_line (start 176.149 95.377) (end 155.702 91.567) (layer B.SilkS) (width 0.2))
-  (gr_line (start 327.0885 80.3275) (end 308.102 76.1365) (layer B.SilkS) (width 0.2))
-  (gr_line (start 332.994 81.661) (end 329.057 80.772) (layer B.SilkS) (width 0.2))
   (gr_line (start 191.7065 93.091) (end 176.149 95.377) (layer B.SilkS) (width 0.2))
   (gr_line (start 210.6295 90.3605) (end 193.548 92.837) (layer B.SilkS) (width 0.2))
@@
   (segment (start 320.363416 81.28) (end 320.904317 81.820901) (width 0.25) (layer B.Cu) (net 154))
   (segment (start 320.904317 81.820901) (end 322.054551 81.820901) (width 0.25) (layer B.Cu) (net 154))
-  (segment (start 322.054551 81.820901) (end 323.409843 80.465609) (width 0.25) (layer B.Cu) (net 154))
-  (segment (start 323.409843 80.465609) (end 327.056234 80.465609) (width 0.25) (layer B.Cu) (net 154))
-  (segment (start 327.056234 80.465609) (end 328.903125 82.3125) (width 0.25) (layer B.Cu) (net 154))
-  (segment (start 328.903125 82.3125) (end 329.803125 82.3125) (width 0.25) (layer B.Cu) (net 154))
+  (segment (start 322.054551 81.817517) (end 323.417568 80.4545) (width 0.25) (layer B.Cu) (net 154))
+  (segment (start 322.054551 81.820901) (end 322.054551 81.817517) (width 0.25) (layer B.Cu) (net 154))
+  (segment (start 323.417568 80.4545) (end 326.136 80.4545) (width 0.25) (layer B.Cu) (net 154))
+  (segment (start 326.136 80.4545) (end 326.7545 79.836) (width 0.25) (layer B.Cu) (net 154))
+  (segment (start 326.7545 79.836) (end 327.7235 79.836) (width 0.25) (layer B.Cu) (net 154))
   (segment (start 296.545 81.28) (end 295.895702 81.28) (width 0.25) (layer B.Cu) (net 155))
   (segment (start 290.221875 82.3125) (end 289.321875 82.3125) (width 0.25) (layer B.Cu) (net 155))
@@
   (segment (start 264.555298 139.446) (end 260.763375 139.446) (width 0.25) (layer B.Cu) (net 156))
   (segment (start 260.763375 139.446) (end 260.746875 139.4625) (width 0.25) (layer B.Cu) (net 156))
+  (segment (start 323.688099 78.584401) (end 325.1365 77.136) (width 0.381) (layer B.Cu) (net 157))
+  (segment (start 325.1365 77.136) (end 327.7235 77.136) (width 0.381) (layer B.Cu) (net 157))
+  (segment (start 311.386219 78.584401) (end 323.688099 78.584401) (width 0.381) (layer B.Cu) (net 157))
+  (segment (start 289.321875 79.6125) (end 297.45988 79.6125) (width 0.381) (layer B.Cu) (net 157))
+  (segment (start 297.45988 79.6125) (end 297.888001 80.040621) (width 0.381) (layer B.Cu) (net 157))
+  (segment (start 297.888001 80.040621) (end 309.929999 80.040621) (width 0.381) (layer B.Cu) (net 157))
+  (segment (start 309.929999 80.040621) (end 311.386219 78.584401) (width 0.381) (layer B.Cu) (net 157))
   (segment (start 127 118.11) (end 127.747481 117.362519) (width 0.381) (layer B.Cu) (net 157))
   (segment (start 127.747481 117.362519) (end 133.081481 117.362519) (width 0.381) (layer B.Cu) (net 157))
@@
   (segment (start 264.922 119.126) (end 264.922 118.618) (width 0.381) (layer F.Cu) (net 157))
   (via (at 264.922 118.618) (size 0.6) (drill 0.4) (layers F.Cu B.Cu) (net 157))
-  (segment (start 329.803125 79.6125) (end 328.772125 79.6125) (width 0.381) (layer B.Cu) (net 157))
-  (segment (start 328.563224 79.403599) (end 328.563224 79.389224) (width 0.381) (layer B.Cu) (net 157))
-  (segment (start 328.772125 79.6125) (end 328.563224 79.403599) (width 0.381) (layer B.Cu) (net 157))
-  (segment (start 328.563224 79.389224) (end 327.758401 78.584401) (width 0.381) (layer B.Cu) (net 157))
-  (segment (start 327.758401 78.584401) (end 311.386219 78.584401) (width 0.381) (layer B.Cu) (net 157))
-  (segment (start 311.386219 78.584401) (end 309.929999 80.040621) (width 0.381) (layer B.Cu) (net 157))
-  (segment (start 290.352875 79.6125) (end 289.321875 79.6125) (width 0.381) (layer B.Cu) (net 157))
-  (segment (start 309.929999 80.040621) (end 297.888001 80.040621) (width 0.381) (layer B.Cu) (net 157))
-  (segment (start 297.888001 80.040621) (end 297.45988 79.6125) (width 0.381) (layer B.Cu) (net 157))
-  (segment (start 297.45988 79.6125) (end 290.352875 79.6125) (width 0.381) (layer B.Cu) (net 157))
   (segment (start 319.0875 60.5625) (end 317.8645 60.5625) (width 0.381) (layer B.Cu) (net 157))
   (segment (start 317.8645 60.5625) (end 317.5 60.198) (width 0.381) (layer B.Cu) (net 157))

Commit message: Move yet another resistor inwards
Parts:
- moved R_LEFT1 0.87 mm to (276.2, 138.4)
Routing:
- net Net-(K_LEFT1-Pad4): track 21.3 -> 20.4 mm
- net LEDGND: track 1296.8 -> 1296.1 mm
Changed lines of the file:
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@@
     (thickness 1.6)
     (drawings 77)
-    (tracks 3246)
+    (tracks 3247)
     (zones 0)
     (modules 258)
@@
   )
   (module Resistors_SMD:R_0805_HandSoldering (layer B.Cu)
-    (at 276.225 139.303125)
+    (at 276.225 138.43)
     (descr "Resistor SMD 0805, hand soldering")
     (tags "resistor 0805")
@@
   (segment (start 247.908125 100.33) (end 248.840625 101.2625) (width 0.25) (layer B.Cu) (net 131))
   (segment (start 248.840625 101.2625) (end 248.840625 101.3625) (width 0.25) (layer B.Cu) (net 131))
+  (segment (start 277.575 138.43) (end 277.575 137.53) (width 0.25) (layer B.Cu) (net 132))
+  (segment (start 277.575 137.53) (end 278.083501 137.021499) (width 0.25) (layer B.Cu) (net 132))
+  (segment (start 278.083501 137.021499) (end 281.180797 137.021499) (width 0.25) (layer B.Cu) (net 132))
   (segment (start 292.236951 139.707501) (end 291.010549 139.707501) (width 0.25) (layer B.Cu) (net 132))
   (segment (start 291.010549 139.707501) (end 289.733048 138.43) (width 0.25) (layer B.Cu) (net 132))
   (segment (start 289.733048 138.43) (end 288.2225 138.43) (width 0.25) (layer B.Cu) (net 132))
-  (segment (start 278.014501 137.021499) (end 281.180797 137.021499) (width 0.25) (layer B.Cu) (net 132))
   (segment (start 281.180797 137.021499) (end 283.866799 139.707501) (width 0.25) (layer B.Cu) (net 132))
   (segment (start 283.866799 139.707501) (end 285.093201 139.707501) (width 0.25) (layer B.Cu) (net 132))
-  (segment (start 277.575 139.303125) (end 277.575 137.461) (width 0.25) (layer B.Cu) (net 132))
-  (segment (start 277.575 137.461) (end 278.014501 137.021499) (width 0.25) (layer B.Cu) (net 132))
   (segment (start 287.02 138.43) (end 286.370702 138.43) (width 0.25) (layer B.Cu) (net 132))
   (segment (start 286.370702 138.43) (end 285.093201 139.707501) (width 0.25) (layer B.Cu) (net 132))
@@
   (segment (start 264.555298 139.446) (end 260.763375 139.446) (width 0.25) (layer B.Cu) (net 156))
   (segment (start 260.763375 139.446) (end 260.746875 139.4625) (width 0.25) (layer B.Cu) (net 156))
+  (segment (start 274.875 138.43) (end 274.875 137.399) (width 0.381) (layer B.Cu) (net 157))
+  (segment (start 274.875 137.399) (end 274.2385 136.7625) (width 0.381) (layer B.Cu) (net 157))
+  (segment (start 274.2385 136.7625) (end 261.777875 136.7625) (width 0.381) (layer B.Cu) (net 157))
+  (segment (start 261.777875 136.7625) (end 260.746875 136.7625) (width 0.381) (layer B.Cu) (net 157))
+  (segment (start 298.846875 136.7625) (end 297.815875 136.7625) (width 0.381) (layer B.Cu) (net 157))
+  (segment (start 297.815875 136.7625) (end 297.559364 136.505989) (width 0.381) (layer B.Cu) (net 157))
+  (segment (start 297.559364 136.505989) (end 276.899011 136.505989) (width 0.381) (layer B.Cu) (net 157))
+  (segment (start 276.899011 136.505989) (end 274.975 138.43) (width 0.381) (layer B.Cu) (net 157))
+  (segment (start 274.975 138.43) (end 274.875 138.43) (width 0.381) (layer B.Cu) (net 157))
   (segment (start 323.688099 78.584401) (end 325.1365 77.136) (width 0.381) (layer B.Cu) (net 157))
   (segment (start 325.1365 77.136) (end 327.7235 77.136) (width 0.381) (layer B.Cu) (net 157))
@@
   (segment (start 119.222125 136.7625) (end 120.253125 136.7625) (width 0.381) (layer B.Cu) (net 157))
   (segment (start 260.746875 136.7625) (end 253.603125 136.7625) (width 0.381) (layer B.Cu) (net 157))
-  (segment (start 260.746875 136.7625) (end 273.365375 136.7625) (width 0.381) (layer B.Cu) (net 157))
-  (segment (start 273.365375 136.7625) (end 274.875 138.272125) (width 0.381) (layer B.Cu) (net 157))
-  (segment (start 274.875 138.272125) (end 274.875 139.303125) (width 0.381) (layer B.Cu) (net 157))
-  (segment (start 298.846875 136.7625) (end 297.815875 136.7625) (width 0.381) (layer B.Cu) (net 157))
-  (segment (start 297.815875 136.7625) (end 297.559364 136.505989) (width 0.381) (layer B.Cu) (net 157))
-  (segment (start 297.559364 136.505989) (end 277.772136 136.505989) (width 0.381) (layer B.Cu) (net 157))
-  (segment (start 277.772136 136.505989) (end 274.975 139.303125) (width 0.381) (layer B.Cu) (net 157))
-  (segment (start 274.975 139.303125) (end 274.875 139.303125) (width 0.381) (layer B.Cu) (net 157))
   (segment (start 311.94375 136.7625) (end 310.91275 136.7625) (width 0.381) (layer B.Cu) (net 157))
   (segment (start 310.91275 136.7625) (end 298.846875 136.7625) (width 0.381) (layer B.Cu) (net 157))

Commit message: Move caps diode to more reasonable location
Parts:
- moved D_CAPS1 7.87 mm to (74.9, 90.0), turned to 180 degrees
- moved SW1 1.59 mm to (77.2, 96.5)
Routing:
- net Net-(D_CAPS1-Pad2): track 28.7 -> 17.6 mm
- net ROW5: track 270.2 -> 276.0 mm
- net Net-(R1-Pad2): track 142.2 -> 143.7 mm
- net LEDGND: track 1296.1 -> 1297.1 mm
- net GND: track 1151.0 -> 1150.1 mm

Commit message: Fix logo on backside
Parts:
- removed G***: LOGO, ai03-logo:AI03-Silkscreen-3.5mm
- added REF**: ai03-20mil, ai03-logo:ai03-20mil, B.Cu at (208.8, 133.3)
Changed lines of the file:
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@@
 (kicad_pcb (version 4) (host pcbnew 4.0.6)
   (general
-    (links 708)
+    (links 0)
     (no_connects 0)
-    (area 45.72 16.35 335.280001 147.0774)
+    (area 31.680193 16.35 335.280001 147.0774)
     (thickness 1.6)
     (drawings 78)
@@
   (page A3)
   (layers
-    (0 F.Cu signal)
+    (0 F.Cu signal hide)
     (31 B.Cu signal)
     (32 B.Adhes user)
@@
     (35 F.Paste user)
     (36 B.SilkS user)
-    (37 F.SilkS user)
+    (37 F.SilkS user hide)
     (38 B.Mask user)
     (39 F.Mask user)
@@
     (pad 17 smd rect (at 2.286 2.286) (size 0.762 0.762) (layers F.Cu F.Paste F.Mask))
   )
-  (module ai03-logo:AI03-Silkscreen-3.5mm (layer B.Cu)
-    (at 56.7944 83.2612 180)
-    (fp_text reference G*** (at 0 -2.9845 180) (layer B.SilkS) hide
-      (effects (font (thickness 0.3)) (justify mirror))
-    )
-    (fp_text value LOGO (at 0.0635 2.794 180) (layer B.SilkS) hide
-      (effects (font (thickness 0.3)) (justify mirror))
-    )
-    (fp_poly (pts (xy 0.065301 1.729321) (xy 0.115554 1.727664) (xy 0.16198 1.725168) (xy 0.202718 1.721842)
-      (xy 0.2286 1.718784) (xy 0.35605 1.69642) (xy 0.479798 1.665647) (xy 0.599679 1.626547)
-      (xy 0.715528 1.579203) (xy 0.827179 1.523698) (xy 0.934466 1.460114) (xy 1.037225 1.388533)
-      (xy 1.13529 1.309038) (xy 1.228496 1.221711) (xy 1.231699 1.218482) (xy 1.318376 1.124528)
-      (xy 1.397088 1.025934) (xy 1.467762 0.922859) (xy 1.530325 0.815461) (xy 1.584705 0.7039)
-      (xy 1.630828 0.588334) (xy 1.668621 0.468923) (xy 1.698012 0.345824) (xy 1.718928 0.219196)
-      (xy 1.72763 0.138718) (xy 1.729989 0.100669) (xy 1.731225 0.055743) (xy 1.731396 0.006223)
-      (xy 1.730561 -0.045606) (xy 1.728778 -0.097461) (xy 1.726105 -0.147059) (xy 1.722599 -0.192116)
-      (xy 1.718318 -0.230348) (xy 1.718242 -0.230909) (xy 1.696346 -0.357219) (xy 1.665896 -0.480105)
-      (xy 1.626987 -0.599374) (xy 1.579716 -0.714833) (xy 1.524182 -0.826291) (xy 1.460481 -0.933554)
-      (xy 1.388709 -1.036429) (xy 1.308965 -1.134726) (xy 1.221345 -1.22825) (xy 1.20936 -1.240068)
-      (xy 1.115255 -1.325963) (xy 1.017137 -1.403614) (xy 0.914886 -1.473079) (xy 0.80838 -1.534416)
-      (xy 0.697498 -1.587683) (xy 0.582119 -1.63294) (xy 0.46212 -1.670244) (xy 0.337382 -1.699655)
-      (xy 0.210127 -1.720914) (xy 0.192703 -1.722648) (xy 0.167667 -1.724297) (xy 0.136644 -1.725824)
-      (xy 0.101259 -1.72719) (xy 0.063138 -1.728359) (xy 0.023903 -1.729293) (xy -0.014819 -1.729956)
-      (xy -0.051405 -1.730309) (xy -0.084228 -1.730317) (xy -0.111666 -1.729941) (xy -0.132092 -1.729144)
-      (xy -0.136237 -1.728849) (xy -0.262609 -1.713906) (xy -0.38666 -1.690067) (xy -0.508114 -1.65744)
-      (xy -0.626697 -1.616138) (xy -0.742132 -1.566269) (xy -0.854144 -1.507944) (xy -0.962458 -1.441272)
-      (xy -1.066798 -1.366365) (xy -1.091985 -1.34656) (xy -1.121061 -1.322125) (xy -1.154265 -1.29227)
-      (xy -1.189858 -1.25871) (xy -1.226101 -1.22316) (xy -1.261253 -1.187332) (xy -1.293577 -1.152941)
-      (xy -1.321332 -1.121702) (xy -1.327152 -1.114825) (xy -1.405579 -1.014265) (xy -1.475594 -0.910061)
-      (xy -1.537263 -0.802061) (xy -1.590654 -0.69011) (xy -1.635831 -0.574057) (xy -1.6519 -0.521854)
-      (xy -0.817418 -0.521854) (xy -0.817418 -0.757382) (xy -0.581891 -0.757382) (xy -0.581891 -0.521854)
-      (xy 0.568036 -0.521854) (xy 0.568036 -0.757382) (xy 0.803563 -0.757382) (xy 0.803563 -0.521854)
-      (xy 0.568036 -0.521854) (xy -0.581891 -0.521854) (xy -0.817418 -0.521854) (xy -1.6519 -0.521854)
-      (xy -1.672864 -0.453749) (xy -1.701817 -0.329034) (xy -1.721084 -0.212436) (xy -1.724677 -0.178209)
-      (xy -1.727371 -0.136653) (xy -1.729174 -0.089631) (xy -1.729629 -0.064654) (xy -0.581891 -0.064654)
-      (xy -0.581891 -0.300182) (xy -0.346364 -0.300182) (xy -0.346364 -0.064654) (xy -0.124691 -0.064654)
-      (xy -0.124691 -0.300182) (xy 0.110836 -0.300182) (xy 0.110836 -0.064654) (xy 0.346363 -0.064654)
-      (xy 0.346363 -0.300182) (xy 0.568036 -0.300182) (xy 0.568036 -0.064654) (xy 0.346363 -0.064654)
-      (xy 0.110836 -0.064654) (xy -0.124691 -0.064654) (xy -0.346364 -0.064654) (xy -0.581891 -0.064654)
-      (xy -1.729629 -0.064654) (xy -1.730097 -0.039006) (xy -1.730149 0.01336) (xy -1.72934 0.065604)
-      (xy -1.727679 0.115863) (xy -1.725176 0.162274) (xy -1.721841 0.202976) (xy -1.718803 0.2286)
-      (xy -1.696449 0.355728) (xy -1.687282 0.392546) (xy -0.346364 0.392546) (xy -0.346364 0.170873)
-      (xy -0.124691 0.170873) (xy -0.124691 0.392546) (xy 0.110836 0.392546) (xy 0.110836 0.170873)
-      (xy 0.346363 0.170873) (xy 0.346363 0.392546) (xy 0.110836 0.392546) (xy -0.124691 0.392546)
-      (xy -0.346364 0.392546) (xy -1.687282 0.392546) (xy -1.665671 0.479333) (xy -1.626584 0.599183)
-      (xy -1.579303 0.715045) (xy -1.523941 0.826686) (xy -1.502132 0.8636) (xy -0.124691 0.8636)
-      (xy -0.124691 0.628073) (xy 0.110836 0.628073) (xy 0.110836 0.8636) (xy -0.124691 0.8636)
-      (xy -1.502132 0.8636) (xy -1.460612 0.933873) (xy -1.389431 1.036372) (xy -1.310511 1.13395)
-      (xy -1.236307 1.213988) (xy -1.142806 1.302513) (xy -1.045015 1.382865) (xy -0.942913 1.455056)
-      (xy -0.836479 1.519095) (xy -0.725692 1.574993) (xy -0.610532 1.622759) (xy -0.490978 1.662405)
-      (xy -0.367009 1.69394) (xy -0.238605 1.717375) (xy -0.212437 1.721084) (xy -0.178277 1.724669)
-      (xy -0.136786 1.727356) (xy -0.089822 1.729155) (xy -0.039247 1.730076) (xy 0.013081 1.730128)
-      (xy 0.065301 1.729321)) (layer B.SilkS) (width 0.01))
+  (module ai03-logo:ai03-20mil (layer B.Cu)
+    (at 208.788 133.35 180)
+    (fp_text reference REF** (at 0 -5.08 180) (layer Dwgs.User)
+      (effects (font (size 1 1) (thickness 0.15)))
+    )
+    (fp_text value ai03-20mil (at 0 5.08 180) (layer Dwgs.User)
+      (effects (font (size 1 1) (thickness 0.15)))
+    )
+    (pad 4 smd rect (at -0.508 0.508 180) (size 0.508 0.508) (layers B.Cu B.Paste B.Mask))
+    (pad 5 smd rect (at -1.016 -0.508 180) (size 0.508 0.508) (layers B.Cu B.Paste B.Mask))
+    (pad 6 smd rect (at 0 -0.508 180) (size 0.508 0.508) (layers B.Cu B.Paste B.Mask))
+    (pad 7 smd rect (at 1.016 -0.508 180) (size 0.508 0.508) (layers B.Cu B.Paste B.Mask))
+    (pad 8 smd rect (at 0.508 0.508 180) (size 0.508 0.508) (layers B.Cu B.Paste B.Mask))
+    (pad 9 smd rect (at 0 1.524 180) (size 0.508 0.508) (layers B.Cu B.Paste B.Mask))
+    (pad 10 smd rect (at -1.524 -1.524 180) (size 0.508 0.508) (layers B.Cu B.Paste B.Mask))
+    (pad 11 smd rect (at 1.524 -1.524 180) (size 0.508 0.508) (layers B.Cu B.Paste B.Mask))
   )
   (dimension 48.196542 (width 0.3) (layer Dwgs.User)
@@
   (gr_line (start 176.149 95.25) (end 238.506 133.477) (layer F.SilkS) (width 0.2))
   (gr_line (start 160.3375 132.715) (end 134.4295 132.715) (layer F.SilkS) (width 0.2))
-  (gr_text www.ai03.me (at 56.134 87.1855) (layer B.SilkS)
+  (gr_text www.ai03.me (at 219.837 133.35) (layer B.SilkS)
     (effects (font (size 1.5 1.5) (thickness 0.3)) (justify mirror))
   )

Commit message: Finalize 1.0 with version text on PCB
Parts:
- moved REF** 0.38 mm to (209.2, 133.3)
Other:
- board text added: "Rev. 1.0"
Changed lines of the file:
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@@
 (kicad_pcb (version 4) (host pcbnew 4.0.6)
   (general
-    (links 0)
+    (links 708)
     (no_connects 0)
-    (area 31.680193 16.35 335.280001 147.0774)
+    (area 0 0 0 0)
     (thickness 1.6)
-    (drawings 78)
+    (drawings 80)
     (tracks 3246)
     (zones 0)
@@
   (page A3)
   (layers
-    (0 F.Cu signal hide)
+    (0 F.Cu signal)
     (31 B.Cu signal)
     (32 B.Adhes user)
@@
     (35 F.Paste user)
     (36 B.SilkS user)
-    (37 F.SilkS user hide)
+    (37 F.SilkS user)
     (38 B.Mask user)
     (39 F.Mask user)
@@
   (module Molex-0548190589:Molex-0548190589 (layer B.Cu)
     (at 66.2 50.00625 270)
-    (fp_text reference USB1 (at 2.032 0 540) (layer B.SilkS)
+    (fp_text reference USB1 (at 1.36525 0 540) (layer B.SilkS)
       (effects (font (size 1 1) (thickness 0.15)) (justify mirror))
     )
@@
   )
   (module ai03-logo:ai03-20mil (layer B.Cu)
-    (at 208.788 133.35 180)
+    (at 209.169 133.35 180)
     (fp_text reference REF** (at 0 -5.08 180) (layer Dwgs.User)
       (effects (font (size 1 1) (thickness 0.15)))
@@
     (pad 11 smd rect (at 1.524 -1.524 180) (size 0.508 0.508) (layers B.Cu B.Paste B.Mask))
   )
+  (gr_text "Rev. 1.0" (at 66.675 56.8325) (layer B.SilkS)
+    (effects (font (size 1 1) (thickness 0.15)) (justify mirror))
+  )
+  (gr_text "Rev. 1.0" (at 72.7075 128.3335) (layer F.SilkS)
+    (effects (font (size 1 1) (thickness 0.15)))
+  )
   (dimension 48.196542 (width 0.3) (layer Dwgs.User)
     (gr_text "48.197 mm" (at 38.180192 72.374081 270.0754885) (layer Dwgs.User)
@@
   (gr_line (start 238.506 133.477) (end 308.102 76.073) (layer F.SilkS) (width 0.2))
   (gr_line (start 176.149 95.25) (end 238.506 133.477) (layer F.SilkS) (width 0.2))
-  (gr_line (start 160.3375 132.715) (end 134.4295 132.715) (layer F.SilkS) (width 0.2))
-  (gr_text www.ai03.me (at 219.837 133.35) (layer B.SilkS)
-    (effects (font (size 1.5 1.5) (thickness 0.3)) (justify mirror))
+  (gr_line (start 160.3375 132.461) (end 134.4295 132.461) (layer F.SilkS) (width 0.2))
+  (gr_text www.ai03.me (at 218.5035 133.35) (layer B.SilkS)
+    (effects (font (size 1 1) (thickness 0.2)) (justify mirror))
   )
   (gr_text "An endless journey into the unknown." (at 218.2495 104.775) (layer B.SilkS)
-    (effects (font (size 1.5 1.5) (thickness 0.3)) (justify mirror))
+    (effects (font (size 1.5 1.5) (thickness 0.25)) (justify mirror))
   )
-  (gr_text "VOYAGER\n" (at 147.3073 126.6444) (layer F.SilkS)
-    (effects (font (size 2.54 3.556) (thickness 0.3)))
+  (gr_text "VOYAGER\n" (at 147.3073 126.3904) (layer F.SilkS)
+    (effects (font (size 2.54 3.556) (thickness 0.35)))
   )
   (gr_text VOYAGER (at 254.6985 104.775) (layer B.SilkS)
-    (effects (font (size 3.048 4.064) (thickness 0.3)) (justify mirror))
+    (effects (font (size 3.048 4.064) (thickness 0.35)) (justify mirror))
   )
-  (gr_text www.ai03.me (at 72.771 141.351) (layer F.SilkS)
-    (effects (font (size 1.5 1.5) (thickness 0.3)))
+  (gr_text www.ai03.me (at 72.5805 138.3665) (layer F.SilkS)
+    (effects (font (size 1 1) (thickness 0.15)))
   )
-  (gr_text "\n60% keyboard PCB\n\nDesigned by ai03\n60% outline by amtra5\n" (at 147.3073 132.9944) (layer F.SilkS)
-    (effects (font (size 1.5 1.5) (thickness 0.3)))
+  (gr_text "\n60% keyboard PCB\n\nDesigned by ai03\n60% outline by amtra5\n" (at 147.3073 132.7404) (layer F.SilkS)
+    (effects (font (size 1.5 1.5) (thickness 0.25)))
   )
   (gr_text "Isolate the entire GND trace on top both sides\nOn bottom on right" (at 144.272 35.052) (layer Cmts.User)
