File: Voyager.kicad_pcb (KiCad board)
At the start: 2 copper layers, 285 x 94.6 mm, 258 parts, among them Q1 NSS40301MZ4T1G, SW1 SW_PUSH, U1 ATMEGA32U2-AU, Y1 16MHz

Commit message: Connect all resistors
Routing:
- net Net-(K_SPACE1-Pad4): track 0.00 -> 22.7 mm
- net Net-(K_LEFT1-Pad4): track 0.00 -> 18.8 mm
- net Net-(K_ALT1-Pad4): track 0.00 -> 16.3 mm
- net Net-(K_RCTRL2-Pad4): track 0.00 -> 16.1 mm
- net Net-(K_ALT2-Pad4): track 0.00 -> 13.6 mm
- net Net-(K_CTRL1-Pad4): track 0.00 -> 11.3 mm
- net Net-(K_FN1-Pad4): track 0.00 -> 8.07 mm
- net Net-(K_DOWN1-Pad4): track 0.00 -> 7.85 mm
- net Net-(K_`1-Pad4): track 0.00 -> 7.28 mm
Changed lines of the file:
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@@
     (thickness 1.6)
     (drawings 78)
-    (tracks 698)
+    (tracks 752)
     (zones 0)
     (modules 258)
@@
   (segment (start 100.0125 97.175) (end 100.0125 97.075) (width 0.25) (layer B.Cu) (net 107))
   (segment (start 96.8575 100.33) (end 100.0125 97.175) (width 0.25) (layer B.Cu) (net 107))
+  (segment (start 115.57 138.43) (end 114.925438 138.43) (width 0.25) (layer B.Cu) (net 108))
+  (segment (start 114.925438 138.43) (end 113.644737 137.149299) (width 0.25) (layer B.Cu) (net 108))
+  (segment (start 113.644737 137.149299) (end 110.909451 137.149299) (width 0.25) (layer B.Cu) (net 108))
+  (segment (start 110.909451 137.149299) (end 109.62875 138.43) (width 0.25) (layer B.Cu) (net 108))
+  (segment (start 109.62875 138.43) (end 108.42625 138.43) (width 0.25) (layer B.Cu) (net 108))
+  (segment (start 115.57 138.43) (end 119.0825 138.43) (width 0.25) (layer B.Cu) (net 108))
+  (segment (start 119.0825 138.43) (end 122.2375 135.275) (width 0.25) (layer B.Cu) (net 108))
+  (segment (start 122.2375 135.275) (end 122.2375 135.175) (width 0.25) (layer B.Cu) (net 108))
+  (segment (start 86.83625 138.43) (end 87.480812 138.43) (width 0.25) (layer B.Cu) (net 109))
+  (segment (start 87.480812 138.43) (end 90.735812 135.175) (width 0.25) (layer B.Cu) (net 109))
+  (segment (start 90.735812 135.175) (end 95.9375 135.175) (width 0.25) (layer B.Cu) (net 109))
+  (segment (start 95.9375 135.175) (end 96.8375 135.175) (width 0.25) (layer B.Cu) (net 109))
+  (segment (start 86.83625 138.43) (end 84.61375 138.43) (width 0.25) (layer B.Cu) (net 109))
   (segment (start 177.4825 119.38) (end 182.5825 119.38) (width 0.25) (layer B.Cu) (net 110))
   (segment (start 182.5825 119.38) (end 185.7375 116.225) (width 0.25) (layer B.Cu) (net 110))
@@
   (segment (start 68.2825 100.33) (end 70.64375 97.96875) (width 0.25) (layer B.Cu) (net 114))
   (segment (start 70.64375 97.96875) (end 70.64375 97.86875) (width 0.25) (layer B.Cu) (net 114))
+  (segment (start 60.6425 138.43) (end 61.287062 138.43) (width 0.25) (layer B.Cu) (net 115))
+  (segment (start 61.287062 138.43) (end 64.542062 135.175) (width 0.25) (layer B.Cu) (net 115))
+  (segment (start 64.542062 135.175) (end 69.74375 135.175) (width 0.25) (layer B.Cu) (net 115))
+  (segment (start 69.74375 135.175) (end 70.64375 135.175) (width 0.25) (layer B.Cu) (net 115))
   (segment (start 129.8575 100.33) (end 134.9575 100.33) (width 0.25) (layer B.Cu) (net 116))
   (segment (start 134.9575 100.33) (end 138.1125 97.175) (width 0.25) (layer B.Cu) (net 116))
@@
   (segment (start 297.7625 58.975) (end 296.8625 58.975) (width 0.25) (layer B.Cu) (net 117))
   (segment (start 302.170438 58.975) (end 297.7625 58.975) (width 0.25) (layer B.Cu) (net 117))
+  (segment (start 306.07 138.43) (end 305.425438 138.43) (width 0.25) (layer B.Cu) (net 118))
+  (segment (start 305.425438 138.43) (end 302.964188 135.96875) (width 0.25) (layer B.Cu) (net 118))
+  (segment (start 302.964188 135.96875) (end 300.14375 135.96875) (width 0.25) (layer B.Cu) (net 118))
+  (segment (start 300.14375 135.96875) (end 299.24375 135.96875) (width 0.25) (layer B.Cu) (net 118))
   (segment (start 125.095 81.28) (end 130.195 81.28) (width 0.25) (layer B.Cu) (net 119))
   (segment (start 130.195 81.28) (end 133.35 78.125) (width 0.25) (layer B.Cu) (net 119))
@@
   (segment (start 151.62625 100.33) (end 154.78125 97.175) (width 0.25) (layer B.Cu) (net 122))
   (segment (start 154.78125 97.175) (end 154.78125 97.075) (width 0.25) (layer B.Cu) (net 122))
+  (segment (start 248.92 138.43) (end 252.4325 138.43) (width 0.25) (layer B.Cu) (net 123))
+  (segment (start 252.4325 138.43) (end 255.5875 135.275) (width 0.25) (layer B.Cu) (net 123))
+  (segment (start 255.5875 135.275) (end 255.5875 135.175) (width 0.25) (layer B.Cu) (net 123))
   (segment (start 167.9575 100.33) (end 167.312938 100.33) (width 0.25) (layer B.Cu) (net 124))
   (segment (start 167.312938 100.33) (end 164.057938 97.075) (width 0.25) (layer B.Cu) (net 124))
@@
   (segment (start 249.2575 100.33) (end 252.4125 97.175) (width 0.25) (layer B.Cu) (net 131))
   (segment (start 252.4125 97.175) (end 252.4125 97.075) (width 0.25) (layer B.Cu) (net 131))
+  (segment (start 294.16375 138.43) (end 293.519188 138.43) (width 0.25) (layer B.Cu) (net 132))
+  (segment (start 292.238487 137.149299) (end 289.503201 137.149299) (width 0.25) (layer B.Cu) (net 132))
+  (segment (start 293.519188 138.43) (end 292.238487 137.149299) (width 0.25) (layer B.Cu) (net 132))
+  (segment (start 289.503201 137.149299) (end 288.2225 138.43) (width 0.25) (layer B.Cu) (net 132))
+  (segment (start 288.2225 138.43) (end 287.02 138.43) (width 0.25) (layer B.Cu) (net 132))
+  (segment (start 287.02 138.43) (end 286.375438 138.43) (width 0.25) (layer B.Cu) (net 132))
+  (segment (start 286.375438 138.43) (end 283.120438 135.175) (width 0.25) (layer B.Cu) (net 132))
+  (segment (start 278.7125 135.175) (end 277.8125 135.175) (width 0.25) (layer B.Cu) (net 132))
+  (segment (start 283.120438 135.175) (end 278.7125 135.175) (width 0.25) (layer B.Cu) (net 132))
   (segment (start 215.5825 119.38) (end 220.6825 119.38) (width 0.25) (layer B.Cu) (net 133))
   (segment (start 220.6825 119.38) (end 223.8375 116.225) (width 0.25) (layer B.Cu) (net 133))
@@
   (segment (start 149.245 81.28) (end 152.4 78.125) (width 0.25) (layer B.Cu) (net 138))
   (segment (start 152.4 78.125) (end 152.4 78.025) (width 0.25) (layer B.Cu) (net 138))
+  (segment (start 325.12 138.43) (end 324.475438 138.43) (width 0.25) (layer B.Cu) (net 139))
+  (segment (start 318.462062 138.43) (end 317.8175 138.43) (width 0.25) (layer B.Cu) (net 139))
+  (segment (start 324.475438 138.43) (end 323.194737 137.149299) (width 0.25) (layer B.Cu) (net 139))
+  (segment (start 323.194737 137.149299) (end 319.742763 137.149299) (width 0.25) (layer B.Cu) (net 139))
+  (segment (start 319.742763 137.149299) (end 318.462062 138.43) (width 0.25) (layer B.Cu) (net 139))
+  (segment (start 317.8175 138.43) (end 313.51125 138.43) (width 0.25) (layer B.Cu) (net 139))
+  (segment (start 311.15 136.06875) (end 311.15 135.96875) (width 0.25) (layer B.Cu) (net 139))
+  (segment (start 313.51125 138.43) (end 311.15 136.06875) (width 0.25) (layer B.Cu) (net 139))
   (segment (start 325.12 119.38) (end 324.475438 119.38) (width 0.25) (layer B.Cu) (net 140))
   (segment (start 316.01875 116.125) (end 315.11875 116.125) (width 0.25) (layer B.Cu) (net 140))
@@
   (segment (start 74.6125 117.01875) (end 74.6125 116.91875) (width 0.25) (layer B.Cu) (net 143))
   (segment (start 72.25125 119.38) (end 74.6125 117.01875) (width 0.25) (layer B.Cu) (net 143))
+  (segment (start 182.346951 137.149299) (end 189.484 137.16) (width 0.25) (layer B.Cu) (net 144))
+  (segment (start 189.484 137.16) (end 188.615263 137.149299) (width 0.25) (layer B.Cu) (net 144))
+  (segment (start 191.77 138.43) (end 191.125438 138.43) (width 0.25) (layer B.Cu) (net 144))
+  (segment (start 191.125438 138.43) (end 189.855438 137.16) (width 0.25) (layer B.Cu) (net 144))
+  (segment (start 189.855438 137.16) (end 189.484 137.16) (width 0.25) (layer B.Cu) (net 144))
+  (segment (start 179.86375 138.43) (end 181.06625 138.43) (width 0.25) (layer B.Cu) (net 144))
+  (segment (start 181.06625 138.43) (end 182.346951 137.149299) (width 0.25) (layer B.Cu) (net 144))
+  (segment (start 191.77 138.43) (end 196.07625 138.43) (width 0.25) (layer B.Cu) (net 144))
+  (segment (start 196.07625 138.43) (end 199.23125 135.275) (width 0.25) (layer B.Cu) (net 144))
+  (segment (start 199.23125 135.275) (end 199.23125 135.175) (width 0.25) (layer B.Cu) (net 144))
   (segment (start 163.195 81.28) (end 168.295 81.28) (width 0.25) (layer B.Cu) (net 145))
   (segment (start 168.295 81.28) (end 171.45 78.125) (width 0.25) (layer B.Cu) (net 145))
@@
   (segment (start 301.625 78.91875) (end 301.625 78.81875) (width 0.25) (layer B.Cu) (net 155))
   (segment (start 299.26375 81.28) (end 301.625 78.91875) (width 0.25) (layer B.Cu) (net 155))
+  (segment (start 267.97 138.43) (end 270.68875 138.43) (width 0.25) (layer B.Cu) (net 156))
+  (segment (start 273.84375 135.275) (end 273.84375 135.175) (width 0.25) (layer B.Cu) (net 156))
+  (segment (start 270.68875 138.43) (end 273.84375 135.275) (width 0.25) (layer B.Cu) (net 156))
   (segment (start 66.2 54.50625) (end 66.2 57.4205) (width 0.25) (layer B.Cu) (net 160))
   (segment (start 66.2 57.4205) (end 68.342 59.5625) (width 0.25) (layer B.Cu) (net 160))
