File: Voyager.kicad_pcb (KiCad board)
At the start: 2 copper layers, 285 x 94.6 mm, 258 parts, among them Q1 NSS40301MZ4T1G, SW1 SW_PUSH, U1 ATMEGA32U2-AU, Y1 16MHz

Commit message: Connect a crap ton of traces
Parts:
- moved R_ISO\1 2.86 mm to (90.5, 119.1), turned to 180 degrees
- moved R_#1 2.25 mm to (85.7, 61.9), turned to 180 degrees
- moved R_ISO`1 2.25 mm to (289.7, 100.0), turned to 0 degrees
- moved R_N1 1.59 mm to (204.8, 119.1), turned to 180 degrees
- moved R_V1 1.59 mm to (166.7, 119.1), turned to 180 degrees
- moved R_.1 1.59 mm to (261.9, 119.1), turned to 180 degrees
- moved R_,1 1.59 mm to (242.9, 119.1), turned to 180 degrees
- moved R_A1 1.59 mm to (100.0, 100.0), turned to 180 degrees
- moved R_ALT1 1.59 mm to (122.2, 138.1), turned to 180 degrees
- moved R_B1 1.59 mm to (185.7, 119.1), turned to 180 degrees
- moved R_C1 1.59 mm to (147.6, 119.1), turned to 180 degrees
- moved R_CTRL1 1.59 mm to (70.6, 138.1), turned to 180 degrees
- moved R_D1 1.59 mm to (138.1, 100.0), turned to 180 degrees
- moved R_E1 1.59 mm to (133.3, 81.0), turned to 180 degrees
- moved R_FN1 1.59 mm to (255.6, 138.1), turned to 180 degrees
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Routing:
- net +5V: track 0.00 -> 1359.8 mm
- net LEDGND: track 0.00 -> 1110.8 mm
- net GND: track 0.00 -> 574.5 mm, vias 0 -> 6
- net COL5: track 0.00 -> 214.9 mm
- net COL6: track 0.00 -> 199.7 mm
- net COL3: track 0.00 -> 192.8 mm
- net COL1: track 0.00 -> 191.0 mm
- net /D_P: track 0.00 -> 166.4 mm, vias 0 -> 2
- net /D_N: track 0.00 -> 165.8 mm, vias 0 -> 2
- net COL4: track 0.00 -> 158.1 mm
- net COL2: track 0.00 -> 157.2 mm
- net COL0: track 21.8 -> 175.8 mm
- net Net-(R1-Pad2): track 0.00 -> 127.7 mm, vias 0 -> 2
- net ROW8: track 136.7 -> 255.0 mm
- net COL7: track 0.00 -> 115.5 mm
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- added copper zone on B.Cu, net GND
- added copper zone on F.Cu, net GND

Commit message: Progress controller
Routing:
- net GND: track 574.5 -> 633.4 mm, vias 6 -> 24
- net ROW7: track 218.9 -> 239.5 mm, vias 0 -> 2
- net COL2: track 157.2 -> 167.7 mm, vias 0 -> 1
- net ROW9: track 202.4 -> 204.1 mm
- net ROW8: track 255.0 -> 256.3 mm
- net Net-(C3-Pad1): track 8.34 -> 9.02 mm

Commit message: Switch pins, connect some bottom rows
Connections:
- U1 pad 7: COL2 -> ROW7
- U1 pad 8: ROW7 -> COL2
Routing:
- net ROW9: track 204.1 -> 284.6 mm, vias 0 -> 4
- net ROW8: track 256.3 -> 335.8 mm, vias 0 -> 4
- net COL0: track 175.8 -> 233.7 mm, vias 0 -> 1
- net COL1: track 191.0 -> 222.5 mm, vias 0 -> 1
- net COL2: track 167.7 -> 174.3 mm
- net ROW7: track 239.5 -> 244.7 mm

Commit message: Work on controller breakout
Connections:
- U1 pad 17: COL7 -> COL4
- U1 pad 18: COL6 -> COL5
- U1 pad 19: COL5 -> COL6
- U1 pad 20: COL4 -> COL7
- U1 pad 22: COL3 -> RGBLED
- U1 pad 23: RGBLED -> COL3
Routing:
- net +5V: track 1359.8 -> 1566.0 mm
- net COL7: track 115.5 -> 305.1 mm, vias 0 -> 3
- net COL6: track 199.7 -> 343.0 mm, vias 0 -> 3
- net COL5: track 214.9 -> 327.0 mm, vias 0 -> 3
- net COL4: track 158.1 -> 249.6 mm, vias 0 -> 3
- net COL3: track 192.8 -> 221.6 mm
- net GND: track 633.4 -> 621.9 mm
- net ROW6: track 241.2 -> 245.0 mm, vias 0 -> 1
- net ROW4: track 204.8 -> 208.5 mm, vias 0 -> 1
- net ROW5: track 236.6 -> 240.2 mm, vias 0 -> 1
- net ROW3: track 247.3 -> 250.5 mm, vias 0 -> 1

Commit message: Even more progress
Connections:
- U1 pad 10: ROW5 -> ROW1
- U1 pad 15: ROW1 -> ROW5
- U1 pad 16: ROW0 -> ROW6
- U1 pad 9: ROW6 -> ROW0
Routing:
- net +5V: track 1566.0 -> 1848.5 mm, vias 0 -> 18
- net GND: track 621.9 -> 858.1 mm, vias 24 -> 28
- net ROW0: track 228.1 -> 315.8 mm, vias 0 -> 2
- net ROW1: track 225.9 -> 310.3 mm, vias 0 -> 2
- net Net-(RGB5-Pad2): track 0.00 -> 83.9 mm, vias 0 -> 2
- net ROW2: track 252.8 -> 330.1 mm, vias 0 -> 2
- net ROW3: track 250.5 -> 320.6 mm, vias 1 -> 2
- net Net-(RGB12-Pad2): track 0.00 -> 63.9 mm, vias 0 -> 2
- net ROW4: track 208.5 -> 250.9 mm, vias 1 -> 2
- net ROW5: track 240.2 -> 276.3 mm, vias 1 -> 2
- net ROW6: track 245.0 -> 261.7 mm, vias 1 -> 2
- net Net-(R5-Pad2): track 15.8 -> 11.7 mm
- net Net-(D_/1-Pad2): track 23.9 -> 26.1 mm
- net COL1: track 222.5 -> 221.3 mm
- net COL0: track 233.7 -> 232.5 mm
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
Commit message: Finalize revision 2.0
Parts:
- removed the REF** at (209.2, 133.3)
- added REF**: AI03-30Mil, ai03-logo:AI03-30Mil, B.Cu at (207.5, 133.3)
Routing:
- net LEDGND: track 1110.8 -> 1378.1 mm, vias 0 -> 20
- net +5V: track 1848.5 -> 1924.8 mm, vias 18 -> 20
- net Net-(D_K1-Pad2): track 0.00 -> 9.56 mm
- net Net-(D_ISO\1-Pad2): track 0.00 -> 9.35 mm
- net VCC: track 0.00 -> 6.23 mm
- net COL7: track 305.8 -> 309.9 mm
- net Net-(D_ALT1-Pad2): track 11.4 -> 14.0 mm
- net Net-(K_SHIFT1-Pad4): track 16.0 -> 17.5 mm
- net Net-(K_BACK1-Pad4): track 11.7 -> 12.9 mm
- net Net-(K_SPACE1-Pad4): track 22.7 -> 21.8 mm
- net ROW0: track 315.8 -> 316.6 mm
- net /D_P: track 166.4 -> 167.0 mm
- net /D_N: track 165.8 -> 166.4 mm
Other:
- net class Default: clearance 0.2032 -> 0.1524
- net class POWER: clearance 0.2032 -> 0.1524
- rule trace_clearance: 0.2032 -> 0.1524
- board text added: "Rev. 2.0"
- board text removed: "Rev. 1.0"
