File: Voyager.sch (KiCad schematic (older format))
At the start: 45 parts, among them Q1 NSS40301MZ4T1G, SW1 SW_PUSH, U1 ATMEGA32U2-AU, Y1 16MHz

Commit message: Update notes on schematic for Voyager 1.0 release
Other:
- note added: "1.0"
- note added: "Voyager Keyboard\n"
- note removed: "Chronos Keyboard\n"
Changed lines of the file:
@@
 LIBS:keyboard_parts
 LIBS:mkl27z256vfm4
-LIBS:Chronos-cache
+LIBS:Voyager-cache
 EELAYER 25 0
 EELAYER END
@@
 $EndSheet
 Text Notes 7350 7500 0    60   ~ 0
-Chronos Keyboard\n
+Voyager Keyboard\n
 Text Notes 8125 7650 0    60   ~ 0
 2017-10-15\n
@@
 Text Notes 5575 2825 0    50   ~ 0
 This is supposed to be a NPN transistor\nFor some reason KiCad keeps flipping the arrow the other way
+Text Notes 10550 7650 0    60   ~ 0
+1.0
 $EndSCHEMATC

Commit message: Switch pins, connect some bottom rows
Connections:
- net COL2: now also U1.8 ((RXD1/AIN1/INT2)PD2); no longer U1.7 ((AIN0/INT1)PD1)
- net ROW7: now also U1.7 ((AIN0/INT1)PD1); no longer U1.8 ((RXD1/AIN1/INT2)PD2)
Changed lines of the file:
@@
 Text GLabel 4250 2800 2    60   Input ~ 0
 COL0
-Text GLabel 4250 2900 2    60   Input ~ 0
+Text GLabel 4250 3000 2    60   Input ~ 0
 COL2
 Text GLabel 4250 3800 2    60   Input ~ 0
@@
 Text GLabel 4250 3100 2    60   Input ~ 0
 ROW6
-Text GLabel 4250 3000 2    60   Input ~ 0
+Text GLabel 4250 2900 2    60   Input ~ 0
 ROW7
 Text Notes 5575 2825 0    50   ~ 0

Commit message: Work on controller breakout
Connections:
- net COL3: now also U1.23 ((OC.1A/PCINT8)PC6); no longer U1.22 ((INT4/ICP1/CLK0)PC7)
- net COL4: now also U1.17 ((PD0/MISO/PCINT3)PB3); no longer U1.20 ((PCINT6)PB6)
- net COL5: now also U1.18 ((T1/PCINT4)PB4); no longer U1.19 ((PCINT5)PB5)
- net COL6: now also U1.19 ((PCINT5)PB5); no longer U1.18 ((T1/PCINT4)PB4)
- net COL7: now also U1.20 ((PCINT6)PB6); no longer U1.17 ((PD0/MISO/PCINT3)PB3)
- net RGBLED: now also U1.22 ((INT4/ICP1/CLK0)PC7); no longer U1.23 ((OC.1A/PCINT8)PC6)
Changed lines of the file:
@@
 Wire Wire Line
 	1175 1975 1275 1975
-Text GLabel 4250 4000 2    60   Input ~ 0
+Text GLabel 4250 4100 2    60   Input ~ 0
 RGBLED
 Text Label 1825 3400 0    60   ~ 0
@@
 Text GLabel 4250 3900 2    60   Input ~ 0
 ROW8
-Text GLabel 4250 4100 2    60   Input ~ 0
+Text GLabel 4250 4000 2    60   Input ~ 0
 COL3
+Text GLabel 4250 2200 2    60   Input ~ 0
+COL4
+Text GLabel 4250 2300 2    60   Input ~ 0
+COL5
+Text GLabel 4250 2400 2    60   Input ~ 0
+COL6
 Text GLabel 4250 2500 2    60   Input ~ 0
-COL4
-Text GLabel 4250 2400 2    60   Input ~ 0
-COL5
-Text GLabel 4250 2300 2    60   Input ~ 0
-COL6
-Text GLabel 4250 2200 2    60   Input ~ 0
 COL7
 Text GLabel 4250 2100 2    60   Input ~ 0

Commit message: Even more progress
Connections:
- net ROW0: now also U1.9 ((TXD1/INT3)PD3); no longer U1.16 ((PDI/MOSI/PCINT2)PB2)
- net ROW1: now also U1.10 ((INT5/AIN3)PD4); no longer U1.15 ((SCLK/PCINT1)PB1)
- net ROW5: now also U1.15 ((SCLK/PCINT1)PB1); no longer U1.10 ((INT5/AIN3)PD4)
- net ROW6: now also U1.16 ((PDI/MOSI/PCINT2)PB2); no longer U1.9 ((TXD1/INT3)PD3)
Changed lines of the file:
@@
 Text GLabel 4250 2500 2    60   Input ~ 0
 COL7
-Text GLabel 4250 2100 2    60   Input ~ 0
+Text GLabel 4250 3100 2    60   Input ~ 0
 ROW0
-Text GLabel 4250 2000 2    60   Input ~ 0
+Text GLabel 4250 3200 2    60   Input ~ 0
 ROW1
 Text GLabel 4250 1900 2    60   Input ~ 0
@@
 Text GLabel 4250 3300 2    60   Input ~ 0
 ROW4
-Text GLabel 4250 3200 2    60   Input ~ 0
+Text GLabel 4250 2000 2    60   Input ~ 0
 ROW5
-Text GLabel 4250 3100 2    60   Input ~ 0
+Text GLabel 4250 2100 2    60   Input ~ 0
 ROW6
 Text GLabel 4250 2900 2    60   Input ~ 0

Commit message: Begin Revision 3
Connections:
- net COL0: no longer names the net of U1.6 ((OC.0B/INT0)PD0)
- net COL1: no longer names the net of U1.5 ((PCINT11/AIN2)PC2)
- net COL2: no longer names the net of U1.8 ((RXD1/AIN1/INT2)PD2)
- net COL3: no longer names the net of U1.23 ((OC.1A/PCINT8)PC6)
- net COL4: no longer names the net of U1.17 ((PD0/MISO/PCINT3)PB3)
- net COL5: no longer names the net of U1.18 ((T1/PCINT4)PB4)
- net COL6: no longer names the net of U1.19 ((PCINT5)PB5)
- net COL7: no longer names the net of U1.20 ((PCINT6)PB6)
- net ROW0: no longer names the net of U1.9 ((TXD1/INT3)PD3)
- net ROW1: no longer names the net of U1.10 ((INT5/AIN3)PD4)
- net ROW2: no longer names the net of U1.14 ((~SS~/PCINT0)PB0)
- net ROW3: no longer names the net of U1.12 ((~RTS~/AIN5/INT6)PD6)
- net ROW4: no longer names the net of U1.11 ((XCK/AIN4/PCINT12)PD5)
- net ROW5: no longer names the net of U1.15 ((SCLK/PCINT1)PB1)
- net ROW6: no longer names the net of U1.16 ((PDI/MOSI/PCINT2)PB2)
- net ROW7: no longer names the net of U1.7 ((AIN0/INT1)PD1)
- net ROW8: no longer names the net of U1.25 ((PCINT9/OC.1B)PC5)
- net ROW9: no longer names the net of U1.26 ((PCINT10)PC4)
Changed lines of the file:
@@
 Text Label 1825 3500 0    60   ~ 0
 D_N
-Text GLabel 4250 3700 2    60   Input ~ 0
-COL1
-Text GLabel 4250 2800 2    60   Input ~ 0
-COL0
-Text GLabel 4250 3000 2    60   Input ~ 0
-COL2
-Text GLabel 4250 3800 2    60   Input ~ 0
-ROW9
-Text GLabel 4250 3900 2    60   Input ~ 0
-ROW8
-Text GLabel 4250 4000 2    60   Input ~ 0
-COL3
-Text GLabel 4250 2200 2    60   Input ~ 0
-COL4
-Text GLabel 4250 2300 2    60   Input ~ 0
-COL5
-Text GLabel 4250 2400 2    60   Input ~ 0
-COL6
-Text GLabel 4250 2500 2    60   Input ~ 0
-COL7
-Text GLabel 4250 3100 2    60   Input ~ 0
-ROW0
-Text GLabel 4250 3200 2    60   Input ~ 0
-ROW1
-Text GLabel 4250 1900 2    60   Input ~ 0
-ROW2
-Text GLabel 4250 3400 2    60   Input ~ 0
-ROW3
-Text GLabel 4250 3300 2    60   Input ~ 0
-ROW4
-Text GLabel 4250 2000 2    60   Input ~ 0
-ROW5
-Text GLabel 4250 2100 2    60   Input ~ 0
-ROW6
-Text GLabel 4250 2900 2    60   Input ~ 0
-ROW7
 Text Notes 5575 2825 0    50   ~ 0
 This is supposed to be a NPN transistor\nFor some reason KiCad keeps flipping the arrow the other way
